File: logicconnectors.kicad_sch (KiCad schematic)
At the start: 26 parts, among them J1 USBC Socket, J2 CANConn, J3 HallConn, J4 Conn_ARM_JTAG_SWD_20, J5 UART2, J6 InputConn, J7 UART, J8 DriverBoardConn, U2 USBLC6-2P6, U3 TJA1051T-3

Commit message: drivers
Connections:
- net +3.3V: now also J8.15 (Pin_15)

Commit message: initial
Parts:
- removed J8: DriverBoardConn, symbol Connector:Conn_01x16_Pin
- added C34: 1u, symbol Device:C
- added J8: LogicConn2, symbol Connector_Generic:Conn_02x10_Counter_Clockwise
- added J9: LogicConn, symbol Connector_Generic:Conn_02x10_Counter_Clockwise
- added R1: 2.2k, symbol Device:R
- R1: value 1k -> 100
Connections:
- net +3.3V: now also J8.20 (Pin_20), J9.20 (Pin_20)
- net CUR1: now also J9.19 (Pin_19)
- net CUR2: now also J9.18 (Pin_18)
- net CUR3: now also J9.17 (Pin_17)
- net GND: now also C34.2, J8.11 (Pin_11), J9.11 (Pin_11)
- net H1: now also J9.8 (Pin_8)
- net H2: now also J9.9 (Pin_9)
- net H3: now also J9.10 (Pin_10)
- net IN_V: now also J8.2 (Pin_2)
- net L1: now also J9.5 (Pin_5)
- net L2: now also J9.6 (Pin_6)
- net L3: now also J9.7 (Pin_7)
- net P_FILTER1: now also J8.4 (Pin_4)
- net P_FILTER2: now also J8.5 (Pin_5)
- net P_FILTER3: now also J8.6 (Pin_6)
- net TEMPMOTOR: now also C34.1, R1.2; no longer J3.2 (Pin_2), R1.2
- net VSENSE1: now also J9.2 (Pin_2)
- net VSENSE2: now also J9.3 (Pin_3)
- net VSENSE3: now also J9.4 (Pin_4)
- net HALL1 renamed HALL1_IN
- net HALL2 renamed HALL2_IN
- net HALL3 renamed HALL3_IN
- new net +15V: J8.1 (Pin_1), J9.1 (Pin_1)
- new net CLEAR_HW_FAULT: J8.17 (Pin_17)
- new net CURR_TRIP_HIGH: J9.13 (Pin_13)
- new net CURR_TRIP_LOW: J9.12 (Pin_12)
- new net MOSTEMP1: J9.16 (Pin_16)
- new net MOSTEMP2: J9.15 (Pin_15)
- new net MOSTEMP3: J9.14 (Pin_14)
- new net POWER_STAGE_DISABLE: J8.19 (Pin_19)
- new net POWER_STAGE_LOCKOUT: J8.18 (Pin_18)
- new net TEMPMOTOR_IN: J3.2 (Pin_2), R1.1, R1.2
- new net VBIAS: J8.3 (Pin_3)
Other:
- moved on the sheet: J3, R1

Commit message: initial
Parts:
- removed J4: Conn_ARM_JTAG_SWD_20, symbol Connector:Conn_ARM_JTAG_SWD_20
- removed J7: UART, symbol Connector:Conn_01x04_Pin
- removed J8: LogicConn2, symbol Connector_Generic:Conn_02x10_Counter_Clockwise
- added J2: LogicConn2, Connector_PinHeader_2.54mm:PinHeader_2x06_P2.54mm_Vertical, symbol Connector_Generic:Conn_02x06_Counter_Clockwise
- added J7: JTAG, Connector_PinHeader_2.54mm:PinHeader_1x05_P2.54mm_Vertical, symbol Connector:Conn_01x05_Pin
- C24: renamed from C13; footprint (none) -> Capacitor_SMD:C_0805_2012Metric
- C25: renamed from C34; footprint (none) -> Capacitor_SMD:C_0805_2012Metric
- C26: renamed from C11; footprint (none) -> Capacitor_SMD:C_0805_2012Metric
- C27: renamed from C12; footprint (none) -> Capacitor_SMD:C_0805_2012Metric
- C5: footprint (none) -> Capacitor_SMD:C_0805_2012Metric
- J1: footprint (none) -> Connector_USB:USB_C_Receptacle_GCT_USB4105-xx-A_16P_TopMnt_Horizontal
- J1: renamed from J6; footprint (none) -> Connector_PinHeader_2.54mm:PinHeader_1x08_P2.54mm_Horizontal
- J3: renamed from J5; footprint (none) -> Connector_PinHeader_2.54mm:PinHeader_1x04_P2.54mm_Horizontal
- J5: renamed from J3; footprint (none) -> Connector_PinHeader_2.54mm:PinHeader_1x06_P2.54mm_Horizontal
- J6: renamed from J9; footprint (none) -> Connector_PinHeader_2.54mm:PinHeader_2x10_P2.54mm_Vertical
- J8: renamed from J2; footprint (none) -> Connector_PinHeader_2.54mm:PinHeader_1x04_P2.54mm_Horizontal
- R1, R3, R4, R5, R6: footprint (none) -> Resistor_SMD:R_0805_2012Metric
- R21: renamed from R7; footprint (none) -> Resistor_SMD:R_0805_2012Metric
- renumbered U3 to U6
Connections:
- net +3.3V: now also J2.12 (Pin_12), J7.1 (Pin_1)
- net +5V: now also U6.3 (VCC), J2.1 (Pin_1)
- net CLEAR_HW_FAULT: now also J2.9 (Pin_9)
- net GND: now also C26.2, C27.2, J2.7 (Pin_7), J2.8 (Pin_8), J7.5 (Pin_5)
- net IN_V: now also J2.2 (Pin_2)
- net NRST: now also J7.2 (Pin_2)
- net POWER_STAGE_DISABLE: now also J2.11 (Pin_11)
- net POWER_STAGE_LOCKOUT: now also J2.10 (Pin_10)
- net P_FILTER1: now also J2.4 (Pin_4)
- net P_FILTER2: now also J2.5 (Pin_5)
- net P_FILTER3: now also J2.6 (Pin_6)
- net SWCLK: now also J7.3 (Pin_3)
- net SWDIO: now also J7.4 (Pin_4)
- net VBIAS: now also J2.3 (Pin_3)
- no-connect marks 7 -> 2
Other:
- moved on the sheet: C26, C27, J3

Commit message: initial
Connections:
- net P_FILTER1 renamed AUX_FAULT
- net P_FILTER2 renamed SENS_FILTER_ENABLE
- net P_FILTER3 renamed AUX_ENABLE
Changed lines of the file:
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@@
+    )
+  )
+  (global_label "SENS_FILTER_ENABLE" (shape input) (at 142.24 101.6 180) (fields_autoplaced)
+    (effects (font (size 1.27 1.27)) (justify right))
+    (property "Intersheetrefs" "${INTERSHEET_REFS}" (at 120.0314 101.6 0)
+      (effects (font (size 1.27 1.27)) (justify right) hide)
     )
   )
@@
     )
   )
+  (global_label "AUX_FAULT" (shape input) (at 142.24 99.06 180) (fields_autoplaced)
+    (effects (font (size 1.27 1.27)) (justify right))
+    (property "Intersheetrefs" "${INTERSHEET_REFS}" (at 129.8888 99.06 0)
+      (effects (font (size 1.27 1.27)) (justify right) hide)
+    )
+  )
   (global_label "MOSTEMP1" (shape input) (at 163.83 52.705 0) (fields_autoplaced)
     (effects (font (size 1.27 1.27)) (justify left))
@@
     )
   )
-  (global_label "P_FILTER3" (shape input) (at 142.24 104.14 180) (fields_autoplaced)
-    (effects (font (size 1.27 1.27)) (justify right))
-    (property "Intersheetrefs" "${INTERSHEET_REFS}" (at 130.4332 104.14 0)
-      (effects (font (size 1.27 1.27)) (justify right) hide)
-    )
-  )
   (global_label "CANTx" (shape input) (at 101.6 160.02 180) (fields_autoplaced)
     (effects (font (size 1.27 1.27)) (justify right))
@@
     )
   )
-  (global_label "P_FILTER1" (shape input) (at 142.24 99.06 180) (fields_autoplaced)
-    (effects (font (size 1.27 1.27)) (justify right))
-    (property "Intersheetrefs" "${INTERSHEET_REFS}" (at 130.4332 99.06 0)
-      (effects (font (size 1.27 1.27)) (justify right) hide)
-    )
-  )
   (global_label "TX_SCL_MOSI" (shape input) (at 38.1 52.07 0) (fields_autoplaced)
     (effects (font (size 1.27 1.27)) (justify left))
@@
     )
   )
-  (global_label "P_FILTER2" (shape input) (at 142.24 101.6 180) (fields_autoplaced)
-    (effects (font (size 1.27 1.27)) (justify right))
-    (property "Intersheetrefs" "${INTERSHEET_REFS}" (at 130.4332 101.6 0)
-      (effects (font (size 1.27 1.27)) (justify right) hide)
-    )
-  )
   (global_label "TX_EXT2" (shape input) (at 41.91 92.075 0) (fields_autoplaced)
     (effects (font (size 1.27 1.27)) (justify left))
@@
     )
   )
+  (global_label "AUX_ENABLE" (shape input) (at 142.24 104.14 180) (fields_autoplaced)
+    (effects (font (size 1.27 1.27)) (justify right))
+    (property "Intersheetrefs" "${INTERSHEET_REFS}" (at 128.377 104.14 0)
+      (effects (font (size 1.27 1.27)) (justify right) hide)
+    )
+  )

Commit message: jlcpcb
Parts:
- removed J1: InputConn, Connector_PinHeader_2.54mm:PinHeader_1x08_P2.54mm_Horizontal, symbol Connector:Conn_01x08_Pin
- added J1: ServoConn, Connector_JST:JST_EH_S4B-EH_1x04_P2.50mm_Horizontal, symbol Connector:Conn_01x04_Pin
- added J4: ADCConn, Connector_JST:JST_EH_S6B-EH_1x06_P2.50mm_Horizontal, symbol Connector:Conn_01x06_Pin
- C27: MPN (none) -> C377773
- J1: MPN (none) -> C2765186
- J2: MPN (none) -> C225521
- J3, J8: footprint Connector_PinHeader_2.54mm:PinHeader_1x04_P2.54mm_Horizontal -> Connector_JST:JST_EH_S4B-EH_1x04_P2.50mm_Horizontal; MPN (none) -> C265068
- J5: footprint Connector_PinHeader_2.54mm:PinHeader_1x06_P2.54mm_Horizontal -> Connector_JST:JST_EH_S6B-EH_1x06_P2.50mm_Horizontal; MPN (none) -> C495208
- J6: MPN (none) -> C2685199
- J7: MPN (none) -> C124379
- R1: MPN (none) -> C17557
- R1: MPN (none) -> C17408
- R4: MPN (none) -> C17561
- R5: MPN (none) -> C118848
- U2: MPN (none) -> C2827693
- U6: footprint Package_SO:SOIC-8_3.9x4.9mm_P1.27mm -> Package_SO:SOP-8_3.9x4.9mm_P1.27mm; MPN (none) -> C5342108
Connections:
- net +3.3V: now also J1.2 (Pin_2), J4.1 (Pin_1)
- net +5V: now also J1.1 (Pin_1)
- net GND: now also J1.4 (Pin_4), J4.6 (Pin_6)
- net MISO_ADC_EXT2: now also J4.3 (Pin_3)
- net RX_SDA_NSS: now also J4.5 (Pin_5)
- net SCK_ADC_EXT: now also J4.2 (Pin_2)
- net TX_SCL_MOSI: now also J4.4 (Pin_4)
- net at R1.1: now also J1.3 (Pin_3)
Other:
- moved on the sheet: C5, J3, R1

Commit message: routinglogic
Parts:
- removed J3: UART2, Connector_JST:JST_EH_S4B-EH_1x04_P2.50mm_Horizontal, symbol Connector:Conn_01x04_Pin
- removed J6: LogicConn, Connector_PinHeader_2.54mm:PinHeader_2x10_P2.54mm_Vertical, symbol Connector_Generic:Conn_02x10_Counter_Clockwise
- added J10: LHConn, Connector_PinHeader_2.54mm:PinHeader_2x04_P2.54mm_Vertical, symbol Connector_Generic:Conn_02x04_Counter_Clockwise
- added J11: MosTempConn, Connector_PinHeader_2.54mm:PinHeader_2x04_P2.54mm_Vertical, symbol Connector_Generic:Conn_02x04_Counter_Clockwise
- added J12: LogicConn, Connector_PinHeader_2.54mm:PinHeader_2x06_P2.54mm_Vertical, symbol Connector_Generic:Conn_02x06_Counter_Clockwise
- added J6: UartSpi, Connector_JST:JST_EH_S5B-EH_1x05_P2.50mm_Horizontal, symbol Connector:Conn_01x05_Pin
- J1: JLCPosOffset (none) -> 0,1.27
- J1, J8: JLCPosOffset (none) -> 3.75,0
- J4, J5: JLCPosOffset (none) -> 6.25,0
- J7: JLCPosOffset (none) -> 5.08,0; JLCRotOffset (none) -> -90
- U2, U6: JLCRotOffset (none) -> -90
Connections:
- net +15V: now also J2.10 (Pin_10), J2.12 (Pin_12)
- net +3.3V: now also J12.1 (Pin_1), J12.2 (Pin_2), J6.1 (Pin_1); no longer J2.12 (Pin_12)
- net +5V: now also J8.1 (Pin_1); no longer J8.4 (Pin_4)
- net CLEAR_HW_FAULT: now also J2.8 (Pin_8); no longer J2.9 (Pin_9)
- net CUR1: now also J12.5 (Pin_5)
- net CUR2: now also J12.7 (Pin_7)
- net CUR3: now also J12.9 (Pin_9)
- net CURR_TRIP_HIGH: now also J11.2 (Pin_2)
- net CURR_TRIP_LOW: now also J11.1 (Pin_1)
- net GND: now also J2.11 (Pin_11), J2.9 (Pin_9), J8.4 (Pin_4), J10.3 (Pin_3), J10.5 (Pin_5), J11.4 (Pin_4), J11.5 (Pin_5), J12.6 (Pin_6), J12.8 (Pin_8), J6.5 (Pin_5); no longer J2.7 (Pin_7), J2.8 (Pin_8), J8.1 (Pin_1)
- net H1: now also J10.1 (Pin_1)
- net H2: now also J10.4 (Pin_4)
- net H3: now also J10.2 (Pin_2)
- net L1: now also J10.8 (Pin_8)
- net L2: now also J10.7 (Pin_7)
- net L3: now also J10.6 (Pin_6)
- net MOSTEMP1: now also J11.7 (Pin_7)
- net MOSTEMP2: now also J11.8 (Pin_8)
- net MOSTEMP3: now also J11.6 (Pin_6)
- net POWER_STAGE_DISABLE: no longer J2.11 (Pin_11)
- net POWER_STAGE_LOCKOUT: now also J2.7 (Pin_7); no longer J2.10 (Pin_10)
- net VSENSE1: now also J12.11 (Pin_11)
- net VSENSE2: now also J12.10 (Pin_10)
- net VSENSE3: now also J12.12 (Pin_12)
- net at R21.1, U6.6 (CANL): now also J8.3 (Pin_3); no longer J8.2 (Pin_2)
- net at R21.2, U6.7 (CANH): now also J8.2 (Pin_2); no longer J8.3 (Pin_3)
- new net EXT2_MOSI: J6.4 (Pin_4)
- new net EXT2_RX_MISO: J6.3 (Pin_3)
- new net EXT2_TX_SCK: J6.2 (Pin_2)
Other:
- moved on the sheet: C25, C5, J1, J2, J4, J5, J7, J8, R1

Commit message: routed
Connections:
- net AUX_ENABLE: now also J2.5 (Pin_5); no longer J2.6 (Pin_6)
- net CLEAR_HW_FAULT: now also J2.6 (Pin_6); no longer J2.8 (Pin_8)
- net GND: now also J11.3 (Pin_3); no longer J11.4 (Pin_4)
- net L1: now also J10.7 (Pin_7); no longer J10.8 (Pin_8)
- net L2: now also J10.6 (Pin_6); no longer J10.7 (Pin_7)
- net L3: now also J10.8 (Pin_8); no longer J10.6 (Pin_6)
- net POWER_STAGE_DISABLE: now also J11.4 (Pin_4)
- net POWER_STAGE_LOCKOUT: now also J2.3 (Pin_3); no longer J2.7 (Pin_7)
- net SENS_FILTER_ENABLE: now also J2.8 (Pin_8); no longer J2.5 (Pin_5)
- net VBIAS: now also J2.7 (Pin_7); no longer J2.3 (Pin_3)
- net VSENSE1: now also J12.12 (Pin_12); no longer J12.11 (Pin_11)
- net VSENSE3: now also J12.11 (Pin_11); no longer J12.12 (Pin_12)

Commit message: driversconnectors
Other:
- moved on the sheet: C25, J2, R1
