File: GigaVesc.kicad_sch (KiCad schematic)
At the start: 0 parts

Commit message: initial
Parts:
- added C1, C11, C13, C6, C9: 100n, Capacitor_SMD:C_0805_2012Metric, symbol Device:C
- added C10, C12, C5, C8: 10n, Capacitor_SMD:C_0805_2012Metric, symbol Device:C
- added C14, C15, C4, C7: 1u, Capacitor_SMD:C_0805_2012Metric, symbol Device:C
- added C2, C3: 15p, Capacitor_SMD:C_0805_2012Metric, symbol Device:C
- added D1: L_RUN, LED_SMD:LED_0805_2012Metric, symbol Device:LED
- added D2: L_FAULT, LED_SMD:LED_0805_2012Metric, symbol Device:LED
- added R1: 10k, Resistor_SMD:R_0805_2012Metric, symbol Device:R
- added R2: 3.3k, Resistor_SMD:R_0805_2012Metric, symbol Device:R
- added R3, R4: 220, Resistor_SMD:R_0805_2012Metric, symbol Device:R
- added SW1: BOOT, Button_Switch_SMD:SW_SPST_CK_RS282G05A3, symbol Switch:SW_Push_Dual
- added SW2: RST, Button_Switch_SMD:SW_SPST_CK_RS282G05A3, symbol Switch:SW_Push_Dual
- added U1: STM32F405RGT7, Package_QFP:LQFP-64_10x10mm_P0.5mm, symbol MCU_ST_STM32F4:STM32F405RGTx
- added U2: REF1933AIDDCT, Package_TO_SOT_SMD:SOT-23-5, symbol GigaVescSymbols:REF1933AIDDCT
- added Y1: Crystal, Crystal:Crystal_SMD_HC49-SD, symbol Device:Crystal
Connections:
- new net: C10.2, C11.2, C12.2, C13.2, C5.2, C6.2, C8.2, C9.2, U1.1 (VBAT), U1.19 (VDD), U1.32 (VDD), U1.48 (VDD), U1.64 (VDD)
- new net: D2.1 (K), R4.1
- new net: C2.1, U1.5 (PH0), Y1.2
- new net: D1.1 (K), R3.1
- new net: C4.1, U1.31 (VCAP_1)
- new net: C7.1, U1.47 (VCAP_2)
- new net: C3.2, U1.6 (PH1), Y1.1
- new net +3.3V: C10.1, C11.1, C12.1, C13.1, C5.1, C6.1, C8.1, C9.1, R1.1, SW1.1, SW1.3
- new net +5V: C14.1, U2.3 (EN), U2.4 (VIN)
- new net BOOT: R2.1, SW1.2, SW1.4, U1.60 (BOOT0)
- new net CANRx: U1.61 (PB8)
- new net CANTx: U1.62 (PB9)
- new net CLEAR_HW_FAULT: U1.4 (PC15)
- new net CUR1: U1.8 (PC0)
- new net CUR2: U1.9 (PC1)
- new net CUR3: U1.10 (PC2)
- new net CURR_TRIP_HIGH: U1.20 (PA4)
- new net CURR_TRIP_LOW: U1.21 (PA5)
- new net GND: C1.2, C14.2, C15.2, C2.2, C3.1, C4.2, C7.2, R2.2, R3.2, R4.2, SW2.2, SW2.4, U1.12 (VSSA), U1.18 (VSS), U1.63 (VSS), U2.2 (GND)
- new net H1: U1.43 (PA10)
- new net H2: U1.42 (PA9)
- new net H3: U1.41 (PA8)
- new net HALL1: U1.37 (PC6)
- new net HALL2: U1.38 (PC7)
- new net HALL3: U1.39 (PC8)
- new net HALL_FILTER_ENABLE: U1.59 (PB7)
- new net IMU_SCL: U1.29 (PB10)
- new net IMU_SDA: U1.30 (PB11)
- new net IN_V: U1.11 (PC3)
- new net L1: U1.36 (PB15)
- new net L2: U1.35 (PB14)
- new net L3: U1.34 (PB13)
- new net LED_FAULT: D2.2 (A), U1.54 (PD2)
- new net LED_RUN: D1.2 (A), U1.28 (PB2)
- new net MISO_ADC_EXT2: U1.22 (PA6)
- new net MOSTEMP1: U1.17 (PA3)
- new net MOSTEMP2: U1.26 (PB0)
- new net MOSTEMP3: U1.27 (PB1)
- new net NRST: C1.1, R1.2, SW2.1, SW2.3, U1.7 (NRST)
- new net POWER_STAGE_DISABLE: U1.57 (PB5)
- new net POWER_STAGE_LOCKOUT: U1.33 (PB12)
- new net P_FILTER1: U1.40 (PC9)
- new net P_FILTER2: U1.2 (PC13)
- new net P_FILTER3: U1.3 (PC14)
- new net RX_EXT2: U1.52 (PC11)
- new net RX_SDA_NSS: U1.50 (PA15)
- new net SCK_ADC_EXT: U1.25 (PC5), U1.55 (PB3)
- new net SENSOR_VOLTAGE_SELECT: U1.56 (PB4)
- new net SERVO: U1.58 (PB6)
- new net SWCLK: U1.49 (PA14)
- new net SWDIO: U1.46 (PA13)
- new net TEMPMOTOR: U1.24 (PC4)
- new net TX_EXT2: U1.51 (PC10)
- new net TX_SCL_MOSI: U1.23 (PA7)
- new net USBD+: U1.45 (PA12)
- new net USBD-: U1.44 (PA11)
- new net VBIAS: U2.1 (VBIAS)
- new net VREF: C15.1, U1.13 (VDDA), U2.5 (VREF)
- new net VSENSE1: U1.16 (PA2)
- new net VSENSE2: U1.15 (PA1)
- new net VSENSE3: U1.14 (PA0)
- no-connect marks 0 -> 1
Other:
- removed sheet LogicBoard
- added sheet AccelGyro (accelgyro.kicad_sch)
- added sheet LogicConnectors (logicconnectors.kicad_sch)
- added sheet LogicPower (logicpower.kicad_sch)
- added sheet Switches (Switches.kicad_sch)

Commit message: initial
Connections:
- net H1: now also U1.41 (PA8); no longer U1.43 (PA10)
- net H3: now also U1.43 (PA10); no longer U1.41 (PA8)
- net L1: now also U1.34 (PB13); no longer U1.36 (PB15)
- net L3: now also U1.36 (PB15); no longer U1.34 (PB13)
- net VSENSE1: now also U1.14 (PA0); no longer U1.16 (PA2)
- net VSENSE3: now also U1.16 (PA2); no longer U1.14 (PA0)
- net P_FILTER1 renamed AUX_FAULT
- net P_FILTER2 renamed SENS_FILTER_ENABLE
- net P_FILTER3 renamed AUX_ENABLE

Commit message: jlcpcb
Parts:
- removed SW1: BOOT, Button_Switch_SMD:SW_SPST_CK_RS282G05A3, symbol Switch:SW_Push_Dual
- removed SW2: RST, Button_Switch_SMD:SW_SPST_CK_RS282G05A3, symbol Switch:SW_Push_Dual
- added SW1: BOOT, Button_Switch_SMD:SW_SPST_Omron_B3FS-100xP, symbol Switch:SW_Push
- added SW3: RST, Button_Switch_SMD:SW_SPST_Omron_B3FS-100xP, symbol Switch:SW_Push
- C1: MPN (none) -> C282732
- C10: MPN (none) -> C83170
- C14: MPN (none) -> C28323
- C2: MPN (none) -> C520056
- D1: MPN (none) -> C434435
- D2: MPN (none) -> C131244
- R1: MPN (none) -> C2930231
- R2: MPN (none) -> C114531
- U1: MPN (none) -> C1337199
- U2: MPN (none) -> C2877564
- Y1: MPN (none) -> C12674
Connections:
- net +3.3V: now also SW1.1
- net BOOT: now also SW1.2
- net GND: now also SW3.2
- net NRST: now also SW3.1
Changed lines of the file:
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@@
   (junction (at 143.51 78.74) (diameter 0) (color 0 0 0 0)
   )
-  (junction (at 48.895 137.16) (diameter 0) (color 0 0 0 0)
-  )
   (junction (at 113.03 99.06) (diameter 0) (color 0 0 0 0)
   )
-  (junction (at 48.26 89.535) (diameter 0) (color 0 0 0 0)
-  )
   (junction (at 226.06 133.35) (diameter 0) (color 0 0 0 0)
   )
@@
   (junction (at 39.37 97.155) (diameter 0) (color 0 0 0 0)
   )
-  (junction (at 32.385 132.08) (diameter 0) (color 0 0 0 0)
-  )
   (junction (at 140.97 64.77) (diameter 0) (color 0 0 0 0)
   )
   (junction (at 146.05 175.26) (diameter 0) (color 0 0 0 0)
-  )
-  (junction (at 58.42 89.535) (diameter 0) (color 0 0 0 0)
   )
   (junction (at 113.03 91.44) (diameter 0) (color 0 0 0 0)
@@
     (stroke (width 0) (type default))
   )
-  (wire (pts (xy 32.385 137.16) (xy 34.925 137.16))
-    (stroke (width 0) (type default))
-  )
   (wire (pts (xy 140.97 78.74) (xy 143.51 78.74))
     (stroke (width 0) (type default))
@@
     (stroke (width 0) (type default))
   )
-  (wire (pts (xy 45.085 137.16) (xy 48.895 137.16))
-    (stroke (width 0) (type default))
-  )
   (wire (pts (xy 113.03 52.07) (xy 113.03 57.15))
     (stroke (width 0) (type default))
@@
     (stroke (width 0) (type default))
   )
-  (wire (pts (xy 48.26 84.455) (xy 48.26 89.535))
+  (wire (pts (xy 48.26 84.455) (xy 48.26 97.155))
     (stroke (width 0) (type default))
   )
@@
     (stroke (width 0) (type default))
   )
-  (wire (pts (xy 32.385 132.08) (xy 32.385 137.16))
-    (stroke (width 0) (type default))
-  )
   (wire (pts (xy 163.83 157.48) (xy 167.64 157.48))
     (stroke (width 0) (type default))
@@
     (stroke (width 0) (type default))
   )
-  (wire (pts (xy 48.26 89.535) (xy 48.26 97.155))
-    (stroke (width 0) (type default))
-  )
   (wire (pts (xy 106.68 91.44) (xy 113.03 91.44))
     (stroke (width 0) (type default))
@@
     (stroke (width 0) (type default))
   )
-  (wire (pts (xy 58.42 84.455) (xy 58.42 89.535))
+  (wire (pts (xy 58.42 84.455) (xy 58.42 92.075))
     (stroke (width 0) (type default))
   )
@@
     (stroke (width 0) (type default))
   )
-  (wire (pts (xy 58.42 89.535) (xy 58.42 92.075))
-    (stroke (width 0) (type default))
-  )
   (wire (pts (xy 109.22 167.64) (xy 115.57 167.64))
     (stroke (width 0) (type default))
@@
         (path "/768a484b-8a27-40cf-8cad-0f63935b1af0"
           (reference "C15") (unit 1)
+        )
+      )
+    )
+  )
+  (symbol (lib_id "Switch:SW_Push") (at 40.005 132.08 0) (unit 1)
+    (in_bom yes) (on_board yes) (dnp no) (fields_autoplaced)
+    (property "Reference" "SW1" (at 40.005 124.46 0)
+      (effects (font (size 1.27 1.27)))
+    )
+    (property "Value" "BOOT" (at 40.005 127 0)
+      (effects (font (size 1.27 1.27)))
+    )
+    (property "Footprint" "Button_Switch_SMD:SW_SPST_Omron_B3FS-100xP" (at 40.005 127 0)
+      (effects (font (size 1.27 1.27)) hide)
+    )
+    (property "Datasheet" "~" (at 40.005 127 0)
+      (effects (font (size 1.27 1.27)) hide)
+    )
+    (property "MPN" "C271750" (at 40.005 132.08 0)
+      (effects (font (size 1.27 1.27)) hide)
+    )
+    (pin "1")
+    (pin "2")
+    (instances
+      (project "GigaVesc"
+        (path "/768a484b-8a27-40cf-8cad-0f63935b1af0"
+          (reference "SW1") (unit 1)
+        )
+      )
+    )
+  )
+  (symbol (lib_id "Switch:SW_Push") (at 53.34 84.455 0) (unit 1)
+    (in_bom yes) (on_board yes) (dnp no) (fields_autoplaced)
+    (property "Reference" "SW3" (at 53.34 76.2 0)
+      (effects (font (size 1.27 1.27)))
+    )
+    (property "Value" "RST" (at 53.34 78.74 0)
+      (effects (font (size 1.27 1.27)))
+    )
+    (property "Footprint" "Button_Switch_SMD:SW_SPST_Omron_B3FS-100xP" (at 53.34 79.375 0)
+      (effects (font (size 1.27 1.27)) hide)
+    )
+    (property "Datasheet" "~" (at 53.34 79.375 0)
+      (effects (font (size 1.27 1.27)) hide)
+    )
+    (property "MPN" "C271750" (at 53.34 84.455 0)
+      (effects (font (size 1.27 1.27)) hide)
+    )
+    (pin "1")
+    (pin "2")
+    (instances
+      (project "GigaVesc"
+        (path "/768a484b-8a27-40cf-8cad-0f63935b1af0"
+          (reference "SW3") (unit 1)
         )
       )
@@
       (effects (font (size 1.27 1.27)) hide)
     )
+    (property "MPN" "C28323" (at 226.06 139.7 0)
+      (effects (font (size 1.27 1.27)) hide)
+    )
     (pin "1")
     (pin "2")
@@
       (effects (font (size 1.27 1.27)) hide)
     )
+    (property "MPN" "C520056" (at 102.87 91.44 90)
+      (effects (font (size 1.27 1.27)) hide)
+    )
     (pin "1")
     (pin "2")
@@
       (effects (font (size 1.27 1.27)) hide)
     )
+    (property "MPN" "C2930231" (at 39.37 93.345 90)
+      (effects (font (size 1.27 1.27)) hide)
+    )
     (pin "1")
     (pin "2")
@@
       (effects (font (size 1.27 1.27)) hide)
     )
+    (property "MPN" "C83170" (at 152.4 60.96 0)
+      (effects (font (size 1.27 1.27)) hide)
+    )
     (pin "1")
     (pin "2")
@@
     )
     (property "Datasheet" "~" (at 48.26 100.965 0)
+      (effects (font (size 1.27 1.27)) hide)
+    )
+    (property "MPN" "C282732" (at 48.26 100.965 0)
       (effects (font (size 1.27 1.27)) hide)
     )
@@
       (effects (font (size 1.27 1.27)) hide)
     )
+    (property "MPN" "C434435" (at 41.91 173.99 90)
+      (effects (font (size 1.27 1.27)) hide)
+    )
     (pin "1")
     (pin "2")
@@
       (effects (font (size 1.27 1.27)) hide)
     )
+    (property "MPN" "C131244" (at 41.91 182.88 90)
+      (effects (font (size 1.27 1.27)) hide)
+    )
     (pin "1")
     (pin "2")
@@
     )
     (property "Datasheet" "" (at 246.38 135.89 0)
+      (effects (font (size 1.27 1.27)) hide)
+    )
+    (property "MPN" "C2877564" (at 246.38 135.89 0)
       (effects (font (size 1.27 1.27)) hide)
     )
@@
       (effects (font (size 1.27 1.27)) hide)
     )
+    (property "MPN" "C114531" (at 48.895 140.97 90)
+      (effects (font (size 1.27 1.27)) hide)
+    )
     (pin "1")
     (pin "2")
@@
         (path "/768a484b-8a27-40cf-8cad-0f63935b1af0"
           (reference "R2") (unit 1)
-        )
-      )
-    )
-  )
-  (symbol (lib_id "Switch:SW_Push_Dual") (at 53.34 84.455 0) (unit 1)
-    (in_bom yes) (on_board yes) (dnp no) (fields_autoplaced)
-    (property "Reference" "SW2" (at 53.34 76.835 0)
-      (effects (font (size 1.27 1.27)))
-    )
-    (property "Value" "RST" (at 53.34 79.375 0)
-      (effects (font (size 1.27 1.27)))
-    )
-    (property "Footprint" "Button_Switch_SMD:SW_SPST_CK_RS282G05A3" (at 53.34 79.375 0)
-      (effects (font (size 1.27 1.27)) hide)
-    )
-    (property "Datasheet" "~" (at 53.34 79.375 0)
-      (effects (font (size 1.27 1.27)) hide)
-    )
-    (pin "1")
-    (pin "2")
-    (pin "3")
-    (pin "4")
-    (instances
-      (project "GigaVesc"
-        (path "/768a484b-8a27-40cf-8cad-0f63935b1af0"
-          (reference "SW2") (unit 1)
         )
       )
@@
       (effects (font (size 1.27 1.27)) hide)
     )
+    (property "MPN" "C12674" (at 113.03 95.25 90)
+      (effects (font (size 1.27 1.27)) hide)
+    )
     (pin "1")
     (pin "2")
@@
     )
     (property "Datasheet" "https://www.st.com/resource/en/datasheet/stm32f405rg.pdf" (at 146.05 127 0)
+      (effects (font (size 1.27 1.27)) hide)
+    )
+    (property "MPN" "C1337199" (at 146.05 127 0)
       (effects (font (size 1.27 1.27)) hide)
     )
@@
         )
       )
-    )
-  )
-  (symbol (lib_id "Switch:SW_Push_Dual") (at 40.005 132.08 0) (unit 1)
-    (in_bom yes) (on_board yes) (dnp no) (fields_autoplaced)
-    (property "Reference" "SW1" (at 40.005 124.46 0)
-      (effects (font (size 1.27 1.27)))
-    )
-    (property "Value" "BOOT" (at 40.005 127 0)
-      (effects (font (size 1.27 1.27)))
-    )
-    (property "Footprint" "Button_Switch_SMD:SW_SPST_CK_RS282G05A3" (at 40.005 127 0)
-      (effects (font (size 1.27 1.27)) hide)
-    )
-    (property "Datasheet" "~" (at 40.005 127 0)
-      (effects (font (size 1.27 1.27)) hide)
-    )
-    (pin "1")
-    (pin "2")
-    (pin "3")
-    (pin "4")
-    (instances
-      (project "GigaVesc"
-        (path "/768a484b-8a27-40cf-8cad-0f63935b1af0"
-          (reference "SW1") (unit 1)
-        )
-      )

Commit message: routinglogic
Parts:
- removed Y1: Crystal, Crystal:Crystal_SMD_HC49-SD, symbol Device:Crystal
- added C35: 100n, Capacitor_SMD:C_0805_2012Metric, symbol Device:C
- added C36, C37, C38, C39, C40, C41, C42, C43: 1n, Capacitor_SMD:C_0805_2012Metric, symbol Device:C
- added X1: S5D8.000000A20F30T, Crystal:Crystal_SMD_5032-4Pin_5.0x3.2mm, symbol Oscillator:SG-5032CCN
- C2: value 15p -> 1n; MPN C520056 -> C94121
- C3: value 15p -> 1n; MPN (none) -> C94121
- U1: value STM32F405RGT7 -> STM32F405RGT6; JLCRotOffset (none) -> -90; MPN C1337199 -> C15742
Connections:
- net +3.3V: now also C35.1, X1.1 (OE), X1.4 (Vcc)
- net CUR1: now also C39.1
- net CUR2: now also C38.1
- net CUR3: now also C37.1
- net GND: now also C3.2, C35.2, C36.2, C37.2, C38.2, C39.2, C40.2, C41.2, C42.2, C43.2, X1.2 (GND); no longer C3.1
- net IN_V: now also C43.1
- net MOSTEMP1: now also C40.1
- net MOSTEMP2: now also C41.1
- net MOSTEMP3: now also C42.1
- net VSENSE1: now also C2.1
- net VSENSE2: now also C36.1
- net VSENSE3: now also C3.1
- net at U1.5 (PH0): now also X1.3 (OUT); no longer C2.1
- net at U1.6 (PH1): no longer C3.2
- net EXT2_MOSI: now reaches U1.53 (PC12)
- net RX_EXT2 renamed EXT2_RX_MISO
- net TX_EXT2 renamed EXT2_TX_SCK

Commit message: routed_again
Parts:
- removed U2: REF1933AIDDCT, Package_TO_SOT_SMD:SOT-23-5, symbol GigaVescSymbols:REF1933AIDDCT
- removed X1: S5D8.000000A20F30T, Crystal:Crystal_SMD_5032-4Pin_5.0x3.2mm, symbol Oscillator:SG-5032CCN
- added C52: 20p, Capacitor_SMD:C_0603_1608Metric, symbol Device:C
- added J3: UpdiConn, Connector_PinHeader_2.54mm:PinHeader_1x03_P2.54mm_Vertical, symbol Connector_Generic:Conn_01x03
- added U14: LM4128AMF-3.3, Package_TO_SOT_SMD:SOT-23-5, symbol Reference_Voltage:LM4128
- added Y1: X50328MSB2GI, Crystal:Crystal_SMD_5032-2Pin_5.0x3.2mm, symbol Device:Crystal
- C1: MPN C282732 -> C28233
- C10: MPN C83170 -> C1710
- C2: MPN C94121 -> C46653
- C35: value 100n -> 20p; footprint Capacitor_SMD:C_0805_2012Metric -> Capacitor_SMD:C_0603_1608Metric; MPN C282732 -> C1648
- D1: MPN C434435 -> C2297
- D2: MPN C131244 -> C84256
- R1: MPN C2930231 -> C17414
- R2: MPN C114531 -> C26010
- SW1, SW3: footprint Button_Switch_SMD:SW_SPST_Omron_B3FS-100xP -> Button_Switch_SMD:SW_Tactile_SPST_NO_Straight_CK_PTS636Sx25SMTRLFS; MPN C271750 -> C329185
Connections:
- net +3.3V: now also C10.2, C11.2, C12.2, C13.2, C5.2, C6.2, C8.2, C9.2, U1.1 (VBAT), U1.19 (VDD), U1.32 (VDD), U1.48 (VDD), U1.64 (VDD); no longer C10.1, C11.1, C12.1, C13.1, C35.1, C5.1, C6.1, C8.1, C9.1
- net +5V: now also U14.3 (EN), U14.4 (VIN)
- net GND: now also C10.1, C11.1, C12.1, C13.1, C35.1, C5.1, C6.1, C8.1, C9.1, C52.2, J3.2 (Pin_2), U14.2 (GND); no longer C35.2
- net at U1.5 (PH0): now also C35.2, Y1.2
- net at U1.6 (PH1): now also C52.1, Y1.1
- net CUR1 renamed CURR1_FILTERED
- net CUR2 renamed CURR2_FILTERED
- net CUR3 renamed CURR3_FILTERED
- net VREF renamed +3.3VADC
- net +3.3VADC: now also U14.5 (VREF)
- new net HardwareProtection/UPDI: J3.1 (Pin_1)
- new net HardwareProtection/UPDI2: J3.3 (Pin_3)
- no-connect marks 1 -> 0
Other:
- added sheet DriverSocket (DriverSocket.kicad_sch)
- added sheet DriverSocket1 (DriverSocket.kicad_sch)
- added sheet DriverSocket2 (DriverSocket.kicad_sch)
- added sheet HardwareProtection (HardwareProtection.kicad_sch)
- moved on the sheet: C1, C14, C15, C2, C3, C35, C36, C37, C38, C39, C40, C41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

Commit message: pre-final
Parts:
- J3: JLCPosOffset (none) -> 2.54,0; JLCRotOffset (none) -> -90
Changed lines of the file:
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@@
+      (effects (font (size 1.27 1.27)) hide)
+    )
+    (property "JLCRotOffset" "-90" (at 71.12 147.32 90)
+      (effects (font (size 1.27 1.27)) hide)
+    )
+    (property "JLCPosOffset" "2.54,0" (at 71.12 147.32 90)
       (effects (font (size 1.27 1.27)) hide)
     )

Commit message: fixes, led R
Parts:
- R3, R4: value 220 -> 10k
Changed lines of the file:
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@@
       (effects (font (size 1.27 1.27)))
     )
-    (property "Value" "220" (at 53.34 182.88 90)
+    (property "Value" "10k" (at 53.34 182.88 90)
       (effects (font (size 1.27 1.27)))
     )
@@
       (effects (font (size 1.27 1.27)))
     )
-    (property "Value" "220" (at 53.34 173.99 90)
-      (effects (font (size 1.27 1.27)))
-    )
+    (property "Value" "10k" (at 53.34 173.99 90)
+      (effects (font (size 1.27 1.27)))
+    )

Commit message: nearfinish
Parts:
- U14: JLCRotOffset (none) -> -180
Changed lines of the file:
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@@
+      (effects (font (size 1.27 1.27)) hide)
+    )
+    (property "JLCRotOffset" "-180" (at 245.11 129.54 0)
       (effects (font (size 1.27 1.27)) hide)
     )
