File: DriverSocket.kicad_sch (KiCad schematic)
At the start: 9 parts, among them J1 Output, J1 OutputDown, J3 Input, U8 74LVC1G125GV,125

Commit message: pre-final
Parts:
- J1: JLCPosOffset (none) -> 3.81,0; JLCRotOffset (none) -> -90; MPN (none) -> C2718488
- J3: JLCPosOffset (none) -> 6.35,0; JLCRotOffset (none) -> -90; MPN (none) -> C40877
Changed lines of the file:
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@@
+      (effects (font (size 1.27 1.27)) hide)
+    )
+    (property "MPN" "C2718488" (at 50.8 114.3 0)
+      (effects (font (size 1.27 1.27)) hide)
+    )
+    (property "JLCRotOffset" "-90" (at 50.8 114.3 0)
+      (effects (font (size 1.27 1.27)) hide)
+    )
+    (property "JLCPosOffset" "3.81,0" (at 50.8 114.3 0)
       (effects (font (size 1.27 1.27)) hide)
     )
@@
       (effects (font (size 1.27 1.27)) hide)
     )
+    (property "MPN" "C40877" (at 40.64 66.04 0)
+      (effects (font (size 1.27 1.27)) hide)
+    )
+    (property "JLCRotOffset" "-90" (at 40.64 66.04 0)
+      (effects (font (size 1.27 1.27)) hide)
+    )
+    (property "JLCPosOffset" "6.35,0" (at 40.64 66.04 0)
+      (effects (font (size 1.27 1.27)) hide)
+    )

Commit message: renamed
Parts:
- removed D19: SS54, Diode_SMD:D_SMA, symbol Device:D_Schottky
Connections:
- net at D19.1 (K), R33.2, U8.2: now also R32.2
Other:
- note added: "Disabled by default until MCU pulls this down."
- moved on the sheet: D19, R32
Changed lines of the file:
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@@
   (junction (at 166.37 78.74) (diameter 0) (color 0 0 0 0)
   )
+  (wire (pts (xy 166.37 93.98) (xy 166.37 99.06))
+    (stroke (width 0) (type default))
+  )
   (wire (pts (xy 62.23 111.76) (xy 62.23 118.11))
     (stroke (width 0) (type default))
   )
-  (wire (pts (xy 205.74 104.14) (xy 205.74 78.74))
-    (stroke (width 0) (type default))
-  )
   (wire (pts (xy 50.8 58.42) (xy 45.72 58.42))
     (stroke (width 0) (type default))
   )
-  (wire (pts (xy 161.29 86.36) (xy 166.37 86.36))
+  (wire (pts (xy 161.29 78.74) (xy 166.37 78.74))
     (stroke (width 0) (type default))
   )
@@
     (stroke (width 0) (type default))
   )
-  (wire (pts (xy 133.35 78.74) (xy 139.7 78.74))
+  (wire (pts (xy 166.37 99.06) (xy 161.29 99.06))
     (stroke (width 0) (type default))
   )
@@
     (stroke (width 0) (type default))
   )
-  (wire (pts (xy 147.32 78.74) (xy 153.67 78.74))
-    (stroke (width 0) (type default))
-  )
   (wire (pts (xy 182.88 88.9) (xy 182.88 91.44))
     (stroke (width 0) (type default))
@@
     (stroke (width 0) (type default))
   )
-  (wire (pts (xy 203.2 104.14) (xy 205.74 104.14))
-    (stroke (width 0) (type default))
-  )
   (wire (pts (xy 55.88 119.38) (xy 55.88 116.84))
     (stroke (width 0) (type default))
@@
     (stroke (width 0) (type default))
   )
-  (wire (pts (xy 161.29 78.74) (xy 166.37 78.74))
-    (stroke (width 0) (type default))
-  )
   (wire (pts (xy 64.77 109.22) (xy 63.5 109.22))
     (stroke (width 0) (type default))
@@
     (stroke (width 0) (type default))
   )
-  (global_label "POWER_STAGE_DISABLE" (shape input) (at 133.35 78.74 180) (fields_autoplaced)
+  (text "Disabled by default until MCU pulls this down." (at 123.19 104.14 0)
+    (effects (font (size 1.27 1.27)) (justify left bottom))
+  )
+  (global_label "POWER_STAGE_LOCKOUT" (shape input) (at 205.74 78.74 0) (fields_autoplaced)
+    (effects (font (size 1.27 1.27)) (justify left))
+    (property "Intersheetrefs" "${INTERSHEET_REFS}" (at 230.6096 78.74 0)
+      (effects (font (size 1.27 1.27)) (justify left) hide)
+    )
+  )
+  (global_label "POWER_STAGE_DISABLE" (shape input) (at 161.29 99.06 180) (fields_autoplaced)
     (effects (font (size 1.27 1.27)) (justify right))
-    (property "Intersheetrefs" "${INTERSHEET_REFS}" (at 109.3876 78.74 0)
-      (effects (font (size 1.27 1.27)) (justify right) hide)
-    )
-  )
-  (global_label "POWER_STAGE_LOCKOUT" (shape input) (at 203.2 104.14 180) (fields_autoplaced)
-    (effects (font (size 1.27 1.27)) (justify right))
-    (property "Intersheetrefs" "${INTERSHEET_REFS}" (at 178.3304 104.14 0)
+    (property "Intersheetrefs" "${INTERSHEET_REFS}" (at 137.3276 99.06 0)
       (effects (font (size 1.27 1.27)) (justify right) hide)
     )
@@
     (effects (font (size 1.27 1.27)) (justify left))
   )
-  (hierarchical_label "EXT_DISABLE" (shape input) (at 153.67 86.36 180) (fields_autoplaced)
+  (hierarchical_label "EXT_DISABLE" (shape input) (at 153.67 78.74 180) (fields_autoplaced)
     (effects (font (size 1.27 1.27)) (justify right))
   )
@@
         (path "/768a484b-8a27-40cf-8cad-0f63935b1af0/693754e5-6fc9-4123-abfe-2e1335cfdb84"
           (reference "J25") (unit 1)
-        )
-      )
-    )
-  )
-  (symbol (lib_id "Device:D_Schottky") (at 157.48 78.74 180) (unit 1)
-    (in_bom yes) (on_board yes) (dnp no)
-    (property "Reference" "D19" (at 162.56 76.2 0)
-      (effects (font (size 1.27 1.27)))
-    )
-    (property "Value" "SS54" (at 151.13 81.28 0)
-      (effects (font (size 1.27 1.27)))
-    )
-    (property "Footprint" "Diode_SMD:D_SMA" (at 157.48 78.74 0)
-      (effects (font (size 1.27 1.27)) hide)
-    )
-    (property "Datasheet" "~" (at 157.48 78.74 0)
-      (effects (font (size 1.27 1.27)) hide)
-    )
-    (property "MPN" "C22452" (at 157.48 78.74 0)
-      (effects (font (size 1.27 1.27)) hide)
-    )
-    (pin "1")
-    (pin "2")
-    (instances
-      (project "GigaVescDrivers"
-        (path "/74b7e1db-46d0-4e07-8500-01cfc2fa8362"
-          (reference "D19") (unit 1)
-        )
-      )
-      (project "GigaVesc"
-        (path "/768a484b-8a27-40cf-8cad-0f63935b1af0/d3d3a06e-f81d-4927-9a88-9ed5502f322c"
-          (reference "D3") (unit 1)
-        )
-        (path "/768a484b-8a27-40cf-8cad-0f63935b1af0/04d6ed87-6b10-45aa-8255-84943212068b"
-          (reference "D4") (unit 1)
-        )
-        (path "/768a484b-8a27-40cf-8cad-0f63935b1af0/693754e5-6fc9-4123-abfe-2e1335cfdb84"
-          (reference "D5") (unit 1)
         )
       )
@@
     )
   )
-  (symbol (lib_id "Device:D_Schottky") (at 157.48 86.36 180) (unit 1)
+  (symbol (lib_id "Device:D_Schottky") (at 157.48 78.74 180) (unit 1)
     (in_bom yes) (on_board yes) (dnp no)
-    (property "Reference" "D19" (at 162.56 83.82 0)
-      (effects (font (size 1.27 1.27)))
-    )
-    (property "Value" "SS54" (at 151.13 88.9 0)
-      (effects (font (size 1.27 1.27)))
-    )
-    (property "Footprint" "Diode_SMD:D_SMA" (at 157.48 86.36 0)
-      (effects (font (size 1.27 1.27)) hide)
-    )
-    (property "Datasheet" "~" (at 157.48 86.36 0)
-      (effects (font (size 1.27 1.27)) hide)
-    )
-    (property "MPN" "C22452" (at 157.48 86.36 0)
+    (property "Reference" "D19" (at 162.56 76.2 0)
+      (effects (font (size 1.27 1.27)))
+    )
+    (property "Value" "SS54" (at 151.13 81.28 0)
+      (effects (font (size 1.27 1.27)))
+    )
+    (property "Footprint" "Diode_SMD:D_SMA" (at 157.48 78.74 0)
+      (effects (font (size 1.27 1.27)) hide)
+    )
+    (property "Datasheet" "~" (at 157.48 78.74 0)
+      (effects (font (size 1.27 1.27)) hide)
+    )
+    (property "MPN" "C22452" (at 157.48 78.74 0)
       (effects (font (size 1.27 1.27)) hide)
     )
@@
     )
   )
-  (symbol (lib_id "Device:R") (at 143.51 78.74 90) (unit 1)
-    (in_bom yes) (on_board yes) (dnp no) (fields_autoplaced)
-    (property "Reference" "R32" (at 143.51 72.39 90)
-      (effects (font (size 1.27 1.27)))
-    )
-    (property "Value" "2.2k" (at 143.51 74.93 90)
-      (effects (font (size 1.27 1.27)))
-    )
-    (property "Footprint" "Resistor_SMD:R_0805_2012Metric" (at 143.51 80.518 90)
-      (effects (font (size 1.27 1.27)) hide)
-    )
-    (property "Datasheet" "~" (at 143.51 78.74 0)
-      (effects (font (size 1.27 1.27)) hide)
-    )
-    (property "MPN" "C17520" (at 143.51 78.74 0)
-      (effects (font (size 1.27 1.27)) hide)
-    )
+  (symbol (lib_id "Device:R") (at 166.37 90.17 180) (unit 1)
+    (in_bom yes) (on_board yes) (dnp no) (fields_autoplaced)
+    (property "Reference" "R32" (at 168.91 88.9 0)
+      (effects (font (size 1.27 1.27)) (justify right))
+    )
+    (property "Value" "2.2k" (at 168.91 91.44 0)
+      (effects (font (size 1.27 1.27)) (justify right))
+    )
+    (property "Footprint" "Resistor_SMD:R_0805_2012Metric" (at 168.148 90.17 90)
+      (effects (font (size 1.27 1.27)) hide)
+    )
+    (property "Datasheet" "~" (at 166.37 90.17 0)
+      (effects (font (size 1.27 1.27)) hide)
+    )
+    (property "MPN" "C17520" (at 166.37 90.17 0)
+      (effects (font (size 1.27 1.27)) hide)
+    )

Commit message: fixes, led R
Parts:
- D19: value SS54 -> 1N5819WS; footprint Diode_SMD:D_SMA -> Diode_SMD:D_SOD-323; MPN C22452 -> C191023
Changed lines of the file:
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@@
       (effects (font (size 1.27 1.27)))
     )
-    (property "Value" "SS54" (at 151.13 81.28 0)
+    (property "Value" "1N5819WS" (at 151.13 81.28 0)
       (effects (font (size 1.27 1.27)))
     )
-    (property "Footprint" "Diode_SMD:D_SMA" (at 157.48 78.74 0)
+    (property "Footprint" "Diode_SMD:D_SOD-323" (at 157.48 78.74 0)
       (effects (font (size 1.27 1.27)) hide)
     )
@@
       (effects (font (size 1.27 1.27)) hide)
     )
-    (property "MPN" "C22452" (at 157.48 78.74 0)
+    (property "MPN" "C191023" (at 157.48 78.74 0)
       (effects (font (size 1.27 1.27)) hide)
     )

Commit message: nearfinish
Parts:
- removed D19: 1N5819WS, Diode_SMD:D_SOD-323, symbol Device:D_Schottky
Connections:
- net EXT_DISABLE: now also R32.2, R33.2, U8.2
Changed lines of the file:
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@@
     (stroke (width 0) (type default))
   )
-  (wire (pts (xy 161.29 78.74) (xy 166.37 78.74))
+  (wire (pts (xy 153.67 78.74) (xy 166.37 78.74))
     (stroke (width 0) (type default))
   )
@@
         )
       )
-    )
-  )
-  (symbol (lib_id "Device:D_Schottky") (at 157.48 78.74 180) (unit 1)
-    (in_bom yes) (on_board yes) (dnp no)
-    (property "Reference" "D19" (at 162.56 76.2 0)
-      (effects (font (size 1.27 1.27)))
-    )
-    (property "Value" "1N5819WS" (at 151.13 81.28 0)
-      (effects (font (size 1.27 1.27)))
-    )
-    (property "Footprint" "Diode_SMD:D_SOD-323" (at 157.48 78.74 0)
-      (effects (font (size 1.27 1.27)) hide)
-    )
-    (property "Datasheet" "~" (at 157.48 78.74 0)
-      (effects (font (size 1.27 1.27)) hide)
-    )
-    (property "MPN" "C191023" (at 157.48 78.74 0)
-      (effects (font (size 1.27 1.27)) hide)
-    )
-    (pin "1")
-    (pin "2")
-    (instances
-      (project "GigaVescDrivers"
-        (path "/74b7e1db-46d0-4e07-8500-01cfc2fa8362"
-          (reference "D19") (unit 1)
-        )
-      )
-      (project "GigaVesc"
-        (path "/768a484b-8a27-40cf-8cad-0f63935b1af0/d3d3a06e-f81d-4927-9a88-9ed5502f322c"
-          (reference "D6") (unit 1)
-        )
-        (path "/768a484b-8a27-40cf-8cad-0f63935b1af0/04d6ed87-6b10-45aa-8255-84943212068b"
-          (reference "D7") (unit 1)
-        )
-        (path "/768a484b-8a27-40cf-8cad-0f63935b1af0/693754e5-6fc9-4123-abfe-2e1335cfdb84"
-          (reference "D8") (unit 1)
-        )
-      )

Commit message: or-gate
Parts:
- removed C15: 100n, Capacitor_SMD:C_0805_2012Metric, symbol Device:C
- removed R32, R33: 2.2k, Resistor_SMD:R_0805_2012Metric, symbol Device:R
- removed U8: 74LVC1G125GV,125, Package_SO:TSOP-5_1.65x3.05mm_P0.95mm, symbol 74xGxx:74LVC1G125
Other:
- note removed: "Disabled by default until MCU pulls this down."
- moved on the sheet: J1, J3
