File: Switches.kicad_sch (KiCad schematic)
At the start: 13 parts, among them U8 RS2057XH, U9 SN74CBT3126PWR

Commit message: initial
Parts:
- C18: renamed from C32; footprint (none) -> Capacitor_SMD:C_0805_2012Metric
- C19: renamed from C31; footprint (none) -> Capacitor_SMD:C_0805_2012Metric
- C20: renamed from C33; footprint (none) -> Capacitor_SMD:C_0805_2012Metric
- C21: renamed from C30; footprint (none) -> Capacitor_SMD:C_0805_2012Metric
- C22: renamed from C29; footprint (none) -> Capacitor_SMD:C_0805_2012Metric
- R4: footprint (none) -> Resistor_SMD:R_0805_2012Metric
- U4: renamed from U9; footprint MODULE -> Package_SO:TSSOP-14_4.4x5mm_P0.65mm
- U5: renamed from U8; footprint MODULE -> Package_TO_SOT_SMD:SOT-23-6

Commit message: jlcpcb
Parts:
- C18: MPN (none) -> C565626
- R4: MPN (none) -> C139913
- U4: MPN (none) -> C7142
- U5: MPN (none) -> C255474
Changed lines of the file:
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@@
+      (effects (font (size 1.27 1.27)) hide)
+    )
+    (property "MPN" "C7142" (at 84.455 92.075 0)
       (effects (font (size 1.27 1.27)) hide)
     )
@@
       (effects (font (size 1.27 1.27)) hide)
     )
+    (property "MPN" "C565626" (at 46.99 108.585 0)
+      (effects (font (size 1.27 1.27)) hide)
+    )
     (pin "1")
     (pin "2")
@@
     )
     (property "Datasheet" "DOCUMENTATION" (at 208.28 85.09 0)
+      (effects (font (size 1.27 1.27)) hide)
+    )
+    (property "MPN" "C255474" (at 208.28 80.01 0)
       (effects (font (size 1.27 1.27)) hide)
     )
@@
       (effects (font (size 1.27 1.27)) hide)
     )
+    (property "MPN" "C139913" (at 221.615 102.87 0)
+      (effects (font (size 1.27 1.27)) hide)
+    )

Commit message: routinglogic
Parts:
- U4: JLCRotOffset (none) -> -90
Changed lines of the file:
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@@
+      (effects (font (size 1.27 1.27)) hide)
+    )
+    (property "JLCRotOffset" "-90" (at 84.455 92.075 0)
       (effects (font (size 1.27 1.27)) hide)
     )

Commit message: routed_again
Parts:
- R4: MPN C139913 -> C17520
Other:
- moved on the sheet: C18, C19, C20, C21, C22, R4, U4, U5

Commit message: nearfinish
Parts:
- U5: JLCRotOffset (none) -> -180
Changed lines of the file:
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@@
+      (effects (font (size 1.27 1.27)) hide)
+    )
+    (property "JLCRotOffset" "-180" (at 205.74 78.74 0)
       (effects (font (size 1.27 1.27)) hide)
     )

Commit message: or-gate
Parts:
- R4: MPN (none) -> C17520
Changed lines of the file:
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@@
+      (effects (font (size 1.27 1.27)) hide)
+    )
+    (property "MPN" "C17520" (at 203.2 106.68 90)
       (effects (font (size 1.27 1.27)) hide)
     )
