File: Drivers/CurrentMeasurement.kicad_sch (KiCad schematic)
At the start: 9 parts, among them U10 INA4181A1IPWR

Commit message: initial
Other:
- note added: "Reverse intended"
- note removed: "Are we sure its this way?"
Changed lines of the file:
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@@
     (stroke (width 0) (type default))
   )
-  (text "Are we sure its this way?" (at 73.66 73.66 0)
+  (text "Reverse intended" (at 80.645 73.025 0)
     (effects (font (size 1.27 1.27)) (justify left bottom))
   )

Commit message: initial
Parts:
- C20, C21, C22, C23, C24: footprint (none) -> Capacitor_SMD:C_0805_2012Metric
- R43, R44, R45: footprint (none) -> Resistor_SMD:R_0805_2012Metric
- U10: footprint SOP65P640X120-20N -> Package_SO:TSSOP-20_4.4x6.5mm_P0.65mm
Changed lines of the file:
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@@
       (effects (font (size 1.27 1.27)) (justify left))
     )
-    (property "Footprint" "" (at 80.9752 119.38 0)
+    (property "Footprint" "Capacitor_SMD:C_0805_2012Metric" (at 80.9752 119.38 0)
       (effects (font (size 1.27 1.27)) hide)
     )
@@
       (effects (font (size 1.27 1.27)))
     )
-    (property "Footprint" "" (at 167.64 100.838 90)
+    (property "Footprint" "Resistor_SMD:R_0805_2012Metric" (at 167.64 100.838 90)
       (effects (font (size 1.27 1.27)) hide)
     )
@@
       (effects (font (size 1.27 1.27)))
     )
-    (property "Footprint" "" (at 167.64 80.518 90)
+    (property "Footprint" "Resistor_SMD:R_0805_2012Metric" (at 167.64 80.518 90)
       (effects (font (size 1.27 1.27)) hide)
     )
@@
       (effects (font (size 1.27 1.27)) (justify left))
     )
-    (property "Footprint" "" (at 201.6252 111.76 0)
+    (property "Footprint" "Capacitor_SMD:C_0805_2012Metric" (at 201.6252 111.76 0)
       (effects (font (size 1.27 1.27)) hide)
     )
@@
       (effects (font (size 1.27 1.27)))
     )
-    (property "Footprint" "SOP65P640X120-20N" (at 118.11 96.52 0)
+    (property "Footprint" "Package_SO:TSSOP-20_4.4x6.5mm_P0.65mm" (at 118.11 96.52 0)
       (effects (font (size 1.27 1.27)) (justify bottom) hide)
     )
@@
       (effects (font (size 1.27 1.27)) (justify left))
     )
-    (property "Footprint" "" (at 145.7452 71.12 0)
+    (property "Footprint" "Capacitor_SMD:C_0805_2012Metric" (at 145.7452 71.12 0)
       (effects (font (size 1.27 1.27)) hide)
     )
@@
       (effects (font (size 1.27 1.27)) (justify left))
     )
-    (property "Footprint" "" (at 178.7652 111.76 0)
+    (property "Footprint" "Capacitor_SMD:C_0805_2012Metric" (at 178.7652 111.76 0)
       (effects (font (size 1.27 1.27)) hide)
     )
@@
       (effects (font (size 1.27 1.27)))
     )
-    (property "Footprint" "" (at 167.64 90.678 90)
+    (property "Footprint" "Resistor_SMD:R_0805_2012Metric" (at 167.64 90.678 90)
       (effects (font (size 1.27 1.27)) hide)
     )
@@
       (effects (font (size 1.27 1.27)) (justify left))
     )
-    (property "Footprint" "" (at 190.1952 111.76 0)
-      (effects (font (size 1.27 1.27)) hide)
-    )
+    (property "Footprint" "Capacitor_SMD:C_0805_2012Metric" (at 190.1952 111.76 0)
+      (effects (font (size 1.27 1.27)) hide)
+    )
