File: Drivers/HardwareProtection.kicad_sch (KiCad schematic)
At the start: 29 parts, among them U3 CD4043BPWR, U4 MCP6564-E_ST, U5 MCP6564-E_ST, U6 CD4043BPWR

Commit message: initial
Parts:
- C3, C4, C5, C6: footprint (none) -> Capacitor_SMD:C_0805_2012Metric
- D10, D11, D12, D5, D6, D7, D8, D9: footprint (none) -> LED_SMD:LED_0805_2012Metric
- R10, R11, R12, R13, R14, R15, R3, R4, R5, R6, R7, R8, R9: footprint (none) -> Resistor_SMD:R_0805_2012Metric
- U3, U6: footprint SOP65P640X120-16N -> Package_SO:TSSOP-16_4.4x5mm_P0.65mm
- U4, U5: footprint MODULE -> Package_SO:TSSOP-14_4.4x5mm_P0.65mm
Changed lines of the file:
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@@
       (effects (font (size 1.27 1.27)))
     )
-    (property "Footprint" "" (at 222.25 44.45 0)
+    (property "Footprint" "LED_SMD:LED_0805_2012Metric" (at 222.25 44.45 0)
       (effects (font (size 1.27 1.27)) hide)
     )
@@
       (effects (font (size 1.27 1.27)) (justify left))
     )
-    (property "Footprint" "" (at 24.892 182.88 90)
+    (property "Footprint" "Resistor_SMD:R_0805_2012Metric" (at 24.892 182.88 90)
       (effects (font (size 1.27 1.27)) hide)
     )
@@
       (effects (font (size 1.27 1.27)))
     )
-    (property "Footprint" "" (at 238.76 46.228 90)
+    (property "Footprint" "Resistor_SMD:R_0805_2012Metric" (at 238.76 46.228 90)
       (effects (font (size 1.27 1.27)) hide)
     )
@@
       (effects (font (size 1.27 1.27)))
     )
-    (property "Footprint" "" (at 238.76 56.388 90)
+    (property "Footprint" "Resistor_SMD:R_0805_2012Metric" (at 238.76 56.388 90)
       (effects (font (size 1.27 1.27)) hide)
     )
@@
       (effects (font (size 1.27 1.27)) (justify left))
     )
-    (property "Footprint" "" (at 63.1952 44.45 0)
+    (property "Footprint" "Capacitor_SMD:C_0805_2012Metric" (at 63.1952 44.45 0)
       (effects (font (size 1.27 1.27)) hide)
     )
@@
       (effects (font (size 1.27 1.27)))
     )
-    (property "Footprint" "MODULE" (at 100.33 135.89 0)
+    (property "Footprint" "Package_SO:TSSOP-14_4.4x5mm_P0.65mm" (at 100.33 135.89 0)
       (effects (font (size 1.27 1.27)) hide)
     )
@@
       (effects (font (size 1.27 1.27)))
     )
-    (property "Footprint" "SOP65P640X120-16N" (at 184.15 57.15 0)
+    (property "Footprint" "Package_SO:TSSOP-16_4.4x5mm_P0.65mm" (at 184.15 57.15 0)
       (effects (font (size 1.27 1.27)) (justify bottom) hide)
     )
@@
       (effects (font (size 1.27 1.27)))
     )
-    (property "Footprint" "" (at 222.25 118.11 0)
+    (property "Footprint" "LED_SMD:LED_0805_2012Metric" (at 222.25 118.11 0)
       (effects (font (size 1.27 1.27)) hide)
     )
@@
       (effects (font (size 1.27 1.27)))
     )
-    (property "Footprint" "" (at 222.25 123.19 0)
+    (property "Footprint" "LED_SMD:LED_0805_2012Metric" (at 222.25 123.19 0)
       (effects (font (size 1.27 1.27)) hide)
     )
@@
       (effects (font (size 1.27 1.27)) (justify left))
     )
-    (property "Footprint" "" (at 24.892 172.72 90)
+    (property "Footprint" "Resistor_SMD:R_0805_2012Metric" (at 24.892 172.72 90)
       (effects (font (size 1.27 1.27)) hide)
     )
@@
       (effects (font (size 1.27 1.27)))
     )
-    (property "Footprint" "" (at 222.25 49.53 0)
+    (property "Footprint" "LED_SMD:LED_0805_2012Metric" (at 222.25 49.53 0)
       (effects (font (size 1.27 1.27)) hide)
     )
@@
       (effects (font (size 1.27 1.27)))
     )
-    (property "Footprint" "" (at 238.76 51.308 90)
+    (property "Footprint" "Resistor_SMD:R_0805_2012Metric" (at 238.76 51.308 90)
       (effects (font (size 1.27 1.27)) hide)
     )
@@
       (effects (font (size 1.27 1.27)) (justify left))
     )
-    (property "Footprint" "" (at 37.592 90.17 90)
+    (property "Footprint" "Resistor_SMD:R_0805_2012Metric" (at 37.592 90.17 90)
       (effects (font (size 1.27 1.27)) hide)
     )
@@
       (effects (font (size 1.27 1.27)))
     )
-    (property "Footprint" "" (at 238.76 124.968 90)
+    (property "Footprint" "Resistor_SMD:R_0805_2012Metric" (at 238.76 124.968 90)
       (effects (font (size 1.27 1.27)) hide)
     )
@@
       (effects (font (size 1.27 1.27)))
     )
-    (property "Footprint" "MODULE" (at 100.33 62.23 0)
+    (property "Footprint" "Package_SO:TSSOP-14_4.4x5mm_P0.65mm" (at 100.33 62.23 0)
       (effects (font (size 1.27 1.27)) hide)
     )
@@
       (effects (font (size 1.27 1.27)))
     )
-    (property "Footprint" "" (at 238.76 119.888 90)
+    (property "Footprint" "Resistor_SMD:R_0805_2012Metric" (at 238.76 119.888 90)
       (effects (font (size 1.27 1.27)) hide)
     )
@@
       (effects (font (size 1.27 1.27)) (justify left))
     )
-    (property "Footprint" "" (at 50.4952 93.98 0)
+    (property "Footprint" "Capacitor_SMD:C_0805_2012Metric" (at 50.4952 93.98 0)
       (effects (font (size 1.27 1.27)) hide)
     )
@@
       (effects (font (size 1.27 1.27)) (justify left))
     )
-    (property "Footprint" "" (at 60.6552 93.98 0)
+    (property "Footprint" "Capacitor_SMD:C_0805_2012Metric" (at 60.6552 93.98 0)
       (effects (font (size 1.27 1.27)) hide)
     )
@@
       (effects (font (size 1.27 1.27)))
     )
-    (property "Footprint" "" (at 222.25 133.35 0)
+    (property "Footprint" "LED_SMD:LED_0805_2012Metric" (at 222.25 133.35 0)
       (effects (font (size 1.27 1.27)) hide)
     )
@@
       (effects (font (size 1.27 1.27)) (justify left))
     )
-    (property "Footprint" "" (at 63.1952 118.11 0)
+    (property "Footprint" "Capacitor_SMD:C_0805_2012Metric" (at 63.1952 118.11 0)
       (effects (font (size 1.27 1.27)) hide)
     )
@@
       (effects (font (size 1.27 1.27)))
     )
-    (property "Footprint" "" (at 222.25 54.61 0)
+    (property "Footprint" "LED_SMD:LED_0805_2012Metric" (at 222.25 54.61 0)
       (effects (font (size 1.27 1.27)) hide)
     )
@@
       (effects (font (size 1.27 1.27)))
     )
-    (property "Footprint" "" (at 222.25 59.69 0)
+    (property "Footprint" "LED_SMD:LED_0805_2012Metric" (at 222.25 59.69 0)
       (effects (font (size 1.27 1.27)) hide)
     )
@@
       (effects (font (size 1.27 1.27)) (justify left))
     )
-    (property "Footprint" "" (at 66.802 182.88 90)
+    (property "Footprint" "Resistor_SMD:R_0805_2012Metric" (at 66.802 182.88 90)
       (effects (font (size 1.27 1.27)) hide)
     )
@@
       (effects (font (size 1.27 1.27)))
     )
-    (property "Footprint" "SOP65P640X120-16N" (at 184.15 130.81 0)
+    (property "Footprint" "Package_SO:TSSOP-16_4.4x5mm_P0.65mm" (at 184.15 130.81 0)
       (effects (font (size 1.27 1.27)) (justify bottom) hide)
     )
@@
       (effects (font (size 1.27 1.27)))
     )
-    (property "Footprint" "" (at 238.76 130.048 90)
+    (property "Footprint" "Resistor_SMD:R_0805_2012Metric" (at 238.76 130.048 90)
       (effects (font (size 1.27 1.27)) hide)
     )
@@
       (effects (font (size 1.27 1.27)))
     )
-    (property "Footprint" "" (at 238.76 135.128 90)
+    (property "Footprint" "Resistor_SMD:R_0805_2012Metric" (at 238.76 135.128 90)
       (effects (font (size 1.27 1.27)) hide)
     )
@@
       (effects (font (size 1.27 1.27)))
     )
-    (property "Footprint" "" (at 222.25 128.27 0)
+    (property "Footprint" "LED_SMD:LED_0805_2012Metric" (at 222.25 128.27 0)
       (effects (font (size 1.27 1.27)) hide)
     )
@@
       (effects (font (size 1.27 1.27)) (justify left))
     )
-    (property "Footprint" "" (at 66.802 172.72 90)
+    (property "Footprint" "Resistor_SMD:R_0805_2012Metric" (at 66.802 172.72 90)
       (effects (font (size 1.27 1.27)) hide)
     )
@@
       (effects (font (size 1.27 1.27)))
     )
-    (property "Footprint" "" (at 238.76 61.468 90)
-      (effects (font (size 1.27 1.27)) hide)
-    )
+    (property "Footprint" "Resistor_SMD:R_0805_2012Metric" (at 238.76 61.468 90)
+      (effects (font (size 1.27 1.27)) hide)
+    )
