File: Drivers/GigaVescDrivers.kicad_sch (KiCad schematic)
At the start: 15 parts, among them J1 LogicConn, U8 74LVC1G125GV,125

Commit message: initial
Connections:
- net CURR_TRIP_HIGH: now also J1.13 (Pin_13)
- net CURR_TRIP_LOW: now also J1.12 (Pin_12)
- net TEMP1: now also J1.16 (Pin_16)
- net TEMP2: now also J1.15 (Pin_15)
- net TEMP3: now also J1.14 (Pin_14)
Other:
- moved on the sheet: J1

Commit message: initial
Parts:
- added J2: LogicConn2, Connector_PinSocket_2.54mm:PinSocket_2x06_P2.54mm_Vertical, symbol Connector_Generic:Conn_02x06_Counter_Clockwise
- added J3: HVConn, Connector_PinHeader_2.54mm:PinHeader_2x04_P2.54mm_Vertical, symbol Connector_Generic:Conn_02x04_Counter_Clockwise
- added J4: HV1Conn, Connector_PinHeader_2.54mm:PinHeader_2x04_P2.54mm_Vertical, symbol Connector_Generic:Conn_02x04_Counter_Clockwise
- added J5: HV2Conn, Connector_PinHeader_2.54mm:PinHeader_2x04_P2.54mm_Vertical, symbol Connector_Generic:Conn_02x04_Counter_Clockwise
- added J6: HV3Conn, Connector_PinHeader_2.54mm:PinHeader_2x04_P2.54mm_Vertical, symbol Connector_Generic:Conn_02x04_Counter_Clockwise
- C15: footprint (none) -> Capacitor_SMD:C_0805_2012Metric
- D19, D20, D21, D22, D23, D24, D25, D26: footprint (none) -> Diode_SMD:D_0402_1005Metric
- D30: footprint (none) -> LED_SMD:LED_0805_2012Metric
- J1: footprint (none) -> Connector_PinSocket_2.54mm:PinSocket_2x10_P2.54mm_Vertical
- R32, R33, R42: footprint (none) -> Resistor_SMD:R_0805_2012Metric
- U8: footprint (none) -> Package_SO:TSOP-5_1.65x3.05mm_P0.95mm
Connections:
- net +3.3V: now also J2.12 (Pin_12)
- net CSR_N1: now also J3.2 (Pin_2)
- net CSR_N2: now also J3.4 (Pin_4)
- net CSR_N3: now also J3.7 (Pin_7)
- net CSR_P1: now also J3.1 (Pin_1), J4.3 (Pin_3), J4.4 (Pin_4)
- net CSR_P2: now also J3.3 (Pin_3), J5.3 (Pin_3), J5.4 (Pin_4)
- net CSR_P3: now also J3.8 (Pin_8), J6.3 (Pin_3), J6.4 (Pin_4)
- net GND: now also J2.7 (Pin_7), J2.8 (Pin_8), J3.5 (Pin_5), J3.6 (Pin_6)
- net PH1: now also J4.7 (Pin_7), J4.8 (Pin_8)
- net PH2: now also J5.7 (Pin_7), J5.8 (Pin_8)
- net PH3: now also J6.7 (Pin_7), J6.8 (Pin_8)
- net PHASE1: now also J4.5 (Pin_5), J4.6 (Pin_6)
- net PHASE2: now also J5.5 (Pin_5), J5.6 (Pin_6)
- net PHASE3: now also J6.5 (Pin_5), J6.6 (Pin_6)
- net PL1: now also J4.1 (Pin_1), J4.2 (Pin_2)
- net PL2: now also J5.1 (Pin_1), J5.2 (Pin_2)
- net PL3: now also J6.1 (Pin_1), J6.2 (Pin_2)
- net VBIAS: now also J2.3 (Pin_3)
- net DRIVE_DISABLE renamed POWER_STAGE_DISABLE
- net POWER_STAGE_DISABLE: now also J2.11 (Pin_11)
- net LOCKOUT renamed POWER_STAGE_LOCKOUT
- net POWER_STAGE_LOCKOUT: now also J2.10 (Pin_10)
- new net +5V: J2.1 (Pin_1)
- new net AUX_ENABLE: J2.6 (Pin_6)
- new net AUX_FAULT: J2.4 (Pin_4)
- new net CLEAR_HW_FAULT: J2.9 (Pin_9)
- new net IN_V: J2.2 (Pin_2)
- new net SENS_FILTER_ENABLE: J2.5 (Pin_5)
Other:
- note added: "Aux Passthru 12v circuit on mos board"

Commit message: routinglogic
Parts:
- added R46: 0, Resistor_SMD:R_0805_2012Metric, symbol Device:R
Connections:
- net GND: now also R46.1
- net POWER_STAGE_LOCKOUT: now also R46.2
Other:
- note added: "Optional bypass"
Changed lines of the file:
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@@
   (junction (at 185.42 64.77) (diameter 0) (color 0 0 0 0)
   )
+  (junction (at 185.42 79.375) (diameter 0) (color 0 0 0 0)
+  )
   (junction (at 52.07 173.355) (diameter 0) (color 0 0 0 0)
   )
@@
     (stroke (width 0) (type default))
   )
+  (wire (pts (xy 175.26 81.915) (xy 175.26 79.375))
+    (stroke (width 0) (type default))
+  )
   (wire (pts (xy 73.66 71.12) (xy 77.47 71.12))
     (stroke (width 0) (type default))
@@
     (stroke (width 0) (type default))
   )
+  (wire (pts (xy 175.26 79.375) (xy 177.8 79.375))
+    (stroke (width 0) (type default))
+  )
   (wire (pts (xy 147.32 95.25) (xy 147.32 104.775))
     (stroke (width 0) (type default))
@@
     (stroke (width 0) (type default))
   )
-  (wire (pts (xy 185.42 101.6) (xy 185.42 64.77))
+  (wire (pts (xy 185.42 101.6) (xy 185.42 79.375))
     (stroke (width 0) (type default))
   )
@@
     (stroke (width 0) (type default))
   )
-  (wire (pts (xy 185.42 112.395) (xy 185.42 101.6))
+  (wire (pts (xy 185.42 101.6) (xy 185.42 112.395))
     (stroke (width 0) (type default))
   )
@@
   )
   (wire (pts (xy 185.42 64.77) (xy 185.42 46.99))
+    (stroke (width 0) (type default))
+  )
+  (wire (pts (xy 185.42 79.375) (xy 185.42 64.77))
     (stroke (width 0) (type default))
   )
@@
     (effects (font (size 1.27 1.27)) (justify left bottom))
   )
-  (text "PB12" (at 171.45 135.89 0)
+  (text "PB12" (at 169.545 109.855 0)
+    (effects (font (size 1.27 1.27)) (justify left bottom))
+  )
+  (text "Optional bypass" (at 167.64 71.12 0)
     (effects (font (size 1.27 1.27)) (justify left bottom))
   )
@@
     )
   )
+  (symbol (lib_id "power:GND") (at 175.26 81.915 0) (unit 1)
+    (in_bom yes) (on_board yes) (dnp no) (fields_autoplaced)
+    (property "Reference" "#PWR066" (at 175.26 88.265 0)
+      (effects (font (size 1.27 1.27)) hide)
+    )
+    (property "Value" "GND" (at 175.26 86.995 0)
+      (effects (font (size 1.27 1.27)))
+    )
+    (property "Footprint" "" (at 175.26 81.915 0)
+      (effects (font (size 1.27 1.27)) hide)
+    )
+    (property "Datasheet" "" (at 175.26 81.915 0)
+      (effects (font (size 1.27 1.27)) hide)
+    )
+    (pin "1")
+    (instances
+      (project "GigaVescDrivers"
+        (path "/74b7e1db-46d0-4e07-8500-01cfc2fa8362"
+          (reference "#PWR066") (unit 1)
+        )
+      )
+    )
+  )
   (symbol (lib_id "Connector_Generic:Conn_02x04_Counter_Clockwise") (at 264.795 132.08 0) (unit 1)
     (in_bom yes) (on_board yes) (dnp no) (fields_autoplaced)
@@
         )
       )
+    )
+  )
+  (symbol (lib_id "Device:R") (at 181.61 79.375 90) (unit 1)
+    (in_bom yes) (on_board yes) (dnp no) (fields_autoplaced)
+    (property "Reference" "R46" (at 181.61 73.66 90)
+      (effects (font (size 1.27 1.27)))
+    )
+    (property "Value" "0" (at 181.61 76.2 90)
+      (effects (font (size 1.27 1.27)))
+    )
+    (property "Footprint" "Resistor_SMD:R_0805_2012Metric" (at 181.61 81.153 90)
+      (effects (font (size 1.27 1.27)) hide)
+    )
+    (property "Datasheet" "~" (at 181.61 79.375 0)
+      (effects (font (size 1.27 1.27)) hide)
+    )
+    (pin "1")
+    (pin "2")
+    (instances
+      (project "GigaVescDrivers"
+        (path "/74b7e1db-46d0-4e07-8500-01cfc2fa8362"
+          (reference "R46") (unit 1)
+        )
+      )

Commit message: driversconnectors
Parts:
- removed J1: LogicConn, Connector_PinSocket_2.54mm:PinSocket_2x10_P2.54mm_Vertical, symbol Connector_Generic:Conn_02x10_Counter_Clockwise
- removed J2: LogicConn2, Connector_PinSocket_2.54mm:PinSocket_2x06_P2.54mm_Vertical, symbol Connector_Generic:Conn_02x06_Counter_Clockwise
Other:
- added sheet DriversConnectors (DriversConnectors.kicad_sch)
- note removed: "Aux Passthru 12v circuit on mos board"
- note removed: "Passthru"
- note removed: "Passthru to phase sensor pull down res close to IC"
