File: MosfetBoard/PhaseMosfets.kicad_sch (KiCad schematic)
At the start: 20 parts, among them Q1 IXTT220N20X4HV, Q2 IXTT220N20X4HV, Q4 IXTT220N20X4HV, Q5 IXTT220N20X4HV, U1 RS2166XC5, U3 ACS773ECB-200B-PFF-T

Commit message: up
Parts:
- U3: footprint Sensor_Current:Allegro_CB_PSF -> GigaVescLibs:Allegro_CB_SMD
Changed lines of the file:
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@@
       (effects (font (size 1.27 1.27)))
     )
-    (property "Footprint" "Sensor_Current:Allegro_CB_PSF" (at 173.99 85.09 0)
+    (property "Footprint" "GigaVescLibs:Allegro_CB_SMD" (at 173.99 85.09 0)
       (effects (font (size 1.27 1.27)) hide)
     )
