File: MosfetBoard/MosfetBoard.kicad_pcb (KiCad board)
At the start: 2 copper layers, 200 x 100 mm, 107 parts, among them J1 DRIVER1, J10 A_PAD, J11 B_PAD, J12 C_PAD, J13 BATT+Conn2, J14 BATT-Conn2, J2 DRIVER2, J3 DRIVER3, J4 PhaseConn1, J5 PhaseConn2, J6 PhaseConn3, J7 VINConn, J8 BATT+Conn1, J9 BATT-Conn1, Q1 IXTT220N20X4HV, Q10 IXTT220N20X4HV, Q11 IXTT220N20X4HV, Q12 IXTT220N20X4HV, Q2 IXTT220N20X4HV, Q3 IXTT220N20X4HV, Q4 IXTT220N20X4HV, Q5 IXTT220N20X4HV, Q6 IXTT220N20X4HV, Q7 IXTT220N20X4HV, Q8 IXTT220N20X4HV, Q9 IXTT220N20X4HV, U1 RS2166XC5, U2 ACS773ECB-200B-PFF-T, U3 ACS773ECB-200B-PFF-T, U4 RDE20110S12, U5 RS2166XC5, U6 ACS773ECB-200B-PFF-T, U7 RS2166XC5

Commit message: up
Parts:
- removed C32, C33: C_Polarized, Capacitor_THT:C_Radial_D18.0mm_H35.5mm_P7.50mm
- added J15: AuxConn, Connector_PinSocket_2.54mm:PinSocket_1x05_P2.54mm_Vertical_SMD_Pin1Left, F.Cu at (301.9, 105.5)
- added REF**: LogicBoard, GigaVescLibs:LogicBoard, F.Cu at (156.0, 75.0)
- C25, C26, C27, C28, C30, C31: value C_Polarized -> 680uF 200V; footprint Capacitor_THT:C_Radial_D18.0mm_H35.5mm_P7.50mm -> Capacitor_THT:CP_Radial_D22.0mm_P10.00mm_SnapIn
- C29, C34, C35, C36, C37, C38, C39, C40, C41, C42, C43, C44, C45, C46, C47, J10, J11, J12, L1, L2, L3, Q1, Q10, Q11, Q12, Q2, Q3, Q4, Q5, Q6, Q7, Q8, Q9, R1, R10, R11, R12, R13, R14, R15, R16, R17, R18, R19, R2, R20, R21, R3, R4, R5, R6, R7, R8, R9, TH1, TH2, TH3, U1, U5, U7: moved to F.Cu
- J1, J2, J3: footprint Connector_PinSocket_2.54mm:PinSocket_1x04_P2.54mm_Vertical -> Connector_PinSocket_2.54mm:PinSocket_2x02_P2.54mm_Vertical_SMD
- J4, J5, J6: footprint Connector_PinSocket_2.54mm:PinSocket_2x03_P2.54mm_Vertical -> Connector_PinSocket_2.54mm:PinSocket_2x03_P2.54mm_Vertical_SMD
- J7: footprint Connector_PinSocket_2.54mm:PinSocket_1x04_P2.54mm_Vertical -> Connector_PinSocket_2.54mm:PinSocket_1x04_P2.54mm_Vertical_SMD_Pin1Left
- U2, U3, U6: footprint Sensor_Current:Allegro_CB_PSF -> GigaVescLibs:Allegro_CB_SMD; moved to F.Cu
- moved U4 189.3 mm to (51.8, 110.2)
- moved J8 171.2 mm to (57.0, 31.5)
- moved C28 165.9 mm to (225.0, 49.5), turned to 0 degrees
- moved R18 149.7 mm to (69.5, 56.0), turned to -90 degrees
- moved J13 142.4 mm to (225.0, 31.5)
- moved Q11 138.1 mm to (72.0, 47.0)
- moved R19 128.6 mm to (96.6, 73.5), turned to 0 degrees
- moved Q12 127.6 mm to (87.5, 71.0)
- moved J12 124.0 mm to (84.0, 117.5), turned to 90 degrees
- moved R10 114.3 mm to (197.6, 91.0), turned to 0 degrees
- moved R16 113.2 mm to (87.0, 56.0), turned to -90 degrees
- moved U3 112.7 mm to (198.5, 106.0)
- moved Q10 108.3 mm to (87.5, 88.5), turned to 180 degrees
- moved Q9 102.6 mm to (89.5, 47.0)
- moved R20 100.5 mm to (92.5, 117.0), turned to 0 degrees
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Connections:
- J1 pad 2: PHASE1 -> PL1
- J1 pad 3: -BATT -> PHASE1
- J1 pad 4: PL1 -> -BATT
- J2 pad 2: PHASE2 -> PL2
- J2 pad 3: -BATT -> PHASE2
- J2 pad 4: PL2 -> -BATT
- J3 pad 2: PHASE3 -> PL3
- J3 pad 3: -BATT -> PHASE3
- J3 pad 4: PL3 -> -BATT
- J4 pad 3: SENS_FILTER_ENABLE -> SENS_FILTER_ENABLE1
- J5 pad 3: SENS_FILTER_ENABLE -> SENS_FILTER_ENABLE2
- J6 pad 3: SENS_FILTER_ENABLE -> SENS_FILTER_ENABLE3
- U1 pad 4: SENS_FILTER_ENABLE -> SENS_FILTER_ENABLE1
- U5 pad 4: SENS_FILTER_ENABLE -> SENS_FILTER_ENABLE2
- U7 pad 4: SENS_FILTER_ENABLE -> SENS_FILTER_ENABLE3
Routing:
- net +3.3V: track 0.00 -> 71.1 mm
- net PL3: track 0.00 -> 46.6 mm
- net PH3: track 0.00 -> 45.5 mm
- net PL1: track 0.00 -> 41.3 mm
- net PL2: track 0.00 -> 40.9 mm
- net PH1: track 0.00 -> 39.2 mm
- net Net-(U6-VCC): track 0.00 -> 32.9 mm
- net MOSTEMP2: track 0.00 -> 28.0 mm
- net PHASE3: track 0.00 -> 16.8 mm
- net CURR2: track 0.00 -> 14.4 mm
- net PHASE2: track 0.00 -> 14.0 mm
- net PHASE1: track 0.00 -> 11.0 mm
- net VSENSE2: track 0.00 -> 8.15 mm
- net Net-(U2-VCC): track 0.00 -> 4.62 mm
- net Net-(Q9-G): track 0.00 -> 2.98 mm
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- added copper zone on F.Cu, net A
- added copper zone on F.Cu, net B
- added copper zone on F.Cu, net C
- added copper zone on F.Cu, net PHASE1
- added copper zone on F.Cu, net PHASE2
- added copper zone on F.Cu, net PHASE3
- removed copper zone on B.Cu, net +BATT
- removed copper zone on B.Cu, net A
- removed copper zone on B.Cu, net PHASE1

Commit message: new_format
Parts:
- added Q13: NTMTSC4D3N15MC, Package_TO_SOT_SMD:PQFN_8x8, F.Cu at (127.5, 131.8)
- moved C31 327.7 mm to (-102.7, 88.0)
- moved C28 327.4 mm to (-102.3, 42.5)
- moved C30 327.2 mm to (-102.2, 65.0)
- moved C27 161.1 mm to (-103.2, 112.0), turned to 0 degrees
- moved U4 155.1 mm to (-98.0, 150.5)
- moved C25 127.7 mm to (-70.7, 53.0)
- moved C26 127.7 mm to (-70.7, 75.5)
- moved J13 12.0 mm to (213.0, 31.0)
- moved J8 9.51 mm to (66.5, 31.0)
- moved REF** 6.50 mm to (156.0, 81.5)
Routing:
- net -BATT: vias 92 -> 52
Other:
- board size 200 x 100 mm -> 155 x 100 mm
