File: MosfetBoard/NTMTSC4D3N15MC/NTMTSC4D3N15MC.kicad_sch (KiCad schematic)
At the start: 47 parts, among them J1 DRIVER1, J10 A_PAD, J10 AuxConn, J11 B_PAD, J12 C_PAD, J13 BATT+Conn2, J14 BATT-Conn2, J2 DRIVER2, J3 DRIVER3, J4 PhaseConn1, J5 PhaseConn2, J6 PhaseConn3, J7 VINConn, J8 BATT+Conn1, J9 BATT-Conn1, Q13 NTMTSC4D3N15MC, U4 RDE20110S12

Commit message: cheap-mosfet-board
Parts:
- removed C1, C10, C11, C12, C13, C14, C15, C16, C17, C18, C19, C2, C20, C21, C22, C23, C24, C3, C4, C5, C6, C7, C8, C9: C, Capacitor_SMD:C_2220_5650Metric, symbol Device:C
- removed C25, C26, C27, C28, C30, C31: 680uF 200V, Capacitor_THT:CP_Radial_D22.0mm_P10.00mm_SnapIn, symbol Device:C_Polarized
- removed J10: A_PAD, Connector_Wire:SolderWirePad_1x01_SMD_5x10mm, symbol Connector:Conn_01x01_Pin
- removed J10: AuxConn, Connector_PinSocket_2.54mm:PinSocket_1x05_P2.54mm_Vertical_SMD_Pin1Left, symbol Connector_Generic:Conn_01x05
- removed J11: B_PAD, Connector_Wire:SolderWirePad_1x01_SMD_5x10mm, symbol Connector:Conn_01x01_Pin
- removed J12: C_PAD, Connector_Wire:SolderWirePad_1x01_SMD_5x10mm, symbol Connector:Conn_01x01_Pin
- removed J7: VINConn, Connector_PinSocket_2.54mm:PinSocket_1x04_P2.54mm_Vertical_SMD_Pin1Left, symbol Connector_Generic:Conn_01x04
- removed Q13: NTMTSC4D3N15MC, Package_TO_SOT_SMD:PQFN_8x8, symbol Transistor_FET:FDMT800152DC
- removed U4: RDE20110S12, Converter_DCDC:Converter_DCDC_TRACO_THN30-xxxx_THT, symbol GigaESCSymbols:RDE20110S12
- J1, J2, J3: MPN (none) -> C3975147
- J4, J5, J6: MPN (none) -> C5160818
Connections:
- removed net +3.3V: J4.5 (Pin_5), J5.5 (Pin_5), J6.5 (Pin_5)
- new net 3.3V_1: J4.5 (Pin_5)
- new net 3.3V_2: J5.5 (Pin_5)
- new net 3.3V_3: J6.5 (Pin_5)
Other:
- sheet PhaseMosfets ports: added 3.3V_IN; removed none
- sheet PhaseMosfets1 ports: added 3.3V_IN; removed none
- sheet PhaseMosfets2 ports: added 3.3V_IN; removed none
- note removed: "Divider on mosfet board"
- note removed: "Total Capacity 4080uF"
