File: MosfetBoard/NTMTSC4D3N15MC/PhaseMosfets.kicad_sch (KiCad schematic)
At the start: 20 parts, among them Q1 NTMTSC4D3N15MC, Q2 NTMTSC4D3N15MC, Q4 NTMTSC4D3N15MC, Q5 NTMTSC4D3N15MC, U1 RS2166XC5, U3 ACS773ECB-200B-PFF-T

Commit message: cheap-mosfet-board
Parts:
- added C1 (x8): 10u 100V, Capacitor_SMD:C_1210_3225Metric, symbol Device:C
- added J12: PHASE_PAD, Connector_Wire:SolderWirePad_1x01_SMD_5x10mm, symbol Connector:Conn_01x01_Pin
Connections:
- net +BATT: now also C1.1, C1.1, C1.1, C1.1
- net -BATT: now also C1.2, C1.2, C1.2, C1.2
- net PHASE: now also U3.5 (IP-); no longer U3.4 (IP+)
- net PHASE_OUT: now also U3.4 (IP+), J12.1 (Pin_1); no longer U3.5 (IP-)
- net +3.3V renamed 3.3V_IN
- new net: C1.1, C1.2 (x4)
Other:
- moved on the sheet: C29, C34, L1, U3
