File: GigaESC/logicconnectors.kicad_sch (KiCad schematic)
At the start: 32 parts, among them J1 ServoConn, J1 USBC Socket, J10 AuxConn, J10 PhaseConn1, J13 VINConn, J18 PhaseConn1, J19 PhaseConn1, J4 ADCConn, J5 HallConn, J6 UartSpi, J7 JTAG, J8 CANConn, U2 USBLC6-2P6, U6 TJA1051T-3

Commit message: up
Connections:
- net at R21.1, U6.6 (CANL): now also J8.2 (Pin_2); no longer J8.3 (Pin_3)
- net at R21.2, U6.7 (CANH): now also J8.3 (Pin_3); no longer J8.2 (Pin_2)
Changed lines of the file:
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@@
   (junction (at 120.65 144.78) (diameter 0) (color 0 0 0 0)
   )
+  (junction (at 144.78 166.37) (diameter 0) (color 0 0 0 0)
+  )
   (junction (at 134.62 167.64) (diameter 0) (color 0 0 0 0)
   )
   (junction (at 50.8 78.74) (diameter 0) (color 0 0 0 0)
-  )
-  (junction (at 144.78 163.83) (diameter 0) (color 0 0 0 0)
   )
   (junction (at 214.63 77.47) (diameter 0) (color 0 0 0 0)
@@
     (stroke (width 0) (type default))
   )
-  (wire (pts (xy 142.24 166.37) (xy 152.4 166.37))
-    (stroke (width 0) (type default))
-  )
   (wire (pts (xy 240.03 40.64) (xy 240.03 50.8))
     (stroke (width 0) (type default))
@@
     (stroke (width 0) (type default))
   )
-  (wire (pts (xy 144.78 182.88) (xy 144.78 163.83))
+  (wire (pts (xy 144.78 182.88) (xy 144.78 166.37))
     (stroke (width 0) (type default))
   )
@@
     (stroke (width 0) (type default))
   )
-  (wire (pts (xy 142.24 163.83) (xy 144.78 163.83))
-    (stroke (width 0) (type default))
-  )
   (wire (pts (xy 134.62 167.64) (xy 134.62 172.72))
     (stroke (width 0) (type default))
@@
     (stroke (width 0) (type default))
   )
+  (wire (pts (xy 142.24 163.83) (xy 152.4 163.83))
+    (stroke (width 0) (type default))
+  )
   (wire (pts (xy 152.4 161.29) (xy 148.59 161.29))
     (stroke (width 0) (type default))
@@
     (stroke (width 0) (type default))
   )
+  (wire (pts (xy 144.78 166.37) (xy 144.78 162.56))
+    (stroke (width 0) (type default))
+  )
   (wire (pts (xy 104.14 162.56) (xy 107.95 162.56))
     (stroke (width 0) (type default))
@@
     (stroke (width 0) (type default))
   )
-  (wire (pts (xy 133.35 162.56) (xy 142.24 162.56))
+  (wire (pts (xy 133.35 162.56) (xy 144.78 162.56))
     (stroke (width 0) (type default))
   )
@@
     (stroke (width 0) (type default))
   )
-  (wire (pts (xy 142.24 162.56) (xy 142.24 163.83))
-    (stroke (width 0) (type default))
-  )
   (wire (pts (xy 26.67 36.83) (xy 29.21 36.83))
     (stroke (width 0) (type default))
@@
     (stroke (width 0) (type default))
   )
-  (wire (pts (xy 142.24 167.64) (xy 142.24 166.37))
+  (wire (pts (xy 142.24 163.83) (xy 142.24 167.64))
     (stroke (width 0) (type default))
   )
@@
     (stroke (width 0) (type default))
   )
+  (wire (pts (xy 144.78 166.37) (xy 152.4 166.37))
+    (stroke (width 0) (type default))
+  )
   (wire (pts (xy 245.11 52.07) (xy 236.22 52.07))
     (stroke (width 0) (type default))
@@
     (stroke (width 0) (type default))
   )
-  (wire (pts (xy 144.78 163.83) (xy 152.4 163.83))
-    (stroke (width 0) (type default))
-  )

Commit message: new_format
Parts:
- removed J10: AuxConn, Connector_PinHeader_2.54mm:PinHeader_1x05_P2.54mm_Vertical, symbol Connector_Generic:Conn_01x05
- removed J13: VINConn, Connector_PinHeader_2.54mm:PinHeader_1x04_P2.54mm_Vertical, symbol Connector_Generic:Conn_01x04
- removed J7: JTAG, Connector_PinHeader_2.54mm:PinHeader_1x05_P2.54mm_Vertical, symbol Connector:Conn_01x05_Pin
- added J2: AuxConn, Connector_JST:JST_XH_S8B-XH-A_1x08_P2.50mm_Horizontal, symbol Connector:Conn_01x08_Pin
- added J7: JTAG, Connector_PinHeader_2.54mm:PinHeader_2x02_P2.54mm_Vertical_SMD, symbol Connector_Generic:Conn_02x02_Counter_Clockwise
- added U10: HM-10, GigaVescLibs:HM10, symbol GigaVescSymbols:HM-10
- J1: footprint Connector_JST:JST_EH_S4B-EH_1x04_P2.50mm_Horizontal -> Connector_JST:JST_XH_S4B-XH-A_1x04_P2.50mm_Horizontal; MPN C265068 -> C157925
- J4, J5: footprint Connector_JST:JST_EH_S6B-EH_1x06_P2.50mm_Horizontal -> Connector_JST:JST_XH_S6B-XH-A_1x06_P2.50mm_Horizontal; MPN C495208 -> C157919
- J6: footprint Connector_JST:JST_EH_S5B-EH_1x05_P2.50mm_Horizontal -> Connector_JST:JST_XH_S5B-XH-A_1x05_P2.50mm_Horizontal; MPN C265103 -> C263757
- J8: footprint Connector_JST:JST_EH_S4B-EH_1x04_P2.50mm_Horizontal -> Connector_JST:JST_XH_S4B-XH-A_1x04_P2.50mm_Horizontal
Connections:
- net +15V: now also J2.1 (Pin_1), J2.2 (Pin_2)
- net +3.3V: now also U10.12 (VCC)
- net +5V: now also J5.6 (Pin_6); no longer J5.1 (Pin_1)
- net AUX_ENABLE: now also J2.6 (Pin_6)
- net AUX_FAULT: now also J2.7 (Pin_7)
- net CLEAR_HW_FAULT: now also J2.8 (Pin_8)
- net EXT2_RX_MISO: now also U10.1 (UART_TX)
- net EXT2_TX_SCK: now also U10.2 (UART_RX)
- net GND: now also J5.1 (Pin_1), J2.3 (Pin_3), J2.4 (Pin_4), J7.2 (Pin_2), U10.13 (GND), U10.14 (GND), U10.21 (GND); no longer J5.6 (Pin_6)
- net IN_V: now also J2.5 (Pin_5)
- net NRST: now also J7.1 (Pin_1)
- net SWCLK: now also J7.3 (Pin_3)
- net SWDIO: now also J7.4 (Pin_4)
- net TEMPMOTOR_IN: now also J5.5 (Pin_5); no longer J5.2 (Pin_2)
- net at R21.1, U6.6 (CANL): now also J8.3 (Pin_3); no longer J8.2 (Pin_2)
- net at R21.2, U6.7 (CANH): now also J8.2 (Pin_2); no longer J8.3 (Pin_3)
- net at R1.2: now also J5.2 (Pin_2); no longer J5.5 (Pin_5)
- net at R1.2: now also J5.3 (Pin_3); no longer J5.4 (Pin_4)
- net at R1.2: now also J5.4 (Pin_4); no longer J5.3 (Pin_3)
Other:
- moved on the sheet: C25, J5, R1

Commit message: shunts
Parts:
- J1: JLCPosOffset 3.75,0 -> -3.75,0; JLCRotOffset (none) -> -180
- J2: JLCPosOffset (none) -> -8.75,0; JLCRotOffset (none) -> -180
- J4, J5: JLCPosOffset 6.25,0 -> -6.25,0; JLCRotOffset (none) -> -180
- J7: JLCRotOffset (none) -> -90; MPN (none) -> C919361
- J8: JLCPosOffset 3.75,0 -> -3.75,0; JLCRotOffset (none) -> -180; MPN C265068 -> C157925
Connections:
- no-connect marks 2 -> 18
Changed lines of the file:
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@@
   (junction (at 229.87 55.88) (diameter 0) (color 0 0 0 0)
   )
+  (no_connect (at 260.35 133.35))
+  (no_connect (at 260.35 118.11))
+  (no_connect (at 260.35 128.27))
+  (no_connect (at 260.35 130.81))
+  (no_connect (at 224.79 110.49))
+  (no_connect (at 260.35 125.73))
+  (no_connect (at 260.35 110.49))
+  (no_connect (at 260.35 120.65))
+  (no_connect (at 224.79 130.81))
+  (no_connect (at 260.35 107.95))
+  (no_connect (at 260.35 105.41))
+  (no_connect (at 260.35 115.57))
   (no_connect (at 229.87 68.58))
+  (no_connect (at 260.35 113.03))
+  (no_connect (at 260.35 135.89))
   (no_connect (at 229.87 66.04))
+  (no_connect (at 224.79 113.03))
+  (no_connect (at 260.35 123.19))
   (wire (pts (xy 48.26 34.29) (xy 50.8 34.29))
     (stroke (width 0) (type default))
@@
       (effects (font (size 1.27 1.27)) hide)
     )
+    (property "MPN" "C919361" (at 166.37 66.04 0)
+      (effects (font (size 1.27 1.27)) hide)
+    )
+    (property "JLCRotOffset" "-90" (at 166.37 66.04 0)
+      (effects (font (size 1.27 1.27)) hide)
+    )
     (pin "1")
     (pin "2")
@@
       (effects (font (size 1.27 1.27)) hide)
     )
+    (property "JLCRotOffset" "-180" (at 81.28 34.29 0)
+      (effects (font (size 1.27 1.27)) hide)
+    )
+    (property "JLCPosOffset" "-8.75,0" (at 81.28 34.29 0)
+      (effects (font (size 1.27 1.27)) hide)
+    )
     (pin "1")
     (pin "2")
@@
       (effects (font (size 1.27 1.27)) hide)
     )
-    (property "JLCPosOffset" "6.25,0" (at 20.32 140.97 0)
+    (property "JLCPosOffset" "-6.25,0" (at 20.32 140.97 0)
+      (effects (font (size 1.27 1.27)) hide)
+    )
+    (property "JLCRotOffset" "-180" (at 20.32 140.97 0)
       (effects (font (size 1.27 1.27)) hide)
     )
@@
       (effects (font (size 1.27 1.27)) hide)
     )
-    (property "MPN" "C265068" (at 157.48 163.83 0)
-      (effects (font (size 1.27 1.27)) hide)
-    )
-    (property "JLCPosOffset" "3.75,0" (at 157.48 163.83 0)
+    (property "MPN" "C157925" (at 157.48 163.83 0)
+      (effects (font (size 1.27 1.27)) hide)
+    )
+    (property "JLCPosOffset" "-3.75,0" (at 157.48 163.83 0)
+      (effects (font (size 1.27 1.27)) hide)
+    )
+    (property "JLCRotOffset" "-180" (at 157.48 163.83 0)
       (effects (font (size 1.27 1.27)) hide)
     )
@@
       (effects (font (size 1.27 1.27)) hide)
     )
-    (property "JLCPosOffset" "6.25,0" (at 19.05 66.04 0)
+    (property "JLCPosOffset" "-6.25,0" (at 19.05 66.04 0)
+      (effects (font (size 1.27 1.27)) hide)
+    )
+    (property "JLCRotOffset" "-180" (at 19.05 66.04 0)
       (effects (font (size 1.27 1.27)) hide)
     )
@@
       (effects (font (size 1.27 1.27)) hide)
     )
-    (property "JLCPosOffset" "3.75,0" (at 21.59 31.75 0)
-      (effects (font (size 1.27 1.27)) hide)
-    )
+    (property "JLCPosOffset" "-3.75,0" (at 21.59 31.75 0)
+      (effects (font (size 1.27 1.27)) hide)
+    )
+    (property "JLCRotOffset" "-180" (at 21.59 31.75 0)
+      (effects (font (size 1.27 1.27)) hide)
+    )
