File: PowerBoard/PowerBoard.kicad_sch (KiCad schematic)
At the start: 13 parts, among them U4 RDE20110S12

Commit message: cheap_board
Parts:
- removed C28, C30: 680uF 200V, Capacitor_THT:CP_Radial_D18.0mm_P7.50mm, symbol Device:C_Polarized
- removed H5, H6: BATT+Hole, MountingHole:MountingHole_3.2mm_M3_Pad_Via, symbol Mechanical:MountingHole_Pad
- removed U4: RDE20110S12, Converter_DCDC:Converter_DCDC_TRACO_THN30-xxxx_THT, symbol GigaESCSymbols:RDE20110S12
- added C10: 47p 25V, Capacitor_SMD:C_0805_2012Metric, symbol Device:C
- added C11, C17: 4.7u 50V, Capacitor_SMD:C_1206_3216Metric, symbol Device:C
- added C12: 47p 100V, Capacitor_SMD:C_0603_1608Metric, symbol Device:C
- added C13: 1n, Capacitor_SMD:C_0603_1608Metric, symbol Device:C
- added C14: 2.2nF, Capacitor_SMD:C_0805_2012Metric, symbol Device:C
- added C15: 47u 16V, Capacitor_SMD:C_1210_3225Metric, symbol Device:C
- added C16: 470u 25V, Capacitor_SMD:CP_Elec_10x10.5, symbol Device:C_Polarized
- added C7: 1u 200V, Capacitor_SMD:C_2220_5650Metric, symbol Device:C
- added C8: 100n 200V, Capacitor_SMD:C_0805_2012Metric, symbol Device:C
- added C9: 100n, Capacitor_SMD:C_0805_2012Metric, symbol Device:C
- added D1: BAV20WS-7-F, Diode_SMD:D_SOD-323, symbol Diode:BAV20
- added D2: US1M, Diode_SMD:D_SMA, symbol Diode:US1M
- added D3: SMBJ188A, Diode_SMD:D_SMB, symbol Diode:SM6T6V8A
- added D4: FSV15120V, Package_TO_SOT_SMD:TO-277A, symbol Device:D_Schottky_AAK
- added D5: 3SMB5928B, Diode_SMD:D_SMB, symbol Device:D_Zener
- added J1: AuxConn, Connector_JST:JST_XH_B5B-XH-A_1x05_P2.50mm_Vertical, symbol Connector_Generic:Conn_01x05
- added Q1: STD11N65M2, Package_TO_SOT_SMD:TO-252-3_TabPin2, symbol Transistor_FET:STD7NK40Z
- added R1: 100k, Resistor_SMD:R_0805_2012Metric, symbol Device:R
- added R10: 121k, Resistor_SMD:R_0805_2012Metric, symbol Device:R
- added R11: 4.99k, Resistor_SMD:R_0805_2012Metric, symbol Device:R
- added R12: 44.2k, Resistor_SMD:R_0805_2012Metric, symbol Device:R
- added R13: 20, Resistor_SMD:R_0805_2012Metric, symbol Device:R
- added R14: 100, Resistor_SMD:R_0805_2012Metric, symbol Device:R
- added R15: 0.05, Resistor_SMD:R_2512_6332Metric, symbol Device:R
- added R16, R4: 20k, Resistor_SMD:R_0805_2012Metric, symbol Device:R
- added R2: 1.8k, Resistor_SMD:R_0805_2012Metric, symbol Device:R
- added R3: 499k, Resistor_SMD:R_1206_3216Metric, symbol Device:R
- added R6: 10k, Resistor_SMD:R_0805_2012Metric, symbol Device:R
- added R7: 56.2k, Resistor_SMD:R_0603_1608Metric, symbol Device:R
- added R8: 10, Resistor_SMD:R_0603_1608Metric, symbol Device:R
- added R9: 10k, Resistor_SMD:R_0603_1608Metric, symbol Device:R
- added SW1: POWER_SW, Connector_JST:JST_XH_B3B-XH-A_1x03_P2.50mm_Vertical, symbol Switch:SW_SPDT
- added T1: 11328-T078, GigaVescLibs:PQ2620, symbol GigaESCSymbols:Transformer_11328-T078
- added U2: LT8316EFE#PBF, GigaVescLibs:IC_LT8316EFE#PBF, symbol GigaESCSymbols:LT8316EFE#PBF
- C25, C26, C27, C31: footprint Capacitor_THT:CP_Radial_D18.0mm_P7.50mm -> Capacitor_THT:CP_Radial_D30.0mm_P10.00mm_SnapIn
- H4: value BATT+Hole -> BATT-Hole
Connections:
- net +BATT: now also C7.1, C8.1, D3.2 (A2), R1.1, R3.1, T1.1 (IN+), U2.1 (VIN), U2.2 (VIN), U2.3 (VIN); no longer H4.1
- net -BATT: now also H4.1, C10.2, C11.2, C13.2, C14.1, C17.2, C7.2, C8.2, C9.2, R11.2, R15.1, R16.1, R2.2, R4.1, R7.1, T1.5 (OUT1B), U2.15 (GND), U2.16 (SMODE), U2.20 (GND), U2.21 (GND); no longer H3.1
- new net: D1.1 (K), R8.2
- new net: C12.1, D1.2 (A), R12.1, T1.6 (OUT2A)
- new net: C11.1, R8.1, U2.9 (BIAS)
- new net: R4.2, SW1.1 (A)
- new net: D2.1 (K), D3.1 (A1)
- new net: R13.1, U2.19 (GATE)
- new net: Q1.1 (G), R13.2
- new net: D2.2 (A), Q1.2 (D), T1.3 (IN-)
- new net: Q1.3 (S), R14.2, R15.2
- new net: R7.2, U2.14 (IREG/SS)
- new net: D4.1 (A), D4.2 (A), T1.10 (PM), T1.11 (PM), T1.12 (PM)
- new net: R16.2, R3.2, SW1.3 (C)
- new net: R10.1, R11.1, R12.2, U2.12 (FB)
- new net: C13.1, R14.1, U2.18 (SENSE)
- new net: C9.1, R6.2
- new net: C12.2, R9.1
- new net: R9.2, U2.10 (DCM)
- new net: C10.1, R6.1, U2.13 (VC)
- new net: C17.1, U2.8 (INTVCC)
- new net: R10.2, U2.11 (TC)
- new net: SW1.2 (B), U2.17 (EN/UVLO)
- new net +12V: C15.1, C16.1, D4.3 (K), D5.1 (K), J1.4 (Pin_4), J1.5 (Pin_5)
- new net GND: C14.2, C15.2, C16.2, D5.2 (A), J1.2 (Pin_2), J1.3 (Pin_3), T1.7 (OUT2B), T1.8 (PM), T1.9 (PM)
- new net IN_V: J1.1 (Pin_1), R1.2, R2.1
- no-connect marks 0 -> 1
Other:
- note added: "EN Voltage divider has to provide voltage > 1.2V but cannot exeed 40V 499k and 20k gives operating range 32-300V+ giving 1.233V and 11.5V"
- note added: "Total Capacity 2720uF"
- note added: "Voltage divider 188V = 3.3V"
- note added: "replacement for CMZ5928B"
- note added: "replacement for FSV20120V 15A should still be plenty"
- note added: "replacement for STD6N90K5"
- note removed: "Total Capacity 4080uF"
- moved on the sheet: H3, H4

Commit message: cheap-mosfet-board
Parts:
- H1, H2, H3, H4: footprint MountingHole:MountingHole_3.2mm_M3_Pad_Via -> MountingHole:MountingHole_3.2mm_M3
Connections:
- net -BATT: no longer H1.1, H2.1, H4.1
- no-connect marks 1 -> 4
Changed lines of the file:
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@@
   (junction (at 196.85 92.71) (diameter 0) (color 0 0 0 0)
   )
-  (junction (at 55.88 30.48) (diameter 0) (color 0 0 0 0)
-  )
   (junction (at 165.1 139.7) (diameter 0) (color 0 0 0 0)
   )
@@
   (junction (at 66.04 99.06) (diameter 0) (color 0 0 0 0)
   )
-  (junction (at 35.56 30.48) (diameter 0) (color 0 0 0 0)
-  )
   (junction (at 196.85 95.25) (diameter 0) (color 0 0 0 0)
   )
@@
   (junction (at 227.33 113.03) (diameter 0) (color 0 0 0 0)
   )
+  (no_connect (at 35.56 30.48))
+  (no_connect (at 55.88 30.48))
   (no_connect (at 120.65 30.48))
+  (no_connect (at 76.2 30.48))
   (wire (pts (xy 116.84 147.32) (xy 129.54 147.32))
     (stroke (width 0) (type default))
@@
     (stroke (width 0) (type default))
   )
-  (wire (pts (xy 30.48 30.48) (xy 35.56 30.48))
-    (stroke (width 0) (type default))
-  )
   (wire (pts (xy 116.84 95.25) (xy 116.84 92.71))
     (stroke (width 0) (type default))
@@
     (stroke (width 0) (type default))
   )
-  (wire (pts (xy 35.56 30.48) (xy 55.88 30.48))
-    (stroke (width 0) (type default))
-  )
   (wire (pts (xy 66.04 83.82) (xy 54.61 83.82))
     (stroke (width 0) (type default))
@@
   )
   (wire (pts (xy 64.77 99.06) (xy 66.04 99.06))
-    (stroke (width 0) (type default))
-  )
-  (wire (pts (xy 55.88 30.48) (xy 76.2 30.48))
     (stroke (width 0) (type default))
   )
@@
     )
   )
-  (symbol (lib_id "power:-BATT") (at 30.48 30.48 90) (unit 1)
-    (in_bom yes) (on_board yes) (dnp no) (fields_autoplaced)
-    (property "Reference" "#PWR015" (at 34.29 30.48 0)
-      (effects (font (size 1.27 1.27)) hide)
-    )
-    (property "Value" "-BATT" (at 27.305 30.48 90)
-      (effects (font (size 1.27 1.27)) (justify left))
-    )
-    (property "Footprint" "" (at 30.48 30.48 0)
-      (effects (font (size 1.27 1.27)) hide)
-    )
-    (property "Datasheet" "" (at 30.48 30.48 0)
-      (effects (font (size 1.27 1.27)) hide)
-    )
-    (pin "1")
-    (instances
-      (project "MosfetBoard"
-        (path "/8a7bb686-c87a-43a6-b3d4-d988e8a2213f"
-          (reference "#PWR015") (unit 1)
-        )
-      )
-      (project "PowerBoard"
-        (path "/bd3f89f6-d222-47d4-8082-7044d630a3f6"
-          (reference "#PWR03") (unit 1)
-        )
-      )
-    )
-  )
   (symbol (lib_id "power:+12V") (at 237.49 60.96 270) (unit 1)
     (in_bom yes) (on_board yes) (dnp no) (fields_autoplaced)
@@
       (effects (font (size 1.27 1.27)) (justify left))
     )
-    (property "Footprint" "MountingHole:MountingHole_3.2mm_M3_Pad_Via" (at 55.88 27.94 0)
+    (property "Footprint" "MountingHole:MountingHole_3.2mm_M3" (at 55.88 27.94 0)
       (effects (font (size 1.27 1.27)) hide)
     )
@@
       (effects (font (size 1.27 1.27)) (justify left))
     )
-    (property "Footprint" "MountingHole:MountingHole_3.2mm_M3_Pad_Via" (at 76.2 27.94 0)
+    (property "Footprint" "MountingHole:MountingHole_3.2mm_M3" (at 76.2 27.94 0)
       (effects (font (size 1.27 1.27)) hide)
     )
@@
       (effects (font (size 1.27 1.27)) (justify left))
     )
-    (property "Footprint" "MountingHole:MountingHole_3.2mm_M3_Pad_Via" (at 35.56 27.94 0)
+    (property "Footprint" "MountingHole:MountingHole_3.2mm_M3" (at 35.56 27.94 0)
       (effects (font (size 1.27 1.27)) hide)
     )
@@
       (effects (font (size 1.27 1.27)) (justify left))
     )
-    (property "Footprint" "MountingHole:MountingHole_3.2mm_M3_Pad_Via" (at 120.65 27.94 0)
-      (effects (font (size 1.27 1.27)) hide)
-    )
+    (property "Footprint" "MountingHole:MountingHole_3.2mm_M3" (at 120.65 27.94 0)
+      (effects (font (size 1.27 1.27)) hide)
+    )

Commit message: shunts
Parts:
- removed C27, C31: 680uF 200V, Capacitor_THT:CP_Radial_D30.0mm_P10.00mm_SnapIn, symbol Device:C_Polarized
- C10: Mouser (none) -> 603-CC805JRNPO9BN470
- C11, C17: Mouser (none) -> 963-UMK316AB7475ML-T
- C12: Mouser (none) -> 80-C0603C470K1GAUTO
- C13: Mouser (none) -> 80-C0603C102K5R7081
- C14: Mouser (none) -> 603-CC805KRX7R0BB222
- C15: Mouser (none) -> 81-GRM32EC81C476KE5K
- C16: Mouser (none) -> 667-EEE-1EA471P
- C25: value 680uF 200V -> 2200uF 200V; MPN C238253 -> C2761574; Mouser (none) -> 661-EKMR201VS222MR50
- C26: value 680uF 200V -> 2200uF 200V; Mouser (none) -> 661-EKMR201VS222MR50
- C7: Mouser (none) -> 81-GRM55DR72D105KW1L
- C8: Mouser (none) -> 810-CGJ4J3X7T2D104K
- C9: Mouser (none) -> 581-08055C104KAT4A
- D1: Mouser (none) -> 621-BAV20WS-F
- D2: Mouser (none) -> 78-US1M-M35AT
- D3: Mouser (none) -> 576-SMBJ188A
- D4: Mouser (none) -> 512-FSV15120V
- D5: Mouser (none) -> 821-1SMB5928
- Q1: footprint Package_TO_SOT_SMD:TO-252-3_TabPin2 -> Package_TO_SOT_SMD:TO-252-2; JLCPosOffset 1.27,0 -> -1.27,0; JLCRotOffset -180 -> 0; Mouser (none) -> 511-STD11N65M2
- R1: Mouser (none) -> 603-RC0805FR-07100KL
- R10: Mouser (none) -> 660-RK73H2ATTD1213F
- R11: Mouser (none) -> 667-ERJ-6ENF4991V
- R12: Mouser (none) -> 603-RC0805FR-0744K2L
- R13: Mouser (none) -> 71-CRCW080520R0FKEAC
- R14: Mouser (none) -> 791-WR08X1000FTL
- R15: Mouser (none) -> 708-CSM2512FT50L0
- R16, R4: Mouser (none) -> 71-CRCW080520K0FKEB
- R2: Mouser (none) -> 71-CRCW0805-1.8K-E3
- R3: Mouser (none) -> 71-CRCW1206499KFKEB
- R6: Mouser (none) -> 603-AC0805JR-0710KL
- R7: Mouser (none) -> 652-CR0603FX-5622ELF
- R8: Mouser (none) -> 603-AF0603FR-0710RL
- R9: Mouser (none) -> 756-WCR0603-10KFI
- T1: Mouser (none) -> 851-11328-T078
- U2: Mouser (none) -> 584-LT8316EFE#PBF
Other:
- note added: "Total Capacity 4400uF"
- note removed: "Total Capacity 2720uF"
