File: PowerBoard/LTC7801/LTC7801.kicad_sch (KiCad schematic)
At the start: 47 parts, among them J1 AuxConn, Q2 BSC520N15NS3, Q3 BSC110N15NS5, SW2 POWER_SW, U1 LTC7801EUFD#PBF

Commit message: fixeddimensions
Parts:
- removed H1, H2, H3, H4: BATT-Hole, MountingHole:MountingHole_3.2mm_M3, symbol Mechanical:MountingHole_Pad
- removed Q2: BSC520N15NS3, Package_SON:Infineon_PG-TDSON-8_6.15x5.15mm, symbol Transistor_FET:STD7NK40Z
- removed Q3: BSC110N15NS5, Package_SON:Infineon_PG-TDSON-8_6.15x5.15mm, symbol Transistor_FET:STD7NK40Z
- added C25, C26 (x2): 330u 150V, Capacitor_THT:CP_Radial_D16.0mm_P7.50mm, symbol Device:C_Polarized
- added Q1: BSC520N15NS3, Package_TO_SOT_SMD:TDSON-8-1, symbol Transistor_FET:BSC079N10NSG
- added Q2: BSC110N15NS5, Package_TO_SOT_SMD:TDSON-8-1, symbol Transistor_FET:BSC079N10NSG
- C23, C28, C3: footprint Capacitor_SMD:C_0805_2012Metric -> GigaVescLibs:C_0603_1608Metric_L; MPN C28233 -> C14663
- C24, C4: footprint Capacitor_SMD:C_0603_1608Metric -> GigaVescLibs:C_0603_1608Metric_L
- C25: footprint Capacitor_SMD:C_1206_3216Metric -> GigaVescLibs:C_0603_1608Metric_L; MPN C29823 -> C19666
- C25, C26: value 2200uF 200V -> 330u 150V; footprint Capacitor_THT:CP_Radial_D30.0mm_P10.00mm_SnapIn -> Capacitor_THT:CP_Radial_D16.0mm_P7.50mm
- C26, C27: footprint Capacitor_SMD:C_0201_0603Metric -> GigaVescLibs:C_0603_1608Metric_L
- L1: value 100MHz 33uH 12A -> 100MHz 33uH 5A; footprint Inductor_SMD:L_Sunlord_MWSA0518S -> Inductor_SMD:L_Sunlord_MWSA1204S-220
- R1, R17, R19, R25: footprint Resistor_SMD:R_0805_2012Metric -> Resistor_SMD:R_0603_1608Metric; MPN C149504 -> C25803
- R18: footprint Resistor_SMD:R_0603_1608Metric -> Resistor_SMD:R_1206_3216Metric; MPN C22859 -> C17903
- R2: footprint Resistor_SMD:R_0805_2012Metric -> Resistor_SMD:R_0603_1608Metric; MPN C17398 -> C4177
- R22: value 80.6k -> 82k; MPN C304783 -> C23254
- R23: value 30.1k -> 30k; MPN C137745 -> C22984
- R26: value 140k 1% -> 130k; MPN C2933144 -> C22795
- R27: value 10k -> 9.1k; footprint Resistor_SMD:R_0805_2012Metric -> Resistor_SMD:R_0603_1608Metric; MPN C17414 -> C23260
- R28: footprint Resistor_SMD:R_0805_2012Metric -> Resistor_SMD:R_0603_1608Metric; MPN C17414 -> C25804
Connections:
- net GND is gone; now on net -BATT: J1.2 (Pin_2), J1.3 (Pin_3)
- net +BATT: now also C25.1, C26.1, C26.1, Q1.5 (D)
- net -BATT: now also C25.2, C26.2, C26.2, Q2.1 (S), Q2.2 (S), Q2.3 (S)
- net at C3.2, L1.1, U1.12 (SW): now also Q1.1 (S), Q1.2 (S), Q1.3 (S), Q2.5 (D)
- net at U1.11 (TG): now also Q1.4 (G)
- net at U1.14 (BG): now also Q2.4 (G)
- no-connect marks 4 -> 0
Other:
- note added: "Total Capacity 1980uF"
- note added: "non isolated"
- note removed: "Total Capacity 4400uF"
- moved on the sheet: J1, R1, R2
