File: PowerBoard/LTC7801/LTC7801.kicad_pcb (KiCad board)
At the start: 2 copper layers, 45 x 100 mm, 47 parts, among them J1 AuxConn, Q2 BSC520N15NS3, Q3 BSC110N15NS5, SW2 POWER_SW, U1 LTC7801EUFD#PBF

Commit message: fixeddimensions
Parts:
- removed H1, H2, H3, H4: BATT-Hole, MountingHole:MountingHole_3.2mm_M3
- removed Q3: BSC110N15NS5, Package_SON:Infineon_PG-TDSON-8_6.15x5.15mm
- added C10: 330u 150V, Capacitor_THT:CP_Radial_D16.0mm_P7.50mm, F.Cu at (66.0, 104.5)
- added C7: 330u 150V, Capacitor_THT:CP_Radial_D16.0mm_P7.50mm, F.Cu at (75.5, 104.5)
- added C8: 330u 150V, Capacitor_THT:CP_Radial_D16.0mm_P7.50mm, F.Cu at (66.0, 121.5)
- added Q1: BSC520N15NS3, Package_TO_SOT_SMD:TDSON-8-1, B.Cu at (70.5, 122.2)
- C1, C2: value 2200uF 200V -> 330u 150V; footprint Capacitor_THT:CP_Radial_D30.0mm_P10.00mm_SnapIn -> Capacitor_THT:CP_Radial_D16.0mm_P7.50mm
- C23, C28, C3: footprint Capacitor_SMD:C_0805_2012Metric -> GigaVescLibs:C_0603_1608Metric_L
- C24, C4: footprint Capacitor_SMD:C_0603_1608Metric -> GigaVescLibs:C_0603_1608Metric_L
- C25: footprint Capacitor_SMD:C_1206_3216Metric -> GigaVescLibs:C_0603_1608Metric_L
- C26, C27: footprint Capacitor_SMD:C_0201_0603Metric -> GigaVescLibs:C_0603_1608Metric_L
- L1: value 100MHz 33uH 12A -> 100MHz 33uH 5A; footprint Inductor_SMD:L_Sunlord_MWSA0518S -> Inductor_SMD:L_Sunlord_MWSA1204S-220; moved to F.Cu
- Q2: value BSC520N15NS3 -> BSC110N15NS5; footprint Package_SON:Infineon_PG-TDSON-8_6.15x5.15mm -> Package_TO_SOT_SMD:TDSON-8-1
- R1, R17, R19, R2, R25, R28: footprint Resistor_SMD:R_0805_2012Metric -> Resistor_SMD:R_0603_1608Metric
- R18: footprint Resistor_SMD:R_0603_1608Metric -> Resistor_SMD:R_1206_3216Metric
- R22: value 80.6k -> 82k
- R23: value 30.1k -> 30k
- R26: value 140k 1% -> 130k
- R27: value 10k -> 9.1k; footprint Resistor_SMD:R_0805_2012Metric -> Resistor_SMD:R_0603_1608Metric
- SW2: moved to F.Cu
- moved C24 90.6 mm to (63.0, 137.5), turned to 90 degrees
- moved R22 90.1 mm to (57.2, 131.5)
- moved R23 89.8 mm to (57.2, 133.0)
- moved U1 85.5 mm to (62.2, 132.0), turned to 90 degrees
- moved R18 83.5 mm to (64.5, 125.0), turned to 90 degrees
- moved R26 82.7 mm to (64.5, 137.5), turned to 90 degrees
- moved R25 81.5 mm to (57.2, 134.5), turned to 0 degrees
- moved R28 79.9 mm to (57.2, 136.2)
- moved C27 78.4 mm to (58.0, 138.5), turned to 90 degrees
- moved R27 77.7 mm to (61.5, 137.5), turned to -90 degrees
- moved C6 77.0 mm to (62.0, 111.0)
- moved C18 76.8 mm to (62.0, 117.0)
- moved C26 76.6 mm to (60.0, 137.2), turned to -90 degrees
- moved C4 72.1 mm to (82.2, 131.5), turned to -90 degrees
- moved R17 71.4 mm to (66.5, 124.5), turned to -90 degrees
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Connections:
- net SENSE- renamed +12V
- C3 pad 2: Net-(Q2-S) -> Net-(Q2-D)
- J1 pad 2: GND -> -BATT
- J1 pad 3: GND -> -BATT
- L1 pad 1: Net-(Q2-S) -> Net-(Q2-D)
- Q2 pad 1: Net-(Q2-G) -> -BATT
- Q2 pad 2: +BATT -> -BATT
- Q2 pad 3: Net-(Q2-S) -> -BATT
- Q2 pad 4: (no net) -> Net-(Q2-G)
- Q2 pad 5: (no net) -> Net-(Q2-D)
- U1 pad 11: Net-(Q2-G) -> Net-(Q1-G)
- U1 pad 12: Net-(Q2-S) -> Net-(Q2-D)
- U1 pad 14: Net-(Q3-G) -> Net-(Q2-G)
Routing:
- net +12V: track 0.00 -> 30.9 mm, vias 0 -> 2
- net -BATT: track 0.00 -> 29.8 mm, vias 36 -> 100
- net Net-(U1-OVLO): track 0.00 -> 27.0 mm
- net Net-(C24-Pad1): track 0.00 -> 24.5 mm
- net SENSE+: track 0.00 -> 22.3 mm, vias 0 -> 12
- net Net-(U1-CPUMP_EN): track 0.00 -> 19.0 mm, vias 0 -> 2
- net Net-(Q2-D): track 0.00 -> 17.0 mm, vias 0 -> 14
- net Net-(SW2-C): track 0.00 -> 17.0 mm, vias 0 -> 1
- net Net-(SW2-B): track 0.00 -> 16.6 mm, vias 0 -> 1
- net Net-(Q1-G): track 0.00 -> 15.4 mm, vias 0 -> 2
- net Net-(Q2-G): track 0.00 -> 11.6 mm, vias 0 -> 2
- net +BATT: track 0.00 -> 10.2 mm, vias 0 -> 30
- net Net-(U1-VIN): track 0.00 -> 8.42 mm
- net Net-(U1-ITH): track 0.00 -> 8.17 mm
- net IN_V: track 0.00 -> 7.38 mm
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- added copper zone on B.Cu, net Net-(Q2-D)
- added copper zone on B.Cu, net SENSE+
- removed copper zone on B.Cu, net (none)
- removed copper zone on F.Cu, net (none)
- removed copper zone on F.Cu, net +12V
- removed copper zone on B.Cu, net GND
Other:
- board size 45 x 100 mm -> 45 x 75 mm
