File: MosfetBoard/IPB072N15N3G/PhaseMosfets.kicad_sch (KiCad schematic)
At the start: 29 parts, among them J12 PHASE_PAD, Q1 IPB072N15N3G, Q2 IPB072N15N3G, Q4 IPB072N15N3G, Q5 IPB072N15N3G, U1 RS2166XC5, U3 ACS773ECB-200B-PFF-T

Commit message: cheap-mosfet-board
Parts:
- Q1, Q2, Q4, Q5: JLCPosOffset (none) -> -2.54,0
- U1: JLCRotOffset (none) -> -180
Connections:
- net PHASE: now also U3.5 (IP-); no longer U3.4 (IP+)
- net PHASE_OUT: now also U3.4 (IP+); no longer U3.5 (IP-)
- net +3.3V renamed 3.3V_IN
Other:
- moved on the sheet: C29, C34, L1, U3

Commit message: shunts
Parts:
- C1: Mouser (none) -> 81-GRM32EC72A106KE5K
- C29, C35, C36: Mouser (none) -> 581-08055C104KAT4A
- C34: Mouser (none) -> 187-CL21B225KPFNNNF
- C37: Mouser (none) -> 187-CL21B105KPFNNNE
- L1: Mouser (none) -> 81-BLM18HE152SN1D
- Q1, Q2, Q4, Q5: Mouser (none) -> 726-IPB072N15N3G
- R1: Mouser (none) -> 603-RT0805FRE07150KL
- R10, R11, R12, R9: Mouser (none) -> 71-TNPW08052R20DEEA
- R2: Mouser (none) -> 603-RT0805FRE072K7L
- R3: Mouser (none) -> 708-RNCP0805FTD10K0
- TH1: Mouser (none) -> 81-NCP18XH103F03RB
- U1: Mouser (none) -> 863-MC74VHC1G66DFT2G
Changed lines of the file:
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@@
+      (effects (font (size 1.27 1.27)) hide)
+    )
+    (property "Mouser" "726-IPB072N15N3G" (at 104.14 90.17 0)
       (effects (font (size 1.27 1.27)) hide)
     )
@@
     )
     (property "Datasheet" "~" (at 137.16 41.91 0)
+      (effects (font (size 1.27 1.27)) hide)
+    )
+    (property "Mouser" "81-GRM32EC72A106KE5K" (at 137.16 41.91 0)
       (effects (font (size 1.27 1.27)) hide)
     )
@@
       (effects (font (size 1.27 1.27)) hide)
     )
+    (property "Mouser" "726-IPB072N15N3G" (at 133.35 74.93 0)
+      (effects (font (size 1.27 1.27)) hide)
+    )
     (pin "1")
     (pin "2")
@@
     )
     (property "MPN" "C17470" (at 163.83 109.22 0)
+      (effects (font (size 1.27 1.27)) hide)
+    )
+    (property "Mouser" "603-RT0805FRE07150KL" (at 163.83 109.22 0)
       (effects (font (size 1.27 1.27)) hide)
     )
@@
       (effects (font (size 1.27 1.27)) hide)
     )
+    (property "Mouser" "726-IPB072N15N3G" (at 104.14 74.93 0)
+      (effects (font (size 1.27 1.27)) hide)
+    )
     (pin "1")
     (pin "2")
@@
       (effects (font (size 1.27 1.27)) hide)
     )
+    (property "Mouser" "81-GRM32EC72A106KE5K" (at 137.16 49.53 0)
+      (effects (font (size 1.27 1.27)) hide)
+    )
     (pin "1")
     (pin "2")
@@
       (effects (font (size 1.27 1.27)) hide)
     )
+    (property "Mouser" "81-NCP18XH103F03RB" (at 93.98 118.11 0)
+      (effects (font (size 1.27 1.27)) hide)
+    )
     (pin "1")
     (pin "2")
@@
       (effects (font (size 1.27 1.27)) hide)
     )
+    (property "Mouser" "81-GRM32EC72A106KE5K" (at 116.84 49.53 0)
+      (effects (font (size 1.27 1.27)) hide)
+    )
     (pin "1")
     (pin "2")
@@
       (effects (font (size 1.27 1.27)) hide)
     )
+    (property "Mouser" "581-08055C104KAT4A" (at 185.42 120.65 0)
+      (effects (font (size 1.27 1.27)) hide)
+    )
     (pin "1")
     (pin "2")
@@
       (effects (font (size 1.27 1.27)) hide)
     )
+    (property "Mouser" "71-TNPW08052R20DEEA" (at 124.46 74.93 0)
+      (effects (font (size 1.27 1.27)) hide)
+    )
     (pin "1")
     (pin "2")
@@
       (effects (font (size 1.27 1.27)) hide)
     )
+    (property "Mouser" "71-TNPW08052R20DEEA" (at 95.25 74.93 0)
+      (effects (font (size 1.27 1.27)) hide)
+    )
     (pin "1")
     (pin "2")
@@
       (effects (font (size 1.27 1.27)) hide)
     )
+    (property "Mouser" "708-RNCP0805FTD10K0" (at 93.98 128.27 0)
+      (effects (font (size 1.27 1.27)) hide)
+    )
     (pin "1")
     (pin "2")
@@
       (effects (font (size 1.27 1.27)) hide)
     )
+    (property "Mouser" "187-CL21B105KPFNNNE" (at 104.14 128.27 0)
+      (effects (font (size 1.27 1.27)) hide)
+    )
     (pin "1")
     (pin "2")
@@
       (effects (font (size 1.27 1.27)) hide)
     )
+    (property "Mouser" "71-TNPW08052R20DEEA" (at 95.25 90.17 0)
+      (effects (font (size 1.27 1.27)) hide)
+    )
     (pin "1")
     (pin "2")
@@
       (effects (font (size 1.27 1.27)) hide)
     )
+    (property "Mouser" "81-BLM18HE152SN1D" (at 167.64 57.15 0)
+      (effects (font (size 1.27 1.27)) hide)
+    )
     (pin "1")
     (pin "2")
@@
       (effects (font (size 1.27 1.27)) hide)
     )
+    (property "Mouser" "71-TNPW08052R20DEEA" (at 124.46 90.17 0)
+      (effects (font (size 1.27 1.27)) hide)
+    )
     (pin "1")
     (pin "2")
@@
     )
     (property "JLCRotOffset" "-180" (at 204.47 130.81 0)
+      (effects (font (size 1.27 1.27)) hide)
+    )
+    (property "Mouser" "863-MC74VHC1G66DFT2G" (at 204.47 130.81 0)
       (effects (font (size 1.27 1.27)) hide)
     )
@@
       (effects (font (size 1.27 1.27)) hide)
     )
+    (property "Mouser" "726-IPB072N15N3G" (at 133.35 90.17 0)
+      (effects (font (size 1.27 1.27)) hide)
+    )
     (pin "1")
     (pin "2")
@@
       (effects (font (size 1.27 1.27)) hide)
     )
+    (property "Mouser" "187-CL21B225KPFNNNF" (at 180.34 60.96 0)
+      (effects (font (size 1.27 1.27)) hide)
+    )
     (pin "1")
     (pin "2")
@@
       (effects (font (size 1.27 1.27)) hide)
     )
+    (property "Mouser" "581-08055C104KAT4A" (at 160.02 62.23 0)
+      (effects (font (size 1.27 1.27)) hide)
+    )
     (pin "1")
     (pin "2")
@@
       (effects (font (size 1.27 1.27)) hide)
     )
+    (property "Mouser" "603-RT0805FRE072K7L" (at 163.83 119.38 0)
+      (effects (font (size 1.27 1.27)) hide)
+    )
     (pin "1")
     (pin "2")
@@
       (effects (font (size 1.27 1.27)) hide)
     )
+    (property "Mouser" "81-GRM32EC72A106KE5K" (at 116.84 41.91 0)
+      (effects (font (size 1.27 1.27)) hide)
+    )
     (pin "1")
     (pin "2")
@@
       (effects (font (size 1.27 1.27)) hide)
     )
+    (property "Mouser" "81-GRM32EC72A106KE5K" (at 106.68 41.91 0)
+      (effects (font (size 1.27 1.27)) hide)
+    )
     (pin "1")
     (pin "2")
@@
       (effects (font (size 1.27 1.27)) hide)
     )
+    (property "Mouser" "81-GRM32EC72A106KE5K" (at 127 41.91 0)
+      (effects (font (size 1.27 1.27)) hide)
+    )
     (pin "1")
     (pin "2")
@@
       (effects (font (size 1.27 1.27)) hide)
     )
+    (property "Mouser" "581-08055C104KAT4A" (at 185.42 138.43 0)
+      (effects (font (size 1.27 1.27)) hide)
+    )
     (pin "1")
     (pin "2")
@@
       (effects (font (size 1.27 1.27)) hide)
     )
+    (property "Mouser" "81-GRM32EC72A106KE5K" (at 127 49.53 0)
+      (effects (font (size 1.27 1.27)) hide)
+    )
     (pin "1")
     (pin "2")
@@
       (effects (font (size 1.27 1.27)) hide)
     )
+    (property "Mouser" "81-GRM32EC72A106KE5K" (at 106.68 49.53 0)
+      (effects (font (size 1.27 1.27)) hide)
+    )

Commit message: nearlyready
Parts:
- C1: MPN (none) -> C5156756
- Q1, Q2, Q4, Q5: MPN (none) -> C459162
- R10, R11, R12, R9: Mouser 71-TNPW08052R20DEEA -> 603-AC0805JR-072R2L
- U3: MPN (none) -> C163288; Mouser (none) -> 250-758ECB200BPSST
Changed lines of the file:
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@@
+      (effects (font (size 1.27 1.27)) hide)
+    )
+    (property "MPN" "C459162" (at 104.14 90.17 0)
       (effects (font (size 1.27 1.27)) hide)
     )
@@
     )
     (property "Mouser" "81-GRM32EC72A106KE5K" (at 137.16 41.91 0)
+      (effects (font (size 1.27 1.27)) hide)
+    )
+    (property "MPN" "C5156756" (at 137.16 41.91 0)
       (effects (font (size 1.27 1.27)) hide)
     )
@@
       (effects (font (size 1.27 1.27)) hide)
     )
+    (property "MPN" "C459162" (at 133.35 74.93 0)
+      (effects (font (size 1.27 1.27)) hide)
+    )
     (pin "1")
     (pin "2")
@@
       (effects (font (size 1.27 1.27)) hide)
     )
+    (property "MPN" "C459162" (at 104.14 74.93 0)
+      (effects (font (size 1.27 1.27)) hide)
+    )
     (pin "1")
     (pin "2")
@@
       (effects (font (size 1.27 1.27)) hide)
     )
+    (property "MPN" "C5156756" (at 137.16 49.53 0)
+      (effects (font (size 1.27 1.27)) hide)
+    )
     (pin "1")
     (pin "2")
@@
       (effects (font (size 1.27 1.27)) hide)
     )
+    (property "MPN" "C5156756" (at 116.84 49.53 0)
+      (effects (font (size 1.27 1.27)) hide)
+    )
     (pin "1")
     (pin "2")
@@
       (effects (font (size 1.27 1.27)) hide)
     )
-    (property "Mouser" "71-TNPW08052R20DEEA" (at 124.46 74.93 0)
+    (property "Mouser" "603-AC0805JR-072R2L" (at 124.46 74.93 0)
       (effects (font (size 1.27 1.27)) hide)
     )
@@
       (effects (font (size 1.27 1.27)) hide)
     )
-    (property "Mouser" "71-TNPW08052R20DEEA" (at 95.25 74.93 0)
+    (property "Mouser" "603-AC0805JR-072R2L" (at 95.25 74.93 0)
       (effects (font (size 1.27 1.27)) hide)
     )
@@
       (effects (font (size 1.27 1.27)) hide)
     )
-    (property "Mouser" "71-TNPW08052R20DEEA" (at 95.25 90.17 0)
+    (property "Mouser" "603-AC0805JR-072R2L" (at 95.25 90.17 0)
       (effects (font (size 1.27 1.27)) hide)
     )
@@
       (effects (font (size 1.27 1.27)) hide)
     )
-    (property "Mouser" "71-TNPW08052R20DEEA" (at 124.46 90.17 0)
+    (property "Mouser" "603-AC0805JR-072R2L" (at 124.46 90.17 0)
       (effects (font (size 1.27 1.27)) hide)
     )
@@
       (effects (font (size 1.27 1.27)) hide)
     )
+    (property "MPN" "C163288" (at 173.99 80.01 0)
+      (effects (font (size 1.27 1.27)) hide)
+    )
+    (property "Mouser" "250-758ECB200BPSST" (at 173.99 80.01 0)
+      (effects (font (size 1.27 1.27)) hide)
+    )
     (pin "1")
     (pin "2")
@@
       (effects (font (size 1.27 1.27)) hide)
     )
+    (property "MPN" "C459162" (at 133.35 90.17 0)
+      (effects (font (size 1.27 1.27)) hide)
+    )
     (pin "1")
     (pin "2")
@@
       (effects (font (size 1.27 1.27)) hide)
     )
+    (property "MPN" "C5156756" (at 116.84 41.91 0)
+      (effects (font (size 1.27 1.27)) hide)
+    )
     (pin "1")
     (pin "2")
@@
       (effects (font (size 1.27 1.27)) hide)
     )
+    (property "MPN" "C5156756" (at 127 41.91 0)
+      (effects (font (size 1.27 1.27)) hide)
+    )
     (pin "1")
     (pin "2")
@@
       (effects (font (size 1.27 1.27)) hide)
     )
+    (property "MPN" "C5156756" (at 127 49.53 0)
+      (effects (font (size 1.27 1.27)) hide)
+    )
     (pin "1")
     (pin "2")
@@
       (effects (font (size 1.27 1.27)) hide)
     )
+    (property "MPN" "C5156756" (at 106.68 49.53 0)
+      (effects (font (size 1.27 1.27)) hide)
+    )

Commit message: fixeddimensions
Parts:
- added J1: DRIVER1, Connector_PinSocket_2.54mm:PinSocket_2x02_P2.54mm_Vertical_SMD, symbol Connector_Generic:Conn_01x04
- added J4: PhaseConn, Connector_PinSocket_2.54mm:PinSocket_2x03_P2.54mm_Vertical_SMD, symbol Connector_Generic:Conn_02x03_Counter_Clockwise
Connections:
- net -BATT: now also J1.4 (Pin_4)
- net 3.3V_IN: now also J4.5 (Pin_5)
- net GND: now also J4.1 (Pin_1)
- net PH: now also J1.1 (Pin_1)
- net PHASE: now also J1.3 (Pin_3)
- net PL: now also J1.2 (Pin_2)
- net SENSE_FILTER_EN: now also J4.3 (Pin_3)
- net CURR renamed CURRENT_SENSE
- net CURRENT_SENSE: now also J4.6 (Pin_6)
- net MOSTEMP renamed MOS_TEMP
- net MOS_TEMP: now also J4.4 (Pin_4)
- net VSENSE renamed V_SENSE
- net V_SENSE: now also J4.2 (Pin_2)

Commit message: cleanup
Parts:
- removed J12: PHASE_PAD, Connector_Wire:SolderWirePad_1x01_SMD_5x10mm, symbol Connector:Conn_01x01_Pin
Changed lines of the file:
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@@
-    (effects (font (size 1.27 1.27)) (justify right bottom))
-  )
-  (label "PHASE_OUT" (at 231.14 102.87 180) (fields_autoplaced)
     (effects (font (size 1.27 1.27)) (justify right bottom))
   )
@@
         )
       )
-    )
-  )
-  (symbol (lib_id "Connector:Conn_01x01_Pin") (at 236.22 102.87 180) (unit 1)
-    (in_bom yes) (on_board yes) (dnp no) (fields_autoplaced)
-    (property "Reference" "J12" (at 235.585 97.79 0)
-      (effects (font (size 1.27 1.27)))
-    )
-    (property "Value" "PHASE_PAD" (at 235.585 100.33 0)
-      (effects (font (size 1.27 1.27)))
-    )
-    (property "Footprint" "Connector_Wire:SolderWirePad_1x01_SMD_5x10mm" (at 236.22 102.87 0)
-      (effects (font (size 1.27 1.27)) hide)
-    )
-    (property "Datasheet" "~" (at 236.22 102.87 0)
-      (effects (font (size 1.27 1.27)) hide)
-    )
-    (pin "1")
-    (instances
-      (project "IPB072N15N3G"
-        (path "/8a7bb686-c87a-43a6-b3d4-d988e8a2213f"
-          (reference "J12") (unit 1)
-        )
-        (path "/8a7bb686-c87a-43a6-b3d4-d988e8a2213f/3d569e84-87d6-4696-b0ce-a4e576394c1a"
-          (reference "J7") (unit 1)
-        )
-        (path "/8a7bb686-c87a-43a6-b3d4-d988e8a2213f/db7451b3-bde8-4d72-ba04-6d13b057caad"
-          (reference "J15") (unit 1)
-        )
-        (path "/8a7bb686-c87a-43a6-b3d4-d988e8a2213f/ccaed507-63cb-4563-a707-3e0cba7d2643"
-          (reference "J16") (unit 1)
-        )
-      )

Commit message: minor
Parts:
- R10, R11, R12, R9: value 2r2 -> 2.2
Changed lines of the file:
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@@
       (effects (font (size 1.27 1.27)))
     )
-    (property "Value" "2r2" (at 124.46 74.93 90)
+    (property "Value" "2.2" (at 124.46 74.93 90)
       (effects (font (size 1.27 1.27)))
     )
@@
       (effects (font (size 1.27 1.27)))
     )
-    (property "Value" "2r2" (at 95.25 74.93 90)
+    (property "Value" "2.2" (at 95.25 74.93 90)
       (effects (font (size 1.27 1.27)))
     )
@@
       (effects (font (size 1.27 1.27)))
     )
-    (property "Value" "2r2" (at 95.25 90.17 90)
+    (property "Value" "2.2" (at 95.25 90.17 90)
       (effects (font (size 1.27 1.27)))
     )
@@
       (effects (font (size 1.27 1.27)))
     )
-    (property "Value" "2r2" (at 124.46 90.17 90)
-      (effects (font (size 1.27 1.27)))
-    )
+    (property "Value" "2.2" (at 124.46 90.17 90)
+      (effects (font (size 1.27 1.27)))
+    )
