File: MosfetBoard/IPB072N15N3G/IPB072N15N3G.kicad_sch (KiCad schematic)
At the start: 10 parts, among them J1 DRIVER1, J13 BATT+Conn2, J14 BATT-Conn2, J2 DRIVER2, J3 DRIVER3, J4 PhaseConn1, J5 PhaseConn2, J6 PhaseConn3, J8 BATT+Conn1, J9 BATT-Conn1

Commit message: cheap-mosfet-board
Parts:
- J1, J2, J3, J4, J5, J6: JLCRotOffset (none) -> -90
Connections:
- removed net +3.3V: J4.5 (Pin_5), J5.5 (Pin_5), J6.5 (Pin_5)
- new net 3.3V_1: J4.5 (Pin_5)
- new net 3.3V_2: J5.5 (Pin_5)
- new net 3.3V_3: J6.5 (Pin_5)
Other:
- sheet PhaseMosfets ports: added 3.3V_IN; removed none
- sheet PhaseMosfets1 ports: added 3.3V_IN; removed none
- sheet PhaseMosfets2 ports: added 3.3V_IN; removed none
Changed lines of the file:
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@@
+    )
+  )
+  (global_label "3.3V_2" (shape input) (at 68.58 95.25 0) (fields_autoplaced)
+    (effects (font (size 1.27 1.27)) (justify left))
+    (property "Intersheetrefs" "${INTERSHEET_REFS}" (at 77.7753 95.25 0)
+      (effects (font (size 1.27 1.27)) (justify left) hide)
     )
   )
@@
     )
   )
+  (global_label "3.3V_3" (shape input) (at 68.58 129.54 0) (fields_autoplaced)
+    (effects (font (size 1.27 1.27)) (justify left))
+    (property "Intersheetrefs" "${INTERSHEET_REFS}" (at 77.7753 129.54 0)
+      (effects (font (size 1.27 1.27)) (justify left) hide)
+    )
+  )
   (global_label "C" (shape input) (at 68.58 123.19 0) (fields_autoplaced)
     (effects (font (size 1.27 1.27)) (justify left))
@@
     )
   )
+  (global_label "3.3V_3" (shape input) (at 115.57 189.23 0) (fields_autoplaced)
+    (effects (font (size 1.27 1.27)) (justify left))
+    (property "Intersheetrefs" "${INTERSHEET_REFS}" (at 124.7653 189.23 0)
+      (effects (font (size 1.27 1.27)) (justify left) hide)
+    )
+  )
+  (global_label "3.3V_1" (shape input) (at 115.57 157.48 0) (fields_autoplaced)
+    (effects (font (size 1.27 1.27)) (justify left))
+    (property "Intersheetrefs" "${INTERSHEET_REFS}" (at 124.7653 157.48 0)
+      (effects (font (size 1.27 1.27)) (justify left) hide)
+    )
+  )
   (global_label "CURR1" (shape input) (at 68.58 72.39 0) (fields_autoplaced)
     (effects (font (size 1.27 1.27)) (justify left))
@@
     )
   )
+  (global_label "3.3V_1" (shape input) (at 68.58 60.96 0) (fields_autoplaced)
+    (effects (font (size 1.27 1.27)) (justify left))
+    (property "Intersheetrefs" "${INTERSHEET_REFS}" (at 77.7753 60.96 0)
+      (effects (font (size 1.27 1.27)) (justify left) hide)
+    )
+  )
   (global_label "PH3" (shape input) (at 38.1 125.73 180) (fields_autoplaced)
     (effects (font (size 1.27 1.27)) (justify right))
@@
     )
   )
+  (global_label "3.3V_2" (shape input) (at 115.57 173.99 0) (fields_autoplaced)
+    (effects (font (size 1.27 1.27)) (justify left))
+    (property "Intersheetrefs" "${INTERSHEET_REFS}" (at 124.7653 173.99 0)
+      (effects (font (size 1.27 1.27)) (justify left) hide)
+    )
+  )
   (global_label "SENS_FILTER_ENABLE1" (shape input) (at 102.87 160.02 180) (fields_autoplaced)
     (effects (font (size 1.27 1.27)) (justify right))
@@
     )
     (property "MPN" "C3975147" (at 67.31 20.32 90)
+      (effects (font (size 1.27 1.27)) hide)
+    )
+    (property "JLCRotOffset" "-90" (at 67.31 20.32 90)
       (effects (font (size 1.27 1.27)) hide)
     )
@@
       (effects (font (size 1.27 1.27)) hide)
     )
+    (property "JLCRotOffset" "-90" (at 50.8 20.32 90)
+      (effects (font (size 1.27 1.27)) hide)
+    )
     (pin "1")
     (pin "2")
@@
     )
   )
-  (symbol (lib_id "power:+3.3V") (at 115.57 189.23 270) (unit 1)
-    (in_bom yes) (on_board yes) (dnp no) (fields_autoplaced)
-    (property "Reference" "#PWR022" (at 111.76 189.23 0)
-      (effects (font (size 1.27 1.27)) hide)
-    )
-    (property "Value" "+3.3V" (at 119.38 189.23 90)
-      (effects (font (size 1.27 1.27)) (justify left))
-    )
-    (property "Footprint" "" (at 115.57 189.23 0)
-      (effects (font (size 1.27 1.27)) hide)
-    )
-    (property "Datasheet" "" (at 115.57 189.23 0)
-      (effects (font (size 1.27 1.27)) hide)
-    )
-    (pin "1")
-    (instances
-      (project "IPB072N15N3G"
-        (path "/8a7bb686-c87a-43a6-b3d4-d988e8a2213f"
-          (reference "#PWR022") (unit 1)
-        )
-      )
-    )
-  )
   (symbol (lib_id "Connector_Generic:Conn_02x03_Counter_Clockwise") (at 107.95 157.48 0) (unit 1)
     (in_bom yes) (on_board yes) (dnp no) (fields_autoplaced)
@@
     )
     (property "MPN" "C5160818" (at 107.95 157.48 0)
+      (effects (font (size 1.27 1.27)) hide)
+    )
+    (property "JLCRotOffset" "-90" (at 107.95 157.48 0)
       (effects (font (size 1.27 1.27)) hide)
     )
@@
       (effects (font (size 1.27 1.27)) hide)
     )
+    (property "JLCRotOffset" "-90" (at 107.95 189.23 0)
+      (effects (font (size 1.27 1.27)) hide)
+    )
     (pin "1")
     (pin "2")
@@
       (effects (font (size 1.27 1.27)) hide)
     )
+    (property "JLCRotOffset" "-90" (at 107.95 173.99 0)
+      (effects (font (size 1.27 1.27)) hide)
+    )
     (pin "1")
     (pin "2")
@@
     )
   )
-  (symbol (lib_id "power:+3.3V") (at 115.57 173.99 270) (unit 1)
-    (in_bom yes) (on_board yes) (dnp no) (fields_autoplaced)
-    (property "Reference" "#PWR021" (at 111.76 173.99 0)
-      (effects (font (size 1.27 1.27)) hide)
-    )
-    (property "Value" "+3.3V" (at 119.38 173.99 90)
-      (effects (font (size 1.27 1.27)) (justify left))
-    )
-    (property "Footprint" "" (at 115.57 173.99 0)
-      (effects (font (size 1.27 1.27)) hide)
-    )
-    (property "Datasheet" "" (at 115.57 173.99 0)
-      (effects (font (size 1.27 1.27)) hide)
-    )
-    (pin "1")
-    (instances
-      (project "IPB072N15N3G"
-        (path "/8a7bb686-c87a-43a6-b3d4-d988e8a2213f"
-          (reference "#PWR021") (unit 1)
-        )
-      )
-    )
-  )
   (symbol (lib_id "Connector:Conn_01x01_Pin") (at 101.6 46.99 0) (unit 1)
     (in_bom yes) (on_board yes) (dnp no)
@@
       (effects (font (size 1.27 1.27)) hide)
     )
+    (property "JLCRotOffset" "-90" (at 34.29 20.32 90)
+      (effects (font (size 1.27 1.27)) hide)
+    )
     (pin "1")
     (pin "2")
@@
         (path "/8a7bb686-c87a-43a6-b3d4-d988e8a2213f"
           (reference "J8") (unit 1)
-        )
-      )
-    )
-  )
-  (symbol (lib_id "power:+3.3V") (at 115.57 157.48 270) (unit 1)
-    (in_bom yes) (on_board yes) (dnp no) (fields_autoplaced)
-    (property "Reference" "#PWR020" (at 111.76 157.48 0)
-      (effects (font (size 1.27 1.27)) hide)
-    )
-    (property "Value" "+3.3V" (at 119.38 157.48 90)
-      (effects (font (size 1.27 1.27)) (justify left))
-    )
-    (property "Footprint" "" (at 115.57 157.48 0)
-      (effects (font (size 1.27 1.27)) hide)
-    )
-    (property "Datasheet" "" (at 115.57 157.48 0)
-      (effects (font (size 1.27 1.27)) hide)
-    )
-    (pin "1")
-    (instances
-      (project "IPB072N15N3G"
-        (path "/8a7bb686-c87a-43a6-b3d4-d988e8a2213f"
-          (reference "#PWR020") (unit 1)
         )
       )
@@
       (effects (font (size 1.27 1.27)) (justify right))
     )
+    (pin "3.3V_IN" input (at 68.58 60.96 0)
+      (effects (font (size 1.27 1.27)) (justify right))
+    )
     (instances
       (project "IPB072N15N3G"
@@
       (effects (font (size 1.27 1.27)) (justify right))
     )
+    (pin "3.3V_IN" input (at 68.58 129.54 0)
+      (effects (font (size 1.27 1.27)) (justify right))
+    )
     (instances
       (project "IPB072N15N3G"
@@
       (effects (font (size 1.27 1.27)) (justify right))
     )
+    (pin "3.3V_IN" input (at 68.58 95.25 0)
+      (effects (font (size 1.27 1.27)) (justify right))
+    )

Commit message: shunts
Parts:
- J1, J2, J3: Mouser (none) -> 855-M20-7870246
- J4, J5, J6: Mouser (none) -> 855-M20-7870346
Changed lines of the file:
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@@
+      (effects (font (size 1.27 1.27)) hide)
+    )
+    (property "Mouser" "855-M20-7870246" (at 67.31 20.32 0)
       (effects (font (size 1.27 1.27)) hide)
     )
@@
       (effects (font (size 1.27 1.27)) hide)
     )
+    (property "Mouser" "855-M20-7870246" (at 50.8 20.32 0)
+      (effects (font (size 1.27 1.27)) hide)
+    )
     (pin "1")
     (pin "2")
@@
     )
     (property "JLCRotOffset" "-90" (at 107.95 157.48 0)
+      (effects (font (size 1.27 1.27)) hide)
+    )
+    (property "Mouser" "855-M20-7870346" (at 107.95 157.48 0)
       (effects (font (size 1.27 1.27)) hide)
     )
@@
       (effects (font (size 1.27 1.27)) hide)
     )
+    (property "Mouser" "855-M20-7870346" (at 107.95 189.23 0)
+      (effects (font (size 1.27 1.27)) hide)
+    )
     (pin "1")
     (pin "2")
@@
     )
     (property "JLCRotOffset" "-90" (at 107.95 173.99 0)
+      (effects (font (size 1.27 1.27)) hide)
+    )
+    (property "Mouser" "855-M20-7870346" (at 107.95 173.99 0)
       (effects (font (size 1.27 1.27)) hide)
     )
@@
       (effects (font (size 1.27 1.27)) hide)
     )
+    (property "Mouser" "855-M20-7870246" (at 34.29 20.32 0)
+      (effects (font (size 1.27 1.27)) hide)
+    )

Commit message: fixeddimensions
Parts:
- removed J1: DRIVER1, Connector_PinSocket_2.54mm:PinSocket_2x02_P2.54mm_Vertical_SMD, symbol Connector_Generic:Conn_01x04
- removed J2: DRIVER2, Connector_PinSocket_2.54mm:PinSocket_2x02_P2.54mm_Vertical_SMD, symbol Connector_Generic:Conn_01x04
- removed J3: DRIVER3, Connector_PinSocket_2.54mm:PinSocket_2x02_P2.54mm_Vertical_SMD, symbol Connector_Generic:Conn_01x04
- removed J4: PhaseConn1, Connector_PinSocket_2.54mm:PinSocket_2x03_P2.54mm_Vertical_SMD, symbol Connector_Generic:Conn_02x03_Counter_Clockwise
- removed J5: PhaseConn2, Connector_PinSocket_2.54mm:PinSocket_2x03_P2.54mm_Vertical_SMD, symbol Connector_Generic:Conn_02x03_Counter_Clockwise
- removed J6: PhaseConn3, Connector_PinSocket_2.54mm:PinSocket_2x03_P2.54mm_Vertical_SMD, symbol Connector_Generic:Conn_02x03_Counter_Clockwise
Other:
- removed sheet PhaseMosfets
- added sheet PhaseMosfets3 (PhaseMosfets.kicad_sch)
- note removed: "Sense filter enable is connected on logic board"

Commit message: cleanup
Other:
- sheet PhaseMosfets1 ports: added none; removed 3.3V_IN, CURR, MOSTEMP, PH, PHASE, PHASE_OUT, PL, SENSE_FILTER_EN, VSENSE
- sheet PhaseMosfets2 ports: added none; removed 3.3V_IN, CURR, MOSTEMP, PH, PHASE, PHASE_OUT, PL, SENSE_FILTER_EN, VSENSE
- sheet PhaseMosfets3 ports: added none; removed 3.3V_IN, CURR, MOSTEMP, PH, PHASE, PHASE_OUT, PL, SENSE_FILTER_EN, VSENSE

Commit message: v3.0.2 - IPB v2
Parts:
- removed J13: BATT+Conn2, Connector_Wire:SolderWirePad_1x01_SMD_5x10mm, symbol Connector:Conn_01x01_Pin
- removed J14: BATT-Conn2, Connector_Wire:SolderWirePad_1x01_SMD_5x10mm, symbol Connector:Conn_01x01_Pin
- removed J8: BATT+Conn1, Connector_Wire:SolderWirePad_1x01_SMD_5x10mm, symbol Connector:Conn_01x01_Pin
- removed J9: BATT-Conn1, Connector_Wire:SolderWirePad_1x01_SMD_5x10mm, symbol Connector:Conn_01x01_Pin
- added H1 (x2): MountingHole_Pad, MountingHole:MountingHole_5.3mm_M5_Pad_Via, symbol Mechanical:MountingHole_Pad
- added H1, H2, H3, H4: MountingHole, MountingHole:MountingHole_3.2mm_M3_ISO14580, symbol Mechanical:MountingHole
- added J1: LogicConnector, Connector_PinSocket_2.54mm:PinSocket_2x15_P2.54mm_Vertical, symbol Connector_Generic:Conn_02x15_Odd_Even
- added JP1: Jumper_2_Open, GigaVescLibs:SolderJumper0.5mm_Open, symbol Jumper:Jumper_2_Open
Connections:
- net +BATT: now also H1.1, JP1.1 (A)
- net -BATT: now also H1.1, J1.29 (Pin_29), J1.30 (Pin_30)
- new net: J1.1 (Pin_1), JP1.2 (B)
- new net 3.3V: J1.2 (Pin_2)
- new net 5V: J1.4 (Pin_4)
- new net PH1: J1.6 (Pin_6)
- new net PH2: J1.14 (Pin_14)
- new net PH3: J1.22 (Pin_22)
- new net PHASE1: J1.8 (Pin_8)
- new net PHASE2: J1.16 (Pin_16)
- new net PHASE3: J1.24 (Pin_24)
- new net PHASE_GROUND1: J1.12 (Pin_12)
- new net PHASE_GROUND2: J1.20 (Pin_20)
- new net PHASE_GROUND3: J1.28 (Pin_28)
- new net PL1: J1.10 (Pin_10)
- new net PL2: J1.18 (Pin_18)
- new net PL3: J1.26 (Pin_26)
- new net PhaseMosfets1/MOS_TEMP: J1.5 (Pin_5)
- new net PhaseMosfets1/SH+: J1.11 (Pin_11)
- new net PhaseMosfets1/SH-: J1.9 (Pin_9)
- new net PhaseMosfets1/V_SENSE: J1.7 (Pin_7)
- new net PhaseMosfets2/MOS_TEMP: J1.13 (Pin_13)
- new net PhaseMosfets2/SH+: J1.19 (Pin_19)
- new net PhaseMosfets2/SH-: J1.17 (Pin_17)
- new net PhaseMosfets2/V_SENSE: J1.15 (Pin_15)
- new net PhaseMosfets3/MOS_TEMP: J1.21 (Pin_21)
- new net PhaseMosfets3/SH+: J1.27 (Pin_27)
- new net PhaseMosfets3/SH-: J1.25 (Pin_25)
- new net PhaseMosfets3/V_SENSE: J1.23 (Pin_23)
Other:
- sheet PhaseMosfets1 ports: added 3.3V_IN, 5V_IN, MOS_TEMP, PH, PHASE, PHASE_GROUND, PL, SH+, SH-, V_SENSE; removed none
- sheet PhaseMosfets2 ports: added 3.3V_IN, 5V_IN, MOS_TEMP, PH, PHASE, PHASE_GROUND, PL, SH+, SH-, V_SENSE; removed none
- sheet PhaseMosfets3 ports: added 3.3V_IN, 5V_IN, MOS_TEMP, PH, PHASE, PHASE_GROUND, PL, SH+, SH-, V_SENSE; removed none

Commit message: v3.0.2 - Prerelease
Connections:
- net PhaseMosfets1/V_SENSE: no longer names the net of J1.7 (Pin_7)
- net PhaseMosfets2/V_SENSE: no longer names the net of J1.15 (Pin_15)
- net PhaseMosfets3/V_SENSE: no longer names the net of J1.23 (Pin_23)
- no-connect marks 0 -> 4
Other:
- sheet PhaseMosfets1 ports: added none; removed V_SENSE
- sheet PhaseMosfets2 ports: added none; removed V_SENSE
- sheet PhaseMosfets3 ports: added none; removed V_SENSE
Changed lines of the file:
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@@
 (kicad_sch (version 20230121) (generator eeschema)
   (paper "A4")
+  (no_connect (at 143.51 104.14))
+  (no_connect (at 143.51 93.98))
+  (no_connect (at 143.51 88.9))
+  (no_connect (at 143.51 114.3))
   (wire (pts (xy 85.09 115.57) (xy 110.49 115.57))
     (stroke (width 0) (type default))
@@
     (stroke (width 0) (type default))
   )
-  (wire (pts (xy 85.09 151.13) (xy 115.57 151.13))
-    (stroke (width 0) (type default))
-  )
   (wire (pts (xy 110.49 115.57) (xy 110.49 109.22))
     (stroke (width 0) (type default))
@@
     (stroke (width 0) (type default))
   )
-  (wire (pts (xy 107.95 69.85) (xy 107.95 93.98))
-    (stroke (width 0) (type default))
-  )
   (wire (pts (xy 102.87 101.6) (xy 143.51 101.6))
     (stroke (width 0) (type default))
   )
-  (wire (pts (xy 115.57 114.3) (xy 115.57 151.13))
-    (stroke (width 0) (type default))
-  )
   (wire (pts (xy 85.09 74.93) (xy 102.87 74.93))
     (stroke (width 0) (type default))
   )
-  (wire (pts (xy 85.09 110.49) (xy 105.41 110.49))
-    (stroke (width 0) (type default))
-  )
   (wire (pts (xy 110.49 67.31) (xy 110.49 91.44))
     (stroke (width 0) (type default))
@@
     (stroke (width 0) (type default))
   )
-  (wire (pts (xy 85.09 69.85) (xy 107.95 69.85))
-    (stroke (width 0) (type default))
-  )
   (wire (pts (xy 85.09 67.31) (xy 110.49 67.31))
     (stroke (width 0) (type default))
   )
-  (wire (pts (xy 105.41 104.14) (xy 143.51 104.14))
-    (stroke (width 0) (type default))
-  )
   (wire (pts (xy 107.95 113.03) (xy 107.95 106.68))
     (stroke (width 0) (type default))
@@
     (stroke (width 0) (type default))
   )
-  (wire (pts (xy 107.95 93.98) (xy 143.51 93.98))
-    (stroke (width 0) (type default))
-  )
   (wire (pts (xy 137.16 86.36) (xy 143.51 86.36))
     (stroke (width 0) (type default))
@@
   )
   (wire (pts (xy 102.87 74.93) (xy 102.87 99.06))
-    (stroke (width 0) (type default))
-  )
-  (wire (pts (xy 105.41 110.49) (xy 105.41 104.14))
-    (stroke (width 0) (type default))
-  )
-  (wire (pts (xy 143.51 114.3) (xy 115.57 114.3))
     (stroke (width 0) (type default))
   )
@@
       (effects (font (size 1.27 1.27)) (justify right))
     )
-    (pin "V_SENSE" input (at 85.09 69.85 0)
-      (effects (font (size 1.27 1.27)) (justify right))
-    )
     (instances
       (project "IPB072N15N3G"
@@
       (effects (font (size 1.27 1.27)) (justify right))
     )
-    (pin "V_SENSE" input (at 85.09 151.13 0)
-      (effects (font (size 1.27 1.27)) (justify right))
-    )
     (instances
       (project "IPB072N15N3G"
@@
       (effects (font (size 1.27 1.27)) (justify right))
     )
-    (pin "V_SENSE" input (at 85.09 110.49 0)
-      (effects (font (size 1.27 1.27)) (justify right))
-    )
