File: MosfetBoard/IPB072N15N3G/IPB072N15N3G.kicad_pcb (KiCad board)
At the start: 2 copper layers, 155 x 100 mm, 97 parts, among them J1 DRIVER1, J13 BATT+Conn2, J14 BATT-Conn2, J15 PHASE_PAD, J16 PHASE_PAD, J2 DRIVER2, J3 DRIVER3, J4 PhaseConn1, J5 PhaseConn2, J6 PhaseConn3, J7 PHASE_PAD, J8 BATT+Conn1, J9 BATT-Conn1, Q1 IPB072N15N3G, Q10 IPB072N15N3G, Q11 IPB072N15N3G, Q12 IPB072N15N3G, Q2 IPB072N15N3G, Q3 IPB072N15N3G, Q4 IPB072N15N3G, Q5 IPB072N15N3G, Q6 IPB072N15N3G, Q7 IPB072N15N3G, Q8 IPB072N15N3G, Q9 IPB072N15N3G, U1 RS2166XC5, U2 ACS773ECB-200B-PFF-T, U3 ACS773ECB-200B-PFF-T, U5 RS2166XC5, U6 ACS773ECB-200B-PFF-T, U7 RS2166XC5

Commit message: cheap-mosfet-board
Parts:
- moved C29 147.3 mm to (168.5, 93.0)
- moved C39 142.9 mm to (121.0, 93.0)
- moved C44 138.5 mm to (73.5, 93.0)
- moved C34 46.9 mm to (168.5, 95.5), turned to 180 degrees
- moved C40 43.4 mm to (121.0, 95.5), turned to 180 degrees
- moved L1 41.2 mm to (171.5, 95.5), turned to -90 degrees
- moved C45 40.0 mm to (73.5, 95.5), turned to 180 degrees
- moved L2 37.9 mm to (124.0, 95.5), turned to -90 degrees
- moved L3 34.8 mm to (76.5, 95.5), turned to -90 degrees
- moved C1 34.2 mm to (197.0, 47.5), turned to -90 degrees
- moved C8 32.9 mm to (193.5, 47.5), turned to -90 degrees
- moved C25 32.6 mm to (149.5, 47.5), turned to -90 degrees
- moved C28 32.3 mm to (186.5, 47.5), turned to -90 degrees
- moved C50 32.2 mm to (190.0, 47.5), turned to -90 degrees
- moved C48 31.5 mm to (102.0, 47.5), turned to -90 degrees
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Connections:
- C29 pad 1: +3.3V -> 3.3V_1
- C36 pad 1: +3.3V -> 3.3V_1
- C39 pad 1: +3.3V -> 3.3V_2
- C42 pad 1: +3.3V -> 3.3V_2
- C44 pad 1: +3.3V -> 3.3V_3
- C47 pad 1: +3.3V -> 3.3V_3
- J4 pad 5: +3.3V -> 3.3V_1
- J5 pad 5: +3.3V -> 3.3V_2
- J6 pad 5: +3.3V -> 3.3V_3
- L1 pad 1: +3.3V -> 3.3V_1
- L2 pad 1: +3.3V -> 3.3V_2
- L3 pad 1: +3.3V -> 3.3V_3
- TH1 pad 1: +3.3V -> 3.3V_1
- TH2 pad 1: +3.3V -> 3.3V_2
- TH3 pad 1: +3.3V -> 3.3V_3
- U1 pad 5: +3.3V -> 3.3V_1
- U2 pad 4: PHASE2 -> B
- U2 pad 5: B -> PHASE2
- U3 pad 4: PHASE1 -> A
- U3 pad 5: A -> PHASE1
- U5 pad 5: +3.3V -> 3.3V_2
- U6 pad 4: PHASE3 -> C
- U6 pad 5: C -> PHASE3
- U7 pad 5: +3.3V -> 3.3V_3
Routing:
- net 3.3V_2: track 0.00 -> 122.7 mm, vias 0 -> 3
- net 3.3V_1: track 0.00 -> 122.0 mm, vias 0 -> 3
- net MOSTEMP2: track 0.00 -> 118.3 mm, vias 0 -> 2
- net MOSTEMP1: track 0.00 -> 118.3 mm, vias 0 -> 2
- net PH2: track 0.00 -> 114.9 mm, vias 0 -> 2
- net PH1: track 0.00 -> 114.9 mm, vias 0 -> 2
- net 3.3V_3: track 0.00 -> 70.3 mm, vias 0 -> 3
- net PH3: track 0.00 -> 59.4 mm, vias 0 -> 2
- net MOSTEMP3: track 0.00 -> 59.2 mm, vias 0 -> 2
- net -BATT: track 0.00 -> 57.2 mm, vias 0 -> 284
- net CURR2: track 0.00 -> 55.6 mm, vias 0 -> 2
- net CURR1: track 0.00 -> 54.9 mm, vias 0 -> 2
- net CURR3: track 0.00 -> 51.2 mm, vias 0 -> 2
- net VSENSE2: track 0.00 -> 32.0 mm, vias 0 -> 2
- net VSENSE1: track 0.00 -> 32.0 mm, vias 0 -> 2
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- added copper zone on B.Cu, net +BATT
- added copper zone on F.Cu, net Net-(C1-Pad2)
- added copper zone on F.Cu, net Net-(C10-Pad2)
- added copper zone on F.Cu, net Net-(C25-Pad2)
- added copper zone on F.Cu, net Net-(C26-Pad2)
- added copper zone on F.Cu, net Net-(C28-Pad2)
- added copper zone on F.Cu, net Net-(C31-Pad2)
- added copper zone on F.Cu, net Net-(C33-Pad2)
- added copper zone on F.Cu, net Net-(C4-Pad1)
- added copper zone on F.Cu, net Net-(C50-Pad2)
- added copper zone on F.Cu, net Net-(C52-Pad2)
- added copper zone on F.Cu, net Net-(C54-Pad2)
- added copper zone on F.Cu, net Net-(C8-Pad2)
- added copper zone on B.Cu, net PHASE1
- added copper zone on F.Cu, net PHASE1
- added copper zone on B.Cu, net PHASE2
- added copper zone on F.Cu, net PHASE2
- added copper zone on B.Cu, net PHASE3
Other:
- board size 155 x 100 mm -> 147 x 87 mm

Commit message: fixeddimensions
Parts:
- J2: value DRIVER2 -> DRIVER1
- J3: value DRIVER3 -> DRIVER1
- J4: value PhaseConn1 -> PhaseConn
- J5: value PhaseConn2 -> PhaseConn
- J6: value PhaseConn3 -> PhaseConn
- moved J6 1.06 mm to (110.2, 119.2), turned to -90 degrees
- moved J4 1.02 mm to (201.8, 119.2), turned to -90 degrees
- moved J5 0.29 mm to (156.0, 119.2), turned to -90 degrees
Connections:
- net 3.3V_1 renamed /PhaseMosfets1/3.3V_IN
- net 3.3V_2 renamed /PhaseMosfets2/3.3V_IN
- net 3.3V_3 renamed /PhaseMosfets3/3.3V_IN
- net A renamed /PhaseMosfets1/PHASE_OUT
- net B renamed /PhaseMosfets2/PHASE_OUT
- net C renamed /PhaseMosfets3/PHASE_OUT
- net CURR1 renamed /PhaseMosfets1/CURRENT_SENSE
- net CURR2 renamed /PhaseMosfets2/CURRENT_SENSE
- net CURR3 renamed /PhaseMosfets3/CURRENT_SENSE
- net MOSTEMP1 renamed /PhaseMosfets1/MOS_TEMP
- net MOSTEMP2 renamed /PhaseMosfets2/MOS_TEMP
- net MOSTEMP3 renamed /PhaseMosfets3/MOS_TEMP
- net PH1 renamed /PhaseMosfets1/PH
- net PH2 renamed /PhaseMosfets2/PH
- net PH3 renamed /PhaseMosfets3/PH
- net PHASE1 renamed /PhaseMosfets1/PHASE
- net PHASE2 renamed /PhaseMosfets2/PHASE
- net PHASE3 renamed /PhaseMosfets3/PHASE
- net PL1 renamed /PhaseMosfets1/PL
- net PL2 renamed /PhaseMosfets2/PL
- net PL3 renamed /PhaseMosfets3/PL
- net SENS_FILTER_ENABLE1 renamed /PhaseMosfets1/SENSE_FILTER_EN
- net SENS_FILTER_ENABLE2 renamed /PhaseMosfets2/SENSE_FILTER_EN
- net SENS_FILTER_ENABLE3 renamed /PhaseMosfets3/SENSE_FILTER_EN
- net VSENSE1 renamed /PhaseMosfets1/V_SENSE
- net VSENSE2 renamed /PhaseMosfets2/V_SENSE
- net VSENSE3 renamed /PhaseMosfets3/V_SENSE
Routing:
- net /PhaseMosfets1/3.3V_IN: track 122.0 -> 79.8 mm, vias 3 -> 2
- net /PhaseMosfets1/MOS_TEMP: track 118.3 -> 76.3 mm
- net /PhaseMosfets2/MOS_TEMP: track 118.3 -> 77.8 mm
- net /PhaseMosfets3/V_SENSE: track 32.0 -> 40.8 mm
- net /PhaseMosfets2/V_SENSE: track 32.0 -> 38.6 mm
- net /PhaseMosfets3/MOS_TEMP: track 59.2 -> 64.6 mm
- net /PhaseMosfets1/V_SENSE: track 32.0 -> 37.2 mm
- net /PhaseMosfets2/3.3V_IN: track 122.7 -> 118.1 mm, vias 3 -> 2
- net /PhaseMosfets3/3.3V_IN: track 70.3 -> 66.4 mm
- net /PhaseMosfets1/SENSE_FILTER_EN: track 14.1 -> 10.8 mm
- net /PhaseMosfets2/SENSE_FILTER_EN: track 14.8 -> 13.4 mm
- net /PhaseMosfets1/CURRENT_SENSE: track 54.9 -> 53.6 mm
- net /PhaseMosfets3/CURRENT_SENSE: track 51.2 -> 52.2 mm
Other:
- board size 147 x 87 mm -> 147 x 100 mm
- board text added: "Board Center X: 136.5 Y: 79 Size H: 100 W: 147"
- board text added: "Keepout 4mm"

Commit message: movedconnectors
Parts:
- moved J1 5.00 mm to (203.5, 63.0)
- moved J2 5.00 mm to (156.0, 63.0)
- moved J3 5.00 mm to (108.5, 63.0)
- moved R10 4.03 mm to (197.0, 66.0)
- moved R17 4.03 mm to (102.0, 66.0)
- moved R6 4.03 mm to (149.5, 66.0)
- moved J15 0.25 mm to (146.0, 99.2)
- moved J16 0.25 mm to (98.5, 99.2)
- moved J7 0.25 mm to (193.5, 99.2)
Routing:
- net /PhaseMosfets1/PL: track 28.4 -> 15.5 mm
- net /PhaseMosfets2/PL: track 28.4 -> 15.5 mm
- net /PhaseMosfets3/PH: track 59.4 -> 64.4 mm
- net /PhaseMosfets2/PH: track 114.9 -> 119.9 mm
- net /PhaseMosfets1/PH: track 114.9 -> 119.9 mm
- net Net-(Q6-G): track 6.91 -> 1.99 mm
- net Net-(Q2-G): track 6.91 -> 1.99 mm
- net /PhaseMosfets3/PHASE: track 16.8 -> 21.6 mm, vias 100 -> 102
- net /PhaseMosfets1/PHASE: track 28.3 -> 33.2 mm, vias 100 -> 102
- net /PhaseMosfets2/PHASE: track 28.3 -> 33.2 mm, vias 100 -> 102
- net Net-(Q10-G): track 3.45 -> 1.90 mm
- net /PhaseMosfets3/PL: track 16.0 -> 15.4 mm
- net -BATT: vias 284 -> 273
Other:
- board text added: "Designed by Kaminaris"
- board text added: "GigaESC MosfetBoard v1.0.0 - IPB072N15N3G"

Commit message: cleanup
Parts:
- removed J15, J16, J7: PHASE_PAD, Connector_Wire:SolderWirePad_1x01_SMD_5x10mm
Changed lines of the file:
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@@
     )
   )
-  (footprint "Connector_Wire:SolderWirePad_1x01_SMD_5x10mm" (layer "F.Cu")
-    (at 146 99.25 90)
-    (descr "Wire Pad, Square, SMD Pad,  5mm x 10mm,")
-    (tags "MesurementPoint Square SMDPad 5mmx10mm ")
-    (property "Sheetfile" "PhaseMosfets.kicad_sch")
-    (property "Sheetname" "PhaseMosfets2")
-    (property "ki_description" "Generic connector, single row, 01x01, script generated")
-    (property "ki_keywords" "connector")
-    (attr smd exclude_from_pos_files)
-    (fp_text reference "J15" (at 0 -3.81 90) (layer "F.SilkS") hide
-        (effects (font (size 1 1) (thickness 0.15)))
-    )
-    (fp_text value "PHASE_PAD" (at 0 6.35 90) (layer "F.Fab")
-        (effects (font (size 1 1) (thickness 0.15)))
-    )
-    (fp_text user "${REFERENCE}" (at 0 0 90) (layer "F.Fab")
-        (effects (font (size 1 1) (thickness 0.15)))
-    )
-    (fp_line (start -2.75 -5.25) (end -2.75 5.25)
-      (stroke (width 0.05) (type solid)) (layer "F.CrtYd"))
-    (fp_line (start -2.75 5.25) (end 2.75 5.25)
-      (stroke (width 0.05) (type solid)) (layer "F.CrtYd"))
-    (fp_line (start 2.75 -5.25) (end -2.75 -5.25)
-      (stroke (width 0.05) (type solid)) (layer "F.CrtYd"))
-    (fp_line (start 2.75 5.25) (end 2.75 -5.25)
-      (stroke (width 0.05) (type solid)) (layer "F.CrtYd"))
-    (pad "1" smd rect (at 0 0 90) (size 5 10) (layers "F.Cu" "F.Paste" "F.Mask")
-      (net 58 "/PhaseMosfets2/PHASE_OUT") (pinfunction "Pin_1") (pintype "passive"))
-  )
   (footprint "Resistor_SMD:R_0805_2012Metric" (layer "F.Cu")
     (at 102 66 180)
@@
     )
   )
-  (footprint "Connector_Wire:SolderWirePad_1x01_SMD_5x10mm" (layer "F.Cu")
-    (at 193.5 99.25 90)
-    (descr "Wire Pad, Square, SMD Pad,  5mm x 10mm,")
-    (tags "MesurementPoint Square SMDPad 5mmx10mm ")
-    (property "Sheetfile" "PhaseMosfets.kicad_sch")
-    (property "Sheetname" "PhaseMosfets1")
-    (property "ki_description" "Generic connector, single row, 01x01, script generated")
-    (property "ki_keywords" "connector")
-    (attr smd exclude_from_pos_files)
-    (fp_text reference "J7" (at 0 -3.81 90) (layer "F.SilkS") hide
-        (effects (font (size 1 1) (thickness 0.15)))
-    )
-    (fp_text value "PHASE_PAD" (at 0 6.35 90) (layer "F.Fab")
-        (effects (font (size 1 1) (thickness 0.15)))
-    )
-    (fp_text user "${REFERENCE}" (at 0 0 90) (layer "F.Fab")
-        (effects (font (size 1 1) (thickness 0.15)))
-    )
-    (fp_line (start -2.75 -5.25) (end -2.75 5.25)
-      (stroke (width 0.05) (type solid)) (layer "F.CrtYd"))
-    (fp_line (start -2.75 5.25) (end 2.75 5.25)
-      (stroke (width 0.05) (type solid)) (layer "F.CrtYd"))
-    (fp_line (start 2.75 -5.25) (end -2.75 -5.25)
-      (stroke (width 0.05) (type solid)) (layer "F.CrtYd"))
-    (fp_line (start 2.75 5.25) (end 2.75 -5.25)
-      (stroke (width 0.05) (type solid)) (layer "F.CrtYd"))
-    (pad "1" smd rect (at 0 0 90) (size 5 10) (layers "F.Cu" "F.Paste" "F.Mask")
-      (net 57 "/PhaseMosfets1/PHASE_OUT") (pinfunction "Pin_1") (pintype "passive"))
-  )
   (footprint "Resistor_SMD:R_0805_2012Metric" (layer "F.Cu")
     (at 70 81.5 -90)
@@
     )
   )
-  (footprint "Connector_Wire:SolderWirePad_1x01_SMD_5x10mm" (layer "F.Cu")
-    (at 98.5 99.25 90)
-    (descr "Wire Pad, Square, SMD Pad,  5mm x 10mm,")
-    (tags "MesurementPoint Square SMDPad 5mmx10mm ")
-    (property "Sheetfile" "PhaseMosfets.kicad_sch")
-    (property "Sheetname" "PhaseMosfets3")
-    (property "ki_description" "Generic connector, single row, 01x01, script generated")
-    (property "ki_keywords" "connector")
-    (attr smd exclude_from_pos_files)
-    (fp_text reference "J16" (at 0 -3.81 90) (layer "F.SilkS") hide
-        (effects (font (size 1 1) (thickness 0.15)))
-    )
-    (fp_text value "PHASE_PAD" (at 0 6.35 90) (layer "F.Fab")
-        (effects (font (size 1 1) (thickness 0.15)))
-    )
-    (fp_text user "${REFERENCE}" (at 0 0 90) (layer "F.Fab")
-        (effects (font (size 1 1) (thickness 0.15)))
-    )
-    (fp_line (start -2.75 -5.25) (end -2.75 5.25)
-      (stroke (width 0.05) (type solid)) (layer "F.CrtYd"))
-    (fp_line (start -2.75 5.25) (end 2.75 5.25)
-      (stroke (width 0.05) (type solid)) (layer "F.CrtYd"))
-    (fp_line (start 2.75 -5.25) (end -2.75 -5.25)
-      (stroke (width 0.05) (type solid)) (layer "F.CrtYd"))
-    (fp_line (start 2.75 5.25) (end 2.75 -5.25)
-      (stroke (width 0.05) (type solid)) (layer "F.CrtYd"))
-    (pad "1" smd rect (at 0 0 90) (size 5 10) (layers "F.Cu" "F.Paste" "F.Mask")
-      (net 59 "/PhaseMosfets3/PHASE_OUT") (pinfunction "Pin_1") (pintype "passive"))
-  )
   (footprint "Resistor_SMD:R_0805_2012Metric" (layer "F.Cu")
     (at 165 81.5 -90)
@@
   (gr_rect (start 114 56) (end 124 79)
     (stroke (width 0.15) (type solid)) (fill solid) (layer "B.Mask"))
-  (gr_rect (start 186.5 90.75) (end 199 102.25)
+  (gr_rect (start 186.5 90.75) (end 199 101.25)
     (stroke (width 0.15) (type solid)) (fill solid) (layer "F.Mask"))
-  (gr_rect (start 91.5 90.5) (end 104 102)
+  (gr_rect (start 91.5 90.5) (end 104 101)
     (stroke (width 0.15) (type solid)) (fill solid) (layer "F.Mask"))
   (gr_poly
@@
     )
     (stroke (width 0.15) (type solid)) (fill solid) (layer "F.Mask"))
-  (gr_rect (start 139 90.75) (end 151.5 102.25)
+  (gr_rect (start 139 90.75) (end 151.5 101.25)
     (stroke (width 0.15) (type solid)) (fill solid) (layer "F.Mask"))
   (gr_rect (start 63 103) (end 210 113)
@@
         (xy 139 90.75)
         (xy 151.5 90.75)
-        (xy 151.5 102.25)
-        (xy 139 102.25)
+        (xy 151.5 101.25)
+        (xy 139 101.25)
       )
     )
@@
         (xy 186.5 90.75)
         (xy 199 90.75)
-        (xy 199 102.25)
-        (xy 186.5 102.25)
+        (xy 199 101.25)
+        (xy 186.5 101.25)
       )
     )
@@
         (xy 91.5 90.5)
         (xy 104 90.5)
-        (xy 104 102)
-        (xy 91.5 102)
+        (xy 104 101)
+        (xy 91.5 101)
       )
     )

Commit message: fix
Parts:
- R1, R13, R14, R2, R20, R21: footprint Resistor_SMD:R_0805_2012Metric -> Resistor_SMD:R_0603_1608Metric
- R10, R11, R12, R16, R17, R18, R19, R5, R6, R7, R8, R9: value 2r2 -> 2.2
- moved R14 0.50 mm to (135.0, 98.0)
- moved R2 0.50 mm to (182.5, 98.0)
- moved R21 0.50 mm to (87.5, 98.0)

Commit message: v3.0.2 - IPB v2
Parts:
- removed C29, C35, C36, C39, C41, C42, C44, C46, C47: 100nF, Capacitor_SMD:C_0805_2012Metric
- removed C34, C40, C45: 2.2u, Capacitor_SMD:C_0805_2012Metric
- removed C37, C38, C43: 1u, Capacitor_SMD:C_0805_2012Metric
- removed J13: BATT+Conn2, Connector_Wire:SolderWirePad_1x01_SMD_5x10mm
- removed J14: BATT-Conn2, Connector_Wire:SolderWirePad_1x01_SMD_5x10mm
- removed J2, J3: DRIVER1, Connector_PinSocket_2.54mm:PinSocket_2x02_P2.54mm_Vertical_SMD
- removed J4, J5, J6: PhaseConn, Connector_PinSocket_2.54mm:PinSocket_2x03_P2.54mm_Vertical_SMD
- removed J8: BATT+Conn1, Connector_Wire:SolderWirePad_1x01_SMD_5x10mm
- removed J9: BATT-Conn1, Connector_Wire:SolderWirePad_1x01_SMD_5x10mm
- removed L1, L2, L3: BLM18HE152SN1D, Inductor_SMD:L_0603_1608Metric
- removed R13, R20: 150k, Resistor_SMD:R_0603_1608Metric
- removed R14, R21: 2.7k, Resistor_SMD:R_0603_1608Metric
- removed R15, R4: 10k, Resistor_SMD:R_0805_2012Metric
- removed U1, U5, U7: RS2166XC5, Package_TO_SOT_SMD:SOT-353_SC-70-5
- removed U2, U3, U6: ACS773ECB-200B-PFF-T, GigaVescLibs:Allegro_CB_SMD
- added C12: 100n, Capacitor_SMD:C_0603_1608Metric, F.Cu at (170.8, 90.2)
- added C13: 10n, Capacitor_SMD:C_0603_1608Metric, F.Cu at (170.8, 93.2)
- added C14: 1n, Capacitor_SMD:C_0603_1608Metric, F.Cu at (167.8, 93.2)
- added C15: 100n, Capacitor_SMD:C_0603_1608Metric, F.Cu at (137.5, 90.2)
- added C16: 10n, Capacitor_SMD:C_0603_1608Metric, F.Cu at (137.5, 93.2)
- added C17: 1n, Capacitor_SMD:C_0603_1608Metric, F.Cu at (134.5, 93.2)
- added C18: 1u, Capacitor_SMD:C_0603_1608Metric, F.Cu at (198.8, 84.8)
- added C19: 1u, Capacitor_SMD:C_0603_1608Metric, F.Cu at (165.5, 84.8)
- added C20: 1u, Capacitor_SMD:C_0603_1608Metric, F.Cu at (132.2, 84.8)
- added C5: 100n, Capacitor_SMD:C_0603_1608Metric, F.Cu at (204.0, 90.2)
- added C6: 10n, Capacitor_SMD:C_0603_1608Metric, F.Cu at (204.0, 93.2)
- added C7: 1n, Capacitor_SMD:C_0603_1608Metric, F.Cu at (201.0, 93.2)
- added H1: MountingHole_Pad, MountingHole:MountingHole_5.3mm_M5_Pad_Via, F.Cu at (200.5, 111.5)
- added H2: MountingHole_Pad, MountingHole:MountingHole_5.3mm_M5_Pad_Via, F.Cu at (167.2, 111.5)
- added H3: MountingHole_Pad, MountingHole:MountingHole_5.3mm_M5_Pad_Via, F.Cu at (134.0, 111.5)
- added H4: MountingHole_Pad, MountingHole:MountingHole_5.3mm_M5_Pad_Via, F.Cu at (112.0, 118.8)
- added H5: MountingHole_Pad, MountingHole:MountingHole_5.3mm_M5_Pad_Via, F.Cu at (112.0, 64.2)
- added H6: MountingHole, MountingHole:MountingHole_3.2mm_M3_ISO14580, F.Cu at (128.0, 61.0)
- added H7: MountingHole, MountingHole:MountingHole_3.2mm_M3_ISO14580, F.Cu at (184.0, 61.0)
- added H8: MountingHole, MountingHole:MountingHole_3.2mm_M3_ISO14580, F.Cu at (119.8, 113.8)
- added H9: MountingHole, MountingHole:MountingHole_3.2mm_M3_ISO14580, F.Cu at (192.2, 113.8)
- added R22: 0.3m, Resistor_SMD:R_2512_6332Metric, F.Cu at (197.8, 102.0)
- added R23: 4.7k, Resistor_SMD:R_0603_1608Metric, F.Cu at (201.0, 91.8)
- added R24: 9.1k, Resistor_SMD:R_0603_1608Metric, F.Cu at (204.0, 91.8)
- added R25: 0.3m, Resistor_SMD:R_2512_6332Metric, F.Cu at (164.5, 102.0)
- added R26: 4.7k, Resistor_SMD:R_0603_1608Metric, F.Cu at (167.8, 91.8)
- added R27: 9.1k, Resistor_SMD:R_0603_1608Metric, F.Cu at (170.8, 91.8)
- added R28: 0.3m, Resistor_SMD:R_2512_6332Metric, F.Cu at (131.2, 102.0)
- added R29: 4.7k, Resistor_SMD:R_0603_1608Metric, F.Cu at (134.5, 91.8)
- added R30: 9.1k, Resistor_SMD:R_0603_1608Metric, F.Cu at (137.5, 91.8)
- added R31: 150k, Resistor_SMD:R_0603_1608Metric, F.Cu at (198.0, 88.2)
- added R32: 2.7k, Resistor_SMD:R_0603_1608Metric, F.Cu at (201.2, 88.2)
- added R33: 150k, Resistor_SMD:R_0603_1608Metric, F.Cu at (164.8, 88.2)
- added R34: 2.7k, Resistor_SMD:R_0603_1608Metric, F.Cu at (168.0, 88.2)
- added R35: 150k, Resistor_SMD:R_0603_1608Metric, F.Cu at (131.5, 88.2)
- added R36: 2.7k, Resistor_SMD:R_0603_1608Metric, F.Cu at (134.8, 88.2)
- added U4: MT9223CT-50BR5, Package_SO:SOP-8_3.9x4.9mm_P1.27mm, F.Cu at (202.5, 97.8)
- added U8: MT9223CT-50BR5, Package_SO:SOP-8_3.9x4.9mm_P1.27mm, F.Cu at (169.2, 97.8)
- added U9: MT9223CT-50BR5, Package_SO:SOP-8_3.9x4.9mm_P1.27mm, F.Cu at (136.0, 97.8)
- J1: value DRIVER1 -> LogicConnector; footprint Connector_PinSocket_2.54mm:PinSocket_2x02_P2.54mm_Vertical_SMD -> Connector_PinSocket_2.54mm:PinSocket_2x15_P2.54mm_Vertical
- Q1, Q10, Q11, Q12, Q2, Q3, Q4, Q5, Q6, Q7, Q8, Q9: footprint GigaVescLibs:TO-263-3_TabPin2_NoLeg -> Package_TO_SOT_SMD:TO-263-2
- R1: value 150k -> 10k
- R10, R11, R12, R16, R17, R18, R19, R3, R5, R6, R7, R8, R9: footprint Resistor_SMD:R_0805_2012Metric -> Resistor_SMD:R_0603_1608Metric
- R2: value 2.7k -> 10k
- moved TH3 55.2 mm to (130.0, 85.5), turned to -90 degrees
- moved C49 54.0 mm to (136.8, 82.0), turned to 0 degrees
- moved C33 53.2 mm to (132.0, 82.0), turned to 0 degrees
- moved Q9 52.8 mm to (123.5, 77.0), turned to 90 degrees
- moved R16 49.9 mm to (119.0, 83.8), turned to -90 degrees
- moved C55 49.3 mm to (136.8, 78.8), turned to 0 degrees
- moved C54 48.4 mm to (132.0, 78.8), turned to 0 degrees
- moved Q10 47.6 mm to (123.5, 98.5), turned to 90 degrees
- moved C27 44.6 mm to (136.8, 75.5), turned to 0 degrees
- moved C26 43.7 mm to (132.0, 75.5), turned to 0 degrees
- moved C31 43.4 mm to (165.2, 82.0), turned to 0 degrees
- moved C32 42.8 mm to (170.0, 82.0), turned to 0 degrees
- moved R17 42.8 mm to (119.0, 105.2), turned to -90 degrees
- moved TH2 41.1 mm to (163.2, 85.5), turned to -90 degrees
- moved R10 40.9 mm to (185.5, 105.2), turned to -90 degrees
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Connections:
- J1 pad 1: /PhaseMosfets1/PH -> Net-(J1-Pin_1)
- J1 pad 2: /PhaseMosfets1/PL -> /3.3V
- J1 pad 3: /PhaseMosfets1/PHASE -> unconnected-(J1-Pin_3-Pad3)
- J1 pad 4: -BATT -> /5V
- Q1 pad 3: /PhaseMosfets1/PHASE -> /PHASE1
- Q10 pad 2: /PhaseMosfets3/PHASE -> /PHASE3
- Q11 pad 3: /PhaseMosfets3/PHASE -> /PHASE3
- Q12 pad 2: /PhaseMosfets3/PHASE -> /PHASE3
- Q2 pad 2: /PhaseMosfets1/PHASE -> /PHASE1
- Q3 pad 3: /PhaseMosfets1/PHASE -> /PHASE1
- Q4 pad 2: /PhaseMosfets1/PHASE -> /PHASE1
- Q5 pad 3: /PhaseMosfets2/PHASE -> /PHASE2
- Q6 pad 2: /PhaseMosfets2/PHASE -> /PHASE2
- Q7 pad 3: /PhaseMosfets2/PHASE -> /PHASE2
- Q8 pad 2: /PhaseMosfets2/PHASE -> /PHASE2
- Q9 pad 3: /PhaseMosfets3/PHASE -> /PHASE3
- R1 pad 1: /PhaseMosfets1/PHASE_OUT -> /PhaseMosfets1/MOS_TEMP
- R1 pad 2: /PhaseMosfets1/V_SENSE -> -BATT
- R10 pad 1: /PhaseMosfets1/PL -> /PL1
- R11 pad 1: /PhaseMosfets1/PH -> /PH1
- R12 pad 1: /PhaseMosfets1/PL -> /PL1
- R16 pad 1: /PhaseMosfets3/PH -> /PH3
- R17 pad 1: /PhaseMosfets3/PL -> /PL3
- R18 pad 1: /PhaseMosfets3/PH -> /PH3
- R19 pad 1: /PhaseMosfets3/PL -> /PL3
- R2 pad 1: /PhaseMosfets1/V_SENSE -> /PhaseMosfets2/MOS_TEMP
- R3 pad 1: /PhaseMosfets1/MOS_TEMP -> /PhaseMosfets3/MOS_TEMP
- R5 pad 1: /PhaseMosfets2/PH -> /PH2
- R6 pad 1: /PhaseMosfets2/PL -> /PL2
- R7 pad 1: /PhaseMosfets2/PH -> /PH2
- R8 pad 1: /PhaseMosfets2/PL -> /PL2
- R9 pad 1: /PhaseMosfets1/PH -> /PH1
- TH1 pad 1: /PhaseMosfets1/3.3V_IN -> /3.3V
- TH2 pad 1: /PhaseMosfets2/3.3V_IN -> /3.3V
- TH3 pad 1: /PhaseMosfets3/3.3V_IN -> /3.3V
Routing:
- net /5V: track 0.00 -> 193.8 mm, vias 0 -> 5
- net /3.3V: track 0.00 -> 139.6 mm, vias 0 -> 6
- net /PhaseMosfets2/PH: track 119.9 -> 0.00 mm, vias 2 -> 0
- net /PhaseMosfets1/PH: track 119.9 -> 0.00 mm, vias 2 -> 0
- net /PhaseMosfets2/3.3V_IN: track 118.0 -> 0.00 mm, vias 2 -> 0
- net /PL2: track 0.00 -> 84.2 mm, vias 0 -> 3
- net /PL3: track 0.00 -> 80.7 mm, vias 0 -> 4
- net /PhaseMosfets1/3.3V_IN: track 79.8 -> 0.00 mm, vias 2 -> 0
- net /PhaseMosfets1/SH-: track 0.00 -> 73.9 mm, vias 0 -> 1
- net /PH1: track 0.00 -> 73.1 mm, vias 0 -> 1
- net /PhaseMosfets1/SH+: track 0.00 -> 68.1 mm, vias 0 -> 1
- net /PL1: track 0.00 -> 67.6 mm, vias 0 -> 1
- net /PhaseMosfets3/3.3V_IN: track 66.2 -> 0.00 mm, vias 3 -> 0
- net /PhaseMosfets3/PH: track 64.4 -> 0.00 mm, vias 2 -> 0
- net /PH3: track 0.00 -> 61.6 mm, vias 0 -> 3
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- added copper zone on F.Cu, net /PHASE1
- added copper zone on F.Cu, net /PHASE2
- added copper zone on F.Cu, net /PHASE3
- removed copper zone on B.Cu, net +BATT
- removed copper zone on B.Cu, net /PhaseMosfets1/PHASE
- removed copper zone on F.Cu, net /PhaseMosfets1/PHASE
- removed copper zone on B.Cu, net /PhaseMosfets2/PHASE
- removed copper zone on F.Cu, net /PhaseMosfets2/PHASE
- removed copper zone on B.Cu, net /PhaseMosfets3/PHASE
- removed copper zone on F.Cu, net /PhaseMosfets3/PHASE
- removed copper zone on F.Cu, net Net-(C1-Pad2)
- removed copper zone on F.Cu, net Net-(C10-Pad2)
- removed copper zone on F.Cu, net Net-(C25-Pad2)
- removed copper zone on F.Cu, net Net-(C26-Pad2)
- removed copper zone on F.Cu, net Net-(C28-Pad2)
- removed copper zone on F.Cu, net Net-(C31-Pad2)
- removed copper zone on F.Cu, net Net-(C33-Pad2)
- removed copper zone on F.Cu, net Net-(C4-Pad1)
- removed copper zone on F.Cu, net Net-(C50-Pad2)
- removed copper zone on F.Cu, net Net-(C52-Pad2)
- removed copper zone on F.Cu, net Net-(C54-Pad2)
- removed copper zone on F.Cu, net Net-(C8-Pad2)
Other:
- board size 147 x 100 mm -> 100 x 75 mm
- board text added: "GigaESC MosfetBoard v2.0.0 - IPB072N15N3G Designed by Kaminaris"
- board text removed: "Designed by Kaminaris"
- board text removed: "GigaESC MosfetBoard v1.0.0 - IPB072N15N3G"

Commit message: v3.0.2 - Prerelease
Parts:
- removed R31, R33, R35: 150k, Resistor_SMD:R_0603_1608Metric
- removed R32, R34, R36: 2.7k, Resistor_SMD:R_0603_1608Metric
- moved C12 3.00 mm to (170.8, 87.2)
- moved C13 3.00 mm to (170.8, 90.2)
- moved C14 3.00 mm to (167.8, 90.2)
- moved C15 3.00 mm to (137.5, 87.2)
- moved C16 3.00 mm to (137.5, 90.2)
- moved C17 3.00 mm to (134.5, 90.2)
- moved C5 3.00 mm to (204.0, 87.2)
- moved C6 3.00 mm to (204.0, 90.2)
- moved C7 3.00 mm to (201.0, 90.2)
- moved R23 3.00 mm to (201.0, 88.8)
- moved R24 3.00 mm to (204.0, 88.8)
- moved R26 3.00 mm to (167.8, 88.8)
- moved R27 3.00 mm to (170.8, 88.8)
- moved R29 3.00 mm to (134.5, 88.8)
- moved R30 3.00 mm to (137.5, 88.8)
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Connections:
- J1 pad 15: /PhaseMosfets2/V_SENSE -> unconnected-(J1-Pin_15-Pad15)
- J1 pad 23: /PhaseMosfets3/V_SENSE -> unconnected-(J1-Pin_23-Pad23)
- J1 pad 7: /PhaseMosfets1/V_SENSE -> unconnected-(J1-Pin_7-Pad7)
Routing:
- net /PhaseMosfets1/V_SENSE: track 56.8 -> 0.00 mm, vias 2 -> 0
- net /PhaseMosfets2/V_SENSE: track 37.8 -> 0.00 mm, vias 1 -> 0
- net /PhaseMosfets3/V_SENSE: track 36.5 -> 0.00 mm, vias 1 -> 0
- net /5V: track 193.8 -> 181.4 mm
- net -BATT: track 61.3 -> 51.3 mm, vias 75 -> 72
- net /PHASE2: track 43.7 -> 39.9 mm, vias 1 -> 41
- net /PHASE3: track 43.8 -> 40.3 mm, vias 2 -> 42
- net /PhaseMosfets1/SH+: track 68.1 -> 65.4 mm
- net /PhaseMosfets3/SH+: track 35.4 -> 33.4 mm
- net /PhaseMosfets2/SH+: track 42.7 -> 41.1 mm
- net /PhaseMosfets2/MOS_TEMP: track 37.1 -> 35.7 mm
- net /PL2: track 84.2 -> 85.7 mm
- net /PhaseMosfets1/SH-: track 73.9 -> 75.2 mm
- net /PhaseMosfets3/MOS_TEMP: track 37.9 -> 38.7 mm
- net /PhaseMosfets1/MOS_TEMP: track 49.9 -> 50.4 mm
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- added copper zone on B.Cu, net +BATT
- added copper zone on B.Cu, net /PHASE1
- added copper zone on B.Cu, net /PHASE2
- added copper zone on B.Cu, net /PHASE3
Other:
- board text added: "GigaESC MosfetBoard v2.0.1 - IPB072N15N3G Designed by Kaminaris"
- board text removed: "GigaESC MosfetBoard v2.0.0 - IPB072N15N3G Designed by Kaminaris"
