File: MosfetBoard/IXTT220N20X4HV/IXTT220N20X4HV.kicad_pcb (KiCad board)
At the start: 2 copper layers, 155 x 100 mm, 108 parts, among them J1 DRIVER1, J10 A_PAD, J11 B_PAD, J12 C_PAD, J13 BATT+Conn2, J14 BATT-Conn2, J15 AuxConn, J2 DRIVER2, J3 DRIVER3, J4 PhaseConn1, J5 PhaseConn2, J6 PhaseConn3, J7 VINConn, J8 BATT+Conn1, J9 BATT-Conn1, Q1 IXTT220N20X4HV, Q10 IXTT220N20X4HV, Q11 IXTT220N20X4HV, Q12 IXTT220N20X4HV, Q13 NTMTSC4D3N15MC, Q2 IXTT220N20X4HV, Q3 IXTT220N20X4HV, Q4 IXTT220N20X4HV, Q5 IXTT220N20X4HV, Q6 IXTT220N20X4HV, Q7 IXTT220N20X4HV, Q8 IXTT220N20X4HV, Q9 IXTT220N20X4HV, U1 RS2166XC5, U2 ACS773ECB-200B-PFF-T, U3 ACS773ECB-200B-PFF-T, U4 RDE20110S12, U5 RS2166XC5, U6 ACS773ECB-200B-PFF-T, U7 RS2166XC5

Commit message: cheap_board
Parts:
- removed C25, C26, C27, C28, C30, C31: 680uF 200V, Capacitor_THT:CP_Radial_D22.0mm_P10.00mm_SnapIn
- removed J15: AuxConn, Connector_PinSocket_2.54mm:PinSocket_1x05_P2.54mm_Vertical_SMD_Pin1Left
- removed J7: VINConn, Connector_PinSocket_2.54mm:PinSocket_1x04_P2.54mm_Vertical_SMD_Pin1Left
- removed Q13: NTMTSC4D3N15MC, Package_TO_SOT_SMD:PQFN_8x8
- removed U4: RDE20110S12, Converter_DCDC:Converter_DCDC_TRACO_THN30-xxxx_THT

Commit message: wholeDevice
Parts:
- removed J12: C_PAD, Connector_Wire:SolderWirePad_1x01_SMD_5x10mm
- removed REF**: LogicBoard, GigaVescLibs:LogicBoard
- added C25: 10u 100V, Capacitor_SMD:C_1210_3225Metric, F.Cu at (207.5, 80.0)
- added C26: 10u 100V, Capacitor_SMD:C_1210_3225Metric, F.Cu at (202.8, 80.0)
- added C27: 10u 100V, Capacitor_SMD:C_1210_3225Metric, F.Cu at (207.5, 83.2)
- added C28: 10u 100V, Capacitor_SMD:C_1210_3225Metric, F.Cu at (202.8, 83.2)
- added C30: 10u 100V, Capacitor_SMD:C_1210_3225Metric, F.Cu at (207.5, 86.5)
- added C31: 10u 100V, Capacitor_SMD:C_1210_3225Metric, F.Cu at (202.8, 86.5)
- added C32: 10u 100V, Capacitor_SMD:C_1210_3225Metric, F.Cu at (207.5, 89.8)
- added C33: 10u 100V, Capacitor_SMD:C_1210_3225Metric, F.Cu at (202.8, 89.8)
- added C48: 10u 100V, Capacitor_SMD:C_1210_3225Metric, F.Cu at (160.0, 80.0)
- added C49: 10u 100V, Capacitor_SMD:C_1210_3225Metric, F.Cu at (155.2, 80.0)
- added C50: 10u 100V, Capacitor_SMD:C_1210_3225Metric, F.Cu at (160.0, 83.2)
- added C51: 10u 100V, Capacitor_SMD:C_1210_3225Metric, F.Cu at (155.2, 83.2)
- added C52: 10u 100V, Capacitor_SMD:C_1210_3225Metric, F.Cu at (160.0, 86.5)
- added C53: 10u 100V, Capacitor_SMD:C_1210_3225Metric, F.Cu at (155.2, 86.5)
- added C54: 10u 100V, Capacitor_SMD:C_1210_3225Metric, F.Cu at (160.0, 89.8)
- added C55: 10u 100V, Capacitor_SMD:C_1210_3225Metric, F.Cu at (155.2, 89.8)
- added C56: 10u 100V, Capacitor_SMD:C_1210_3225Metric, F.Cu at (112.5, 80.0)
- added C57: 10u 100V, Capacitor_SMD:C_1210_3225Metric, F.Cu at (107.8, 80.0)
- added C58: 10u 100V, Capacitor_SMD:C_1210_3225Metric, F.Cu at (112.5, 83.2)
- added C59: 10u 100V, Capacitor_SMD:C_1210_3225Metric, F.Cu at (107.8, 83.2)
- added C60: 10u 100V, Capacitor_SMD:C_1210_3225Metric, F.Cu at (112.5, 86.5)
- added C61: 10u 100V, Capacitor_SMD:C_1210_3225Metric, F.Cu at (107.8, 86.5)
- added C62: 10u 100V, Capacitor_SMD:C_1210_3225Metric, F.Cu at (112.5, 89.8)
- added C63: 10u 100V, Capacitor_SMD:C_1210_3225Metric, F.Cu at (107.8, 89.8)
- added J7: PhasePad, Connector_Wire:SolderWirePad_1x01_SMD_5x10mm, F.Cu at (178.8, 116.5)
- C1, C10, C11, C12, C13, C14, C15, C16, C17, C18, C19, C2, C20, C21, C22, C23, C24, C3, C4, C5, C6, C7, C8, C9: value C -> 10u 100V; footprint Capacitor_SMD:C_2220_5650Metric -> Capacitor_SMD:C_1210_3225Metric
- C29, C35, C36, C39, C41, C42, C44, C46, C47: value 100nF -> 100n; footprint Capacitor_SMD:C_0805_2012Metric -> GigaVescLibs:C_0603_1608Metric_L
- C34, C37, C38, C40, C43, C45: footprint Capacitor_SMD:C_0805_2012Metric -> GigaVescLibs:C_0603_1608Metric_L
- J10: value A_PAD -> PhasePad
- J11: value B_PAD -> PhasePad
- J2: value DRIVER2 -> DRIVER1
- J3: value DRIVER3 -> DRIVER1
- J4: value PhaseConn1 -> PhaseConn
- J5: value PhaseConn2 -> PhaseConn
- J6: value PhaseConn3 -> PhaseConn
- R1, R13, R14, R15, R2, R20, R21, R3, R4: footprint Resistor_SMD:R_0805_2012Metric -> Resistor_SMD:R_0603_1608Metric
- R10, R11, R12, R16, R17, R18, R19, R5, R6, R7, R8, R9: value 2r2 -> 2.2
- moved C44 116.3 mm to (93.2, 120.2)
- moved C18 107.8 mm to (107.8, 67.0)
- moved C24 98.9 mm to (107.8, 76.8)
- moved C4 97.9 mm to (202.8, 70.2)
- moved J9 91.3 mm to (211.8, 119.5)
- moved J14 89.8 mm to (64.0, 119.5)
- moved C29 85.7 mm to (188.2, 120.2), turned to 180 degrees
- moved C13 57.3 mm to (160.0, 73.5)
- moved C11 56.2 mm to (160.0, 70.2)
- moved C22 55.9 mm to (107.8, 73.5)
- moved C7 54.8 mm to (207.5, 76.8)
- moved C14 54.7 mm to (155.2, 73.5)
- moved J10 54.3 mm to (131.2, 116.5)
- moved J11 50.8 mm to (83.8, 116.5)
- moved C5 49.0 mm to (207.5, 73.5)
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Connections:
- net CURR1 renamed /PhaseMosfets1/CURRENT_SENSE
- net CURR2 renamed /PhaseMosfets2/CURRENT_SENSE
- net CURR3 renamed /PhaseMosfets3/CURRENT_SENSE
- net MOSTEMP1 renamed /PhaseMosfets1/MOS_TEMP
- net MOSTEMP2 renamed /PhaseMosfets2/MOS_TEMP
- net MOSTEMP3 renamed /PhaseMosfets3/MOS_TEMP
- net PH1 renamed /PhaseMosfets1/PH
- net PH2 renamed /PhaseMosfets2/PH
- net PH3 renamed /PhaseMosfets3/PH
- net PHASE1 renamed /PhaseMosfets1/PHASE
- net PHASE2 renamed /PhaseMosfets2/PHASE
- net PHASE3 renamed /PhaseMosfets3/PHASE
- net PL1 renamed /PhaseMosfets1/PL
- net PL2 renamed /PhaseMosfets2/PL
- net PL3 renamed /PhaseMosfets3/PL
- net SENS_FILTER_ENABLE1 renamed /PhaseMosfets1/SENSE_FILTER_EN
- net SENS_FILTER_ENABLE2 renamed /PhaseMosfets2/SENSE_FILTER_EN
- net SENS_FILTER_ENABLE3 renamed /PhaseMosfets3/SENSE_FILTER_EN
- net VSENSE1 renamed /PhaseMosfets1/V_SENSE
- net VSENSE2 renamed /PhaseMosfets2/V_SENSE
- net VSENSE3 renamed /PhaseMosfets3/V_SENSE
- C10 pad 1: +BATT -> Net-(C10-Pad1)
- C10 pad 2: Net-(C10-Pad2) -> -BATT
- C11 pad 1: Net-(C10-Pad2) -> +BATT
- C11 pad 2: -BATT -> Net-(C11-Pad2)
- C12 pad 1: Net-(C12-Pad1) -> Net-(C11-Pad2)
- C18 pad 1: +BATT -> Net-(C17-Pad2)
- C18 pad 2: Net-(C18-Pad2) -> -BATT
- C21 pad 1: Net-(C17-Pad2) -> +BATT
- C21 pad 2: -BATT -> Net-(C21-Pad2)
- C22 pad 1: +BATT -> Net-(C21-Pad2)
- C22 pad 2: Net-(C22-Pad2) -> -BATT
- C23 pad 1: Net-(C22-Pad2) -> +BATT
- C23 pad 2: -BATT -> Net-(C23-Pad2)
- C24 pad 1: Net-(C18-Pad2) -> Net-(C23-Pad2)
- C29 pad 1: +3.3V -> /PhaseMosfets1/3.3V_IN
- C3 pad 1: Net-(C3-Pad1) -> +BATT
- C3 pad 2: -BATT -> Net-(C3-Pad2)
- C36 pad 1: +3.3V -> /PhaseMosfets1/3.3V_IN
- C39 pad 1: +3.3V -> /PhaseMosfets2/3.3V_IN
- C4 pad 1: Net-(C4-Pad1) -> Net-(C3-Pad2)
- C42 pad 1: +3.3V -> /PhaseMosfets2/3.3V_IN
- C44 pad 1: +3.3V -> /PhaseMosfets3/3.3V_IN
- C47 pad 1: +3.3V -> /PhaseMosfets3/3.3V_IN
- C6 pad 1: +BATT -> Net-(C5-Pad2)
- C6 pad 2: Net-(C12-Pad1) -> -BATT
- C7 pad 1: Net-(C5-Pad2) -> +BATT
- C7 pad 2: -BATT -> Net-(C7-Pad2)
- C8 pad 1: +BATT -> Net-(C7-Pad2)
- C8 pad 2: Net-(C3-Pad1) -> -BATT
- C9 pad 2: Net-(C4-Pad1) -> Net-(C10-Pad1)
- J10 pad 1: A -> /PhaseMosfets2/PHASE_OUT
- J11 pad 1: B -> /PhaseMosfets3/PHASE_OUT
- J4 pad 5: +3.3V -> /PhaseMosfets1/3.3V_IN
- J5 pad 5: +3.3V -> /PhaseMosfets2/3.3V_IN
- J6 pad 5: +3.3V -> /PhaseMosfets3/3.3V_IN
- L1 pad 1: +3.3V -> /PhaseMosfets1/3.3V_IN
- L2 pad 1: +3.3V -> /PhaseMosfets2/3.3V_IN
- L3 pad 1: +3.3V -> /PhaseMosfets3/3.3V_IN
- R1 pad 1: A -> /PhaseMosfets1/PHASE_OUT
- R13 pad 1: B -> /PhaseMosfets2/PHASE_OUT
- R20 pad 1: C -> /PhaseMosfets3/PHASE_OUT
- TH1 pad 1: +3.3V -> /PhaseMosfets1/3.3V_IN
- TH2 pad 1: +3.3V -> /PhaseMosfets2/3.3V_IN
- TH3 pad 1: +3.3V -> /PhaseMosfets3/3.3V_IN
- U1 pad 5: +3.3V -> /PhaseMosfets1/3.3V_IN
- U2 pad 5: B -> /PhaseMosfets2/PHASE_OUT
- U3 pad 5: A -> /PhaseMosfets1/PHASE_OUT
- U5 pad 5: +3.3V -> /PhaseMosfets2/3.3V_IN
- U6 pad 5: C -> /PhaseMosfets3/PHASE_OUT
- U7 pad 5: +3.3V -> /PhaseMosfets3/3.3V_IN
Routing:
- net +3.3V: track 71.1 -> 0.00 mm
- net -BATT: track 2.92 -> 46.9 mm, vias 52 -> 203
- net /PhaseMosfets2/PH: track 0.00 -> 39.5 mm
- net /PhaseMosfets3/3.3V_IN: track 0.00 -> 39.3 mm
- net /PhaseMosfets2/3.3V_IN: track 0.00 -> 37.6 mm
- net /PhaseMosfets1/3.3V_IN: track 0.00 -> 35.8 mm
- net /PhaseMosfets3/MOS_TEMP: track 2.02 -> 35.3 mm
- net /PhaseMosfets1/MOS_TEMP: track 0.00 -> 31.6 mm
- net /PhaseMosfets3/V_SENSE: track 2.02 -> 27.8 mm, vias 0 -> 2
- net Net-(U3-VCC): track 0.00 -> 24.7 mm, vias 0 -> 2
- net /PhaseMosfets1/CURRENT_SENSE: track 0.00 -> 24.2 mm
- net /PhaseMosfets1/V_SENSE: track 0.00 -> 23.9 mm, vias 0 -> 2
- net /PhaseMosfets3/CURRENT_SENSE: track 0.00 -> 21.0 mm
- net Net-(U2-VCC): track 4.62 -> 24.4 mm, vias 0 -> 2
- net /PhaseMosfets3/SENSE_FILTER_EN: track 0.00 -> 19.0 mm, vias 0 -> 2
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- added copper zone on B.Cu, net +BATT
- added copper zone on B.Cu, net /PhaseMosfets1/PHASE
- added copper zone on F.Cu, net /PhaseMosfets1/PHASE_OUT
- added copper zone on B.Cu, net /PhaseMosfets2/PHASE
- added copper zone on F.Cu, net /PhaseMosfets2/PHASE_OUT
- added copper zone on B.Cu, net /PhaseMosfets3/PHASE
- added copper zone on F.Cu, net /PhaseMosfets3/PHASE_OUT
- added copper zone on F.Cu, net Net-(C1-Pad2)
- added copper zone on F.Cu, net Net-(C10-Pad1)
- added copper zone on F.Cu, net Net-(C11-Pad2)
- added copper zone on F.Cu, net Net-(C13-Pad2)
- added copper zone on F.Cu, net Net-(C15-Pad2)
- added copper zone on F.Cu, net Net-(C17-Pad2)
- added copper zone on F.Cu, net Net-(C19-Pad2)
- added copper zone on F.Cu, net Net-(C21-Pad2)
- added copper zone on F.Cu, net Net-(C23-Pad2)
- added copper zone on F.Cu, net Net-(C25-Pad2)
- added copper zone on F.Cu, net Net-(C27-Pad2)
- added copper zone on F.Cu, net Net-(C3-Pad2)
- added copper zone on F.Cu, net Net-(C30-Pad2)
- added copper zone on F.Cu, net Net-(C32-Pad2)
- added copper zone on F.Cu, net Net-(C48-Pad2)
- added copper zone on F.Cu, net Net-(C5-Pad2)
- added copper zone on F.Cu, net Net-(C50-Pad2)
- added copper zone on F.Cu, net Net-(C52-Pad2)
- added copper zone on F.Cu, net Net-(C54-Pad2)
- added copper zone on F.Cu, net Net-(C56-Pad2)
- added copper zone on F.Cu, net Net-(C58-Pad2)
- added copper zone on F.Cu, net Net-(C60-Pad2)
- added copper zone on F.Cu, net Net-(C62-Pad2)
- added copper zone on F.Cu, net Net-(C7-Pad2)
- removed copper zone on F.Cu, net A
- removed copper zone on F.Cu, net B
- removed copper zone on F.Cu, net C

Commit message: fixeddimensions
Other:
- board text added: "Center X: 137.5 Y: 80"
- board text added: "Designed by Kaminaris"
- board text added: "GigaESC MosfetBoard v1.0.0 - IXTT220N20X4HV"
Changed lines of the file:
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@@
       (xy 84.5 54)
       (xy 84.5 60.5)
-      (xy 84.5 60.5)
       (xy 90.25 60.5)
     )
     (stroke (width 0.15) (type solid)) (fill solid) (layer "B.Mask"))
-  (gr_rect (start 60 33) (end 215 51)
+  (gr_rect (start 60 34) (end 215 51)
     (stroke (width 0.15) (type solid)) (fill solid) (layer "B.Mask"))
   (gr_poly
@@
       (xy 132 54)
       (xy 132 60.5)
-      (xy 132 60.5)
       (xy 137.75 60.5)
     )
@@
       (xy 179.5 54)
       (xy 179.5 60.5)
-      (xy 179.5 60.5)
       (xy 185.25 60.5)
     )
     (stroke (width 0.15) (type solid)) (fill solid) (layer "B.Mask"))
-  (gr_rect (start 60 110) (end 69 127)
+  (gr_rect (start 60 110) (end 69 126)
     (stroke (width 0.15) (type solid)) (fill solid) (layer "F.Mask"))
   (gr_poly
@@
       (xy 132 54)
       (xy 132 60.5)
-      (xy 132 60.5)
       (xy 137.75 60.5)
     )
     (stroke (width 0.15) (type solid)) (fill solid) (layer "F.Mask"))
-  (gr_rect (start 208 111) (end 215 127)
+  (gr_rect (start 208 111) (end 215 126)
     (stroke (width 0.15) (type solid)) (fill solid) (layer "F.Mask"))
   (gr_poly
@@
     )
     (stroke (width 0.15) (type solid)) (fill solid) (layer "F.Mask"))
-  (gr_rect (start 60 33) (end 215 51)
+  (gr_rect (start 60 34) (end 215 51)
     (stroke (width 0.15) (type solid)) (fill solid) (layer "F.Mask"))
   (gr_poly
@@
       (xy 179.5 54)
       (xy 179.5 60.5)
-      (xy 179.5 60.5)
       (xy 185.25 60.5)
     )
@@
       (xy 84.5 54)
       (xy 84.5 60.5)
-      (xy 84.5 60.5)
       (xy 90.25 60.5)
     )
@@
   (gr_line (start 70.75 106.25) (end 229 106.25)
     (stroke (width 0.15) (type default)) (layer "User.7"))
+  (gr_text "GigaESC MosfetBoard\nv1.0.0 - IXTT220N20X4HV" (at 64.75 86.25 90) (layer "F.SilkS")
+    (effects (font (size 1 1) (thickness 0.15)) (justify bottom))
+  )
+  (gr_text "Designed by Kaminaris" (at 69 109 90) (layer "F.SilkS")
+    (effects (font (size 1 1) (thickness 0.15)) (justify left bottom))
+  )
+  (gr_text "Center\nX: 137.5\nY: 80" (at 45.5 21.5) (layer "User.6")
+    (effects (font (size 1 1) (thickness 0.15)) (justify left bottom))
+  )
   (dimension (type aligned) (layer "User.1")
     (pts (xy 218 130) (xy 218 30))
@@
   )
   (dimension (type aligned) (layer "User.6")
+    (pts (xy 215 130) (xy 215 126))
+    (height 3.25)
+    (gr_text "4.0000 mm" (at 217.1 128 90) (layer "User.6")
+      (effects (font (size 1 1) (thickness 0.15)))
+    )
+    (format (prefix "") (suffix "") (units 3) (units_format 1) (precision 4))
+    (style (thickness 0.15) (arrow_length 1.27) (text_position_mode 0) (extension_height 0.58642) (extension_offset 0.5) keep_text_aligned)
+  )
+  (dimension (type aligned) (layer "User.6")
     (pts (xy 114.6 123.75) (xy 151.7 123.75))
     (height 8.16)
@@
   )
   (dimension (type aligned) (layer "User.6")
-    (pts (xy 218 30) (xy 218 33))
+    (pts (xy 60 130) (xy 60 126))
     (height -3.25)
-    (gr_text "3.0000 mm" (at 220.1 31.5 90) (layer "User.6")
+    (gr_text "4.0000 mm" (at 55.6 128 90) (layer "User.6")
+      (effects (font (size 1 1) (thickness 0.15)))
+    )
+    (format (prefix "") (suffix "") (units 3) (units_format 1) (precision 4))
+    (style (thickness 0.15) (arrow_length 1.27) (text_position_mode 0) (extension_height 0.58642) (extension_offset 0.5) keep_text_aligned)
+  )
+  (dimension (type aligned) (layer "User.6")
+    (pts (xy 215 30) (xy 215 34))
+    (height -3.25)
+    (gr_text "4.0000 mm" (at 217.1 32 90) (layer "User.6")
       (effects (font (size 1 1) (thickness 0.15)))
     )
@@
   )
   (dimension (type aligned) (layer "User.6")
-    (pts (xy 63 30) (xy 63 33))
+    (pts (xy 60 30) (xy 60 34))
     (height 3.25)
-    (gr_text "3.0000 mm" (at 58.6 31.5 90) (layer "User.6")
+    (gr_text "4.0000 mm" (at 55.6 32 90) (layer "User.6")
       (effects (font (size 1 1) (thickness 0.15)))
     )
@@
       (pts
         (xy 60 30)
-        (xy 60 33)
-        (xy 215 33)
+        (xy 60 34)
+        (xy 215 34)
         (xy 215 30)
       )
@@
         (xy 84.5 54)
         (xy 84.5 60.5)
-        (xy 84.5 60.5)
         (xy 90.25 60.5)
       )
@@
     (polygon
       (pts
-        (xy 60 127)
+        (xy 60 126)
         (xy 60 130)
         (xy 215 130)
-        (xy 215 127)
+        (xy 215 126)
       )
     )
@@
     (polygon
       (pts
-        (xy 60 30)
+        (xy 60 34)
         (xy 60 51)
         (xy 215 51)
-        (xy 215 30)
+        (xy 215 34)
       )
     )
@@
         (xy 132 54)
         (xy 132 60.5)
-        (xy 132 60.5)
         (xy 137.75 60.5)
       )
@@
         (xy 179.500856 54)
         (xy 179.500856 60.5)
-        (xy 179.500856 60.5)
         (xy 185.250856 60.5)

Commit message: movedconnectors
Parts:
- moved C1 5.00 mm to (207.5, 72.0)
- moved C10 5.00 mm to (155.2, 72.0)
- moved C11 5.00 mm to (160.0, 75.2)
- moved C12 5.00 mm to (155.2, 75.2)
- moved C13 5.00 mm to (160.0, 78.5)
- moved C14 5.00 mm to (155.2, 78.5)
- moved C15 5.00 mm to (160.0, 81.8)
- moved C16 5.00 mm to (155.2, 81.8)
- moved C17 5.00 mm to (112.5, 72.0)
- moved C18 5.00 mm to (107.8, 72.0)
- moved C19 5.00 mm to (112.5, 75.2)
- moved C2 5.00 mm to (202.8, 72.0)
- moved C20 5.00 mm to (107.8, 75.2)
- moved C21 5.00 mm to (112.5, 78.5)
- moved C22 5.00 mm to (107.8, 78.5)
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Routing:
- net /PhaseMosfets3/PH: track 39.5 -> 44.5 mm
- net /PhaseMosfets2/PH: track 39.5 -> 44.5 mm
- net /PhaseMosfets1/PH: track 39.5 -> 44.5 mm
- net /PhaseMosfets2/PHASE: track 13.7 -> 15.7 mm
- net /PhaseMosfets1/PHASE: track 13.7 -> 15.5 mm
- net /PhaseMosfets3/PHASE: track 13.7 -> 15.2 mm
- net /PhaseMosfets1/PL: track 42.0 -> 43.0 mm
- net /PhaseMosfets2/PL: track 41.8 -> 42.9 mm
- net /PhaseMosfets3/PL: track 41.8 -> 42.4 mm
- net -BATT: vias 203 -> 189
Other:
- board text added: "Center X: 137.5 Y: 79"
- board text removed: "Center X: 137.5 Y: 80"

Commit message: fix
Parts:
- removed C29, C35, C36, C39, C41, C42, C44, C46, C47: 100n, GigaVescLibs:C_0603_1608Metric_L
- removed C34, C40, C45: 2.2u, GigaVescLibs:C_0603_1608Metric_L
- removed L1, L2, L3: BLM18HE152SN1D, Inductor_SMD:L_0603_1608Metric
- removed U1, U5, U7: RS2166XC5, Package_TO_SOT_SMD:SOT-353_SC-70-5
- removed U2, U3, U6: ACS773ECB-200B-PFF-T, GigaVescLibs:Allegro_CB_SMD
- added JP1: DummyJumper, GigaVescLibs:SolderJumper0.3mm, F.Cu at (194.5, 110.0)
- added JP2: DummyJumper, GigaVescLibs:SolderJumper0.3mm, F.Cu at (148.8, 110.0)
- added JP3: DummyJumper, GigaVescLibs:SolderJumper0.3mm, F.Cu at (103.0, 110.0)
- added R22: 0.5m, Resistor_SMD:R_2512_6332Metric, F.Cu at (194.5, 107.8)
- added R23: 0.5m, Resistor_SMD:R_2512_6332Metric, F.Cu at (148.8, 107.8)
- added R24: 0.5m, Resistor_SMD:R_2512_6332Metric, F.Cu at (103.0, 107.8)
- added R25: 0.5m, Resistor_SMD:R_2512_6332Metric, F.Cu at (190.5, 107.8)
- added R26: 0.5m, Resistor_SMD:R_2512_6332Metric, F.Cu at (144.8, 107.8)
- added R27: 0.5m, Resistor_SMD:R_2512_6332Metric, F.Cu at (99.0, 107.8)
- added R28: 0.5m, Resistor_SMD:R_2512_6332Metric, F.Cu at (212.8, 107.8)
- added R29: 0.5m, Resistor_SMD:R_2512_6332Metric, F.Cu at (167.0, 107.8)
- added R30: 0.5m, Resistor_SMD:R_2512_6332Metric, F.Cu at (121.2, 107.8)
- added R31: 0.5m, Resistor_SMD:R_2512_6332Metric, F.Cu at (208.8, 107.8)
- added R32: 0.5m, Resistor_SMD:R_2512_6332Metric, F.Cu at (163.0, 107.8)
- added R33: 0.5m, Resistor_SMD:R_2512_6332Metric, F.Cu at (117.2, 107.8)
- moved C18 78.5 mm to (116.0, 150.0), turned to -90 degrees
- moved C10 78.3 mm to (161.8, 150.0), turned to -90 degrees
- moved C2 78.2 mm to (207.5, 150.0), turned to -90 degrees
- moved C20 75.7 mm to (119.2, 150.0), turned to -90 degrees
- moved C12 75.4 mm to (165.0, 150.0), turned to -90 degrees
- moved C4 75.2 mm to (210.8, 150.0), turned to -90 degrees
- moved C17 73.4 mm to (116.0, 145.3), turned to -90 degrees
- moved C9 73.3 mm to (161.8, 145.3), turned to -90 degrees
- moved C1 73.3 mm to (207.5, 145.3), turned to -90 degrees
- moved C19 70.3 mm to (119.2, 145.3), turned to -90 degrees
- moved C11 70.2 mm to (165.0, 145.3), turned to -90 degrees
- moved C3 70.1 mm to (210.8, 145.3), turned to -90 degrees
- moved J11 49.6 mm to (108.5, 73.5), turned to -90 degrees
- moved J10 48.8 mm to (154.3, 73.5), turned to -90 degrees
- moved J7 48.0 mm to (200.0, 73.5), turned to -90 degrees
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Connections:
- J10 pad 1: /PhaseMosfets2/PHASE_OUT -> /PhaseMosfets2/PHASE
- J11 pad 1: /PhaseMosfets3/PHASE_OUT -> /PhaseMosfets3/PHASE
- J4 pad 3: /PhaseMosfets1/SENSE_FILTER_EN -> /PhaseMosfets1/SH-
- J4 pad 6: /PhaseMosfets1/CURRENT_SENSE -> /PhaseMosfets1/SH+
- J5 pad 3: /PhaseMosfets2/SENSE_FILTER_EN -> /PhaseMosfets2/SH-
- J5 pad 6: /PhaseMosfets2/CURRENT_SENSE -> /PhaseMosfets2/SH+
- J6 pad 3: /PhaseMosfets3/SENSE_FILTER_EN -> /PhaseMosfets3/SH-
- J6 pad 6: /PhaseMosfets3/CURRENT_SENSE -> /PhaseMosfets3/SH+
- J7 pad 1: /PhaseMosfets1/PHASE_OUT -> /PhaseMosfets1/PHASE
- Q10 pad 3: -BATT -> /PhaseMosfets3/SH+
- Q12 pad 3: -BATT -> /PhaseMosfets3/SH+
- Q2 pad 3: -BATT -> /PhaseMosfets1/SH+
- Q4 pad 3: -BATT -> /PhaseMosfets1/SH+
- Q6 pad 3: -BATT -> /PhaseMosfets2/SH+
- Q8 pad 3: -BATT -> /PhaseMosfets2/SH+
- R1 pad 1: /PhaseMosfets1/PHASE_OUT -> /PhaseMosfets1/PHASE
- R13 pad 1: /PhaseMosfets2/PHASE_OUT -> /PhaseMosfets2/PHASE
- R20 pad 1: /PhaseMosfets3/PHASE_OUT -> /PhaseMosfets3/PHASE
Routing:
- net -BATT: track 46.9 -> 0.00 mm, vias 189 -> 0
- net /PhaseMosfets3/PH: track 44.5 -> 0.00 mm
- net /PhaseMosfets2/PH: track 44.5 -> 0.00 mm
- net /PhaseMosfets1/PH: track 44.5 -> 0.00 mm
- net /PhaseMosfets1/PL: track 43.0 -> 0.00 mm
- net /PhaseMosfets2/PL: track 42.9 -> 0.00 mm
- net /PhaseMosfets3/PL: track 42.4 -> 0.00 mm
- net /PhaseMosfets3/3.3V_IN: track 39.3 -> 0.00 mm
- net /PhaseMosfets2/3.3V_IN: track 37.6 -> 0.00 mm
- net /PhaseMosfets1/3.3V_IN: track 35.8 -> 0.00 mm
- net /PhaseMosfets3/MOS_TEMP: track 35.3 -> 0.00 mm
- net /PhaseMosfets2/MOS_TEMP: track 33.6 -> 0.00 mm
- net /PhaseMosfets1/MOS_TEMP: track 31.6 -> 0.00 mm
- net /PhaseMosfets3/V_SENSE: track 27.8 -> 0.00 mm, vias 2 -> 0
- net /PhaseMosfets2/V_SENSE: track 25.8 -> 0.00 mm, vias 2 -> 0
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- removed copper zone on B.Cu, net /PhaseMosfets1/PHASE
- removed copper zone on F.Cu, net /PhaseMosfets1/PHASE
- removed copper zone on F.Cu, net /PhaseMosfets1/PHASE_OUT
- removed copper zone on B.Cu, net /PhaseMosfets2/PHASE
- removed copper zone on F.Cu, net /PhaseMosfets2/PHASE
- removed copper zone on F.Cu, net /PhaseMosfets2/PHASE_OUT
- removed copper zone on B.Cu, net /PhaseMosfets3/PHASE
- removed copper zone on F.Cu, net /PhaseMosfets3/PHASE
- removed copper zone on F.Cu, net /PhaseMosfets3/PHASE_OUT
- removed copper zone on F.Cu, net Net-(C1-Pad2)
- removed copper zone on F.Cu, net Net-(C10-Pad1)
- removed copper zone on F.Cu, net Net-(C11-Pad2)
- removed copper zone on F.Cu, net Net-(C13-Pad2)
- removed copper zone on F.Cu, net Net-(C15-Pad2)
- removed copper zone on F.Cu, net Net-(C25-Pad2)
- removed copper zone on F.Cu, net Net-(C27-Pad2)
- removed copper zone on F.Cu, net Net-(C3-Pad2)
- removed copper zone on F.Cu, net Net-(C30-Pad2)
- removed copper zone on F.Cu, net Net-(C32-Pad2)
- removed copper zone on F.Cu, net Net-(C48-Pad2)
- removed copper zone on F.Cu, net Net-(C5-Pad2)
- removed copper zone on F.Cu, net Net-(C50-Pad2)
- removed copper zone on F.Cu, net Net-(C52-Pad2)
- removed copper zone on F.Cu, net Net-(C54-Pad2)
- removed copper zone on F.Cu, net Net-(C7-Pad2)
