File: MosfetBoard/IXTT220N20X4HV/PhaseMosfets.kicad_sch (KiCad schematic)
At the start: 20 parts, among them Q1 IXTT220N20X4HV, Q2 IXTT220N20X4HV, Q4 IXTT220N20X4HV, Q5 IXTT220N20X4HV, U1 RS2166XC5, U3 ACS773ECB-200B-PFF-T

Commit message: wholeDevice
Parts:
- added C1 (x16): 10u 100V, Capacitor_SMD:C_1210_3225Metric, symbol Device:C
- added J1: DRIVER1, Connector_PinSocket_2.54mm:PinSocket_2x02_P2.54mm_Vertical_SMD, symbol Connector_Generic:Conn_01x04
- added J12: PhasePad, Connector_Wire:SolderWirePad_1x01_SMD_5x10mm, symbol Connector:Conn_01x01_Pin
- added J4: PhaseConn, Connector_PinSocket_2.54mm:PinSocket_2x03_P2.54mm_Vertical_SMD, symbol Connector_Generic:Conn_02x03_Counter_Clockwise
- C29, C35, C36: value 100nF -> 100n; footprint Capacitor_SMD:C_0805_2012Metric -> GigaVescLibs:C_0603_1608Metric_L; MPN C28233 -> C14663
- C34: footprint Capacitor_SMD:C_0805_2012Metric -> GigaVescLibs:C_0603_1608Metric_L; MPN C49217 -> C23630
- C37: footprint Capacitor_SMD:C_0805_2012Metric -> GigaVescLibs:C_0603_1608Metric_L; MPN C28323 -> C15849
- R1: footprint Resistor_SMD:R_0805_2012Metric -> Resistor_SMD:R_0603_1608Metric; MPN C17470 -> C22807
- R10, R11, R12, R9: value 2r2 -> 2.2
- R2: footprint Resistor_SMD:R_0805_2012Metric -> Resistor_SMD:R_0603_1608Metric; MPN C17530 -> C13167
- R3: footprint Resistor_SMD:R_0805_2012Metric -> Resistor_SMD:R_0603_1608Metric; MPN C17414 -> C25804
Connections:
- net +BATT: now also C1.1, C1.1, C1.1, C1.1, C1.1, C1.1, C1.1, C1.1
- net -BATT: now also C1.2, C1.2, C1.2, C1.2, C1.2, C1.2, C1.2, C1.2, J1.4 (Pin_4)
- net GND: now also J4.1 (Pin_1)
- net PH: now also J1.1 (Pin_1)
- net PHASE: now also J1.3 (Pin_3)
- net PHASE_OUT: now also J12.1 (Pin_1)
- net PL: now also J1.2 (Pin_2)
- net SENSE_FILTER_EN: now also J4.3 (Pin_3)
- net +3.3V renamed 3.3V_IN
- net 3.3V_IN: now also J4.5 (Pin_5)
- net CURR renamed CURRENT_SENSE
- net CURRENT_SENSE: now also J4.6 (Pin_6)
- net MOSTEMP renamed MOS_TEMP
- net MOS_TEMP: now also J4.4 (Pin_4)
- net VSENSE renamed V_SENSE
- net V_SENSE: now also J4.2 (Pin_2)
- new net: C1.1, C1.2 (x8)
Other:
- note added: "Sense filter enable is connected on logic board"

Commit message: fix
Parts:
- removed C29, C35, C36: 100n, GigaVescLibs:C_0603_1608Metric_L, symbol Device:C
- removed C34: 2.2u, GigaVescLibs:C_0603_1608Metric_L, symbol Device:C
- removed L1: BLM18HE152SN1D, Inductor_SMD:L_0603_1608Metric, symbol Device:L
- removed U1: RS2166XC5, Package_TO_SOT_SMD:SOT-353_SC-70-5, symbol GigaESCSymbols:RS2166XC5
- removed U3: ACS773ECB-200B-PFF-T, GigaVescLibs:Allegro_CB_SMD, symbol Sensor_Current:ACS770xCB-200B-PSF
- added JP1: DummyJumper, GigaVescLibs:SolderJumper0.3mm, symbol Jumper:Jumper_2_Bridged
- added R22, R25, R28, R31: 0.5m, Resistor_SMD:R_2512_6332Metric, symbol Device:R_US
Connections:
- net PHASE_OUT is gone; now on net PHASE: J12.1 (Pin_1), R1.1
- net -BATT: now also JP1.1 (A), R22.2, R25.2, R28.2, R31.2; no longer Q4.3 (S), Q5.3 (S)
- net CURRENT_SENSE renamed SH+
- net SH+: now also Q4.3 (S), Q5.3 (S), R22.1, R25.1, R28.1, R31.1
- net SENSE_FILTER_EN renamed SH-
- net SH-: now also JP1.2 (B)
Other:
- note added: "Total 0.000125Ω"
- note removed: "Sense filter enable is connected on logic board"
- moved on the sheet: C37, J12, R1, R2, R3, TH1
