File: PowerBoard/LT8316/LT8316.kicad_pcb (KiCad board)
At the start: 2 copper layers, 45 x 100 mm, 42 parts, among them J1 AuxConn, Q1 STD11N65M2, SW1 POWER_SW, T1 11328-T078, U2 LT8316EFE#PBF

Commit message: fixeddimensions
Parts:
- removed C1, C2: 2200uF 200V, Capacitor_THT:CP_Radial_D30.0mm_P10.00mm_SnapIn
- removed H1, H2, H3, H4: BATT-Hole, MountingHole:MountingHole_3.2mm_M3
- added C18: 330u 200V, Capacitor_THT:CP_Radial_D18.0mm_P7.50mm, F.Cu at (64.0, 83.0)
- added C19: 330u 200V, Capacitor_THT:CP_Radial_D18.0mm_P7.50mm, F.Cu at (75.5, 82.5)
- added C20: 330u 200V, Capacitor_THT:CP_Radial_D18.0mm_P7.50mm, F.Cu at (64.0, 63.5)
- added C21: 330u 200V, Capacitor_THT:CP_Radial_D18.0mm_P7.50mm, F.Cu at (76.5, 61.0)
- added C5: 330u 200V, Capacitor_THT:CP_Radial_D18.0mm_P7.50mm, F.Cu at (64.0, 101.5)
- added C6: 330u 200V, Capacitor_THT:CP_Radial_D18.0mm_P7.50mm, F.Cu at (75.5, 101.5)
- C12: value 47p 100V -> 47p; footprint Capacitor_SMD:C_0603_1608Metric -> Capacitor_SMD:C_0805_2012Metric
- C8: footprint Capacitor_SMD:C_0805_2012Metric -> Capacitor_SMD:C_1206_3216Metric
- R10: value 121k -> 120k
- R11: value 4.99k -> 6.2k
- R12: value 44.2k -> 56k
- R3: value 499k -> 470k; footprint Resistor_SMD:R_1206_3216Metric -> Resistor_SMD:R_0805_2012Metric
- R7: value 56.2k -> 56k
- moved R4 44.3 mm to (93.5, 94.0), turned to 90 degrees
- moved SW1 40.6 mm to (91.0, 93.5), turned to 90 degrees
- moved R16 28.1 mm to (82.8, 90.5)
- moved D5 26.6 mm to (66.5, 136.0), turned to 180 degrees
- moved R3 23.7 mm to (79.2, 91.5), turned to 0 degrees
- moved C16 22.0 mm to (88.0, 130.5), turned to 180 degrees
- moved C15 21.3 mm to (66.0, 132.0), turned to 180 degrees
- moved D4 16.2 mm to (73.0, 135.8), turned to 0 degrees
- moved J1 6.52 mm to (92.0, 112.0)
- moved R6 3.64 mm to (56.5, 95.0)
- moved C7 3.54 mm to (78.0, 107.0)
- moved R14 3.51 mm to (63.8, 98.5)
- moved C14 3.20 mm to (87.5, 114.5), turned to 0 degrees
- moved R11 3.20 mm to (56.5, 97.0), turned to 180 degrees
- moved C8 2.76 mm to (79.2, 111.2)
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Routing:
- net Net-(SW1-B): track 14.4 -> 38.3 mm, vias 0 -> 3
- net +12V: track 13.8 -> 35.1 mm, vias 12 -> 5
- net Net-(SW1-C): track 21.4 -> 11.6 mm, vias 1 -> 0
- net Net-(Q1-S): track 0.00 -> 7.22 mm
- net -BATT: track 31.8 -> 24.7 mm, vias 110 -> 90
- net +BATT: track 24.7 -> 31.8 mm, vias 12 -> 6
- net Net-(Q1-G): track 8.85 -> 2.35 mm
- net IN_V: track 22.0 -> 15.7 mm
- net Net-(U2-SENSE): track 21.6 -> 17.7 mm
- net GND: track 61.3 -> 64.4 mm, vias 9 -> 2
- net Net-(U2-VC): track 8.12 -> 6.12 mm
- net Net-(D1-A): track 37.0 -> 36.1 mm
- net Net-(U2-GATE): track 16.6 -> 15.8 mm
- net Net-(SW1-A): track 2.09 -> 2.70 mm
- net Net-(D2-K): track 4.56 -> 4.06 mm
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- removed copper zone on B.Cu, net GND
- removed copper zone on F.Cu, net Net-(D4-A-Pad1)
Other:
- board text added: "Center: X: 72.5 Y: 100"
- board text added: "GigaESC PowerBoard v1.0.0 - LT8316"

Commit message: small changes for lt
Parts:
- C10: value 47p 25V -> 47p; footprint Capacitor_SMD:C_0805_2012Metric -> GigaVescLibs:C_0603_1608Metric_L
- C12, C9: footprint Capacitor_SMD:C_0805_2012Metric -> GigaVescLibs:C_0603_1608Metric_L
- C14: footprint Capacitor_SMD:C_0805_2012Metric -> Capacitor_SMD:C_0603_1608Metric
- R1, R10, R11, R12, R13, R14, R16, R2, R3, R4, R6: footprint Resistor_SMD:R_0805_2012Metric -> Resistor_SMD:R_0603_1608Metric
- moved C15 26.2 mm to (90.2, 122.0)
- moved D5 25.5 mm to (90.0, 126.0)
- moved D4 18.6 mm to (91.0, 131.2), turned to -90 degrees
- moved R3 13.5 mm to (91.2, 97.8)
- moved R16 11.1 mm to (92.2, 96.2), turned to 180 degrees
- moved C8 6.50 mm to (79.0, 104.8)
- moved C14 3.50 mm to (87.5, 111.0)
- moved J1 3.50 mm to (92.0, 108.5)
- moved C13 2.80 mm to (57.0, 88.8), turned to 180 degrees
- moved C7 2.50 mm to (79.5, 109.0)
- moved R10 1.58 mm to (59.5, 95.5)
- moved R11 1.50 mm to (56.5, 95.5)
- moved C9 1.41 mm to (57.2, 91.2)
- moved R12 1.12 mm to (59.5, 94.0)
- moved R14 1.06 mm to (63.0, 97.8)
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Routing:
- net Net-(D4-A-Pad1): track 0.00 -> 25.4 mm
- net +12V: track 35.1 -> 14.6 mm, vias 5 -> 4
- net -BATT: track 24.7 -> 19.2 mm, vias 90 -> 99
- net IN_V: track 15.7 -> 11.8 mm
- net Net-(U2-SENSE): track 17.7 -> 14.4 mm
- net Net-(U2-FB): track 7.56 -> 5.90 mm
- net Net-(U2-TC): track 4.07 -> 2.81 mm
- net Net-(Q1-S): track 7.22 -> 8.37 mm
- net Net-(SW1-C): track 11.6 -> 10.4 mm, vias 0 -> 1
- net GND: track 64.4 -> 65.2 mm, vias 2 -> 6
- net Net-(C9-Pad1): track 2.07 -> 2.58 mm
- net +BATT: track 31.8 -> 32.0 mm, vias 6 -> 5
- removed copper zone on B.Cu, net +12V
- removed copper zone on F.Cu, net +12V
- removed copper zone on B.Cu, net Net-(D4-A-Pad1)
Other:
- outline, holes or cut-outs redrawn

Commit message: fix
Parts:
- R1: value 100k -> 150k
- R2: value 1.8k -> 2.7k
Changed lines of the file:
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@@
     (descr "Resistor SMD 0603 (1608 Metric), square (rectangular) end terminal, IPC_7351 nominal, (Body size source: IPC-SM-782 page 72, https://www.pcb-3d.com/wordpress/wp-content/uploads/ipc-sm-782a_amendment_1_and_2.pdf), generated with kicad-footprint-generator")
     (tags "resistor")
-    (property "MPN" "C25803")
+    (property "MPN" "C22807")
     (property "Mouser" "603-RC0805FR-07100KL")
     (property "Sheetfile" "LT8316.kicad_sch")
@@
         (effects (font (size 1 1) (thickness 0.15)) (justify mirror))
     )
-    (fp_text value "100k" (at 0 -1.43 180) (layer "B.Fab")
+    (fp_text value "150k" (at 0 -1.43 180) (layer "B.Fab")
         (effects (font (size 1 1) (thickness 0.15)) (justify mirror))
     )
@@
     (descr "Resistor SMD 0603 (1608 Metric), square (rectangular) end terminal, IPC_7351 nominal, (Body size source: IPC-SM-782 page 72, https://www.pcb-3d.com/wordpress/wp-content/uploads/ipc-sm-782a_amendment_1_and_2.pdf), generated with kicad-footprint-generator")
     (tags "resistor")
-    (property "MPN" "C4177")
+    (property "MPN" "C13167")
     (property "Mouser" "71-CRCW0805-1.8K-E3")
     (property "Sheetfile" "LT8316.kicad_sch")
@@
         (effects (font (size 1 1) (thickness 0.15)) (justify mirror))
     )
-    (fp_text value "1.8k" (at 0 -1.43 270) (layer "B.Fab")
+    (fp_text value "2.7k" (at 0 -1.43 270) (layer "B.Fab")
         (effects (font (size 1 1) (thickness 0.15)) (justify mirror))
     )
