File: LogicBoard/DevKit/ESP32BT.kicad_sch (KiCad schematic)
At the start: 16 parts, among them J1 USBC Socket, J15 ESPUartConn, J17 Micro_SD_Card_Det1, U10 ESP32-C3-WROOM-02-N4

Commit message: initialv2
Parts:
- added D8: 1N5819WS, Diode_SMD:D_SOD-323, symbol Device:D_Schottky
Connections:
- net CAN_TX is gone; now on net CAN2_RX: D7.2 (A), R28.2
- net CAN_RX renamed CAN2_RX
- net CAN2_RX: now also D8.2 (A)
- new net CAN2_TX: D8.1 (K)
Changed lines of the file:
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@@
 (kicad_sch (version 20230121) (generator eeschema)
   (paper "A4")
+  (junction (at 73.66 67.31) (diameter 0) (color 0 0 0 0)
+  )
+  (junction (at 73.66 64.77) (diameter 0) (color 0 0 0 0)
+  )
   (junction (at 107.95 46.99) (diameter 0) (color 0 0 0 0)
   )
   (junction (at 199.39 71.12) (diameter 0) (color 0 0 0 0)
-  )
-  (junction (at 73.66 67.31) (diameter 0) (color 0 0 0 0)
   )
   (junction (at 184.15 96.52) (diameter 0) (color 0 0 0 0)
@@
     (stroke (width 0) (type default))
   )
+  (wire (pts (xy 73.66 64.77) (xy 113.03 64.77))
+    (stroke (width 0) (type default))
+  )
   (wire (pts (xy 205.74 64.77) (xy 205.74 49.53))
     (stroke (width 0) (type default))
@@
     (stroke (width 0) (type default))
   )
-  (wire (pts (xy 66.04 67.31) (xy 73.66 67.31))
-    (stroke (width 0) (type default))
-  )
-  (wire (pts (xy 66.04 64.77) (xy 113.03 64.77))
+  (wire (pts (xy 66.04 64.77) (xy 73.66 64.77))
     (stroke (width 0) (type default))
   )
@@
   )
   (wire (pts (xy 199.39 69.85) (xy 199.39 71.12))
+    (stroke (width 0) (type default))
+  )
+  (wire (pts (xy 73.66 64.77) (xy 73.66 67.31))
     (stroke (width 0) (type default))
   )
@@
     (effects (font (size 3.27 3.27)) (justify left bottom))
   )
-  (global_label "CAN_TX" (shape input) (at 66.04 67.31 180) (fields_autoplaced)
-    (effects (font (size 1.27 1.27)) (justify right))
-    (property "Intersheetrefs" "${INTERSHEET_REFS}" (at 56.9546 67.31 0)
-      (effects (font (size 1.27 1.27)) (justify right) hide)
-    )
-  )
   (global_label "ESP_FAULT_LED" (shape input) (at 158.75 138.43 180) (fields_autoplaced)
     (effects (font (size 1.27 1.27)) (justify right))
@@
     )
   )
-  (global_label "CAN_RX" (shape input) (at 66.04 64.77 180) (fields_autoplaced)
-    (effects (font (size 1.27 1.27)) (justify right))
-    (property "Intersheetrefs" "${INTERSHEET_REFS}" (at 56.6522 64.77 0)
+  (global_label "CAN2_TX" (shape input) (at 66.04 67.31 180) (fields_autoplaced)
+    (effects (font (size 1.27 1.27)) (justify right))
+    (property "Intersheetrefs" "${INTERSHEET_REFS}" (at 55.7451 67.31 0)
       (effects (font (size 1.27 1.27)) (justify right) hide)
     )
@@
     (property "Intersheetrefs" "${INTERSHEET_REFS}" (at 158.5825 69.85 0)
       (effects (font (size 1.27 1.27)) (justify left) hide)
+    )
+  )
+  (global_label "CAN2_RX" (shape input) (at 66.04 64.77 180) (fields_autoplaced)
+    (effects (font (size 1.27 1.27)) (justify right))
+    (property "Intersheetrefs" "${INTERSHEET_REFS}" (at 55.4427 64.77 0)
+      (effects (font (size 1.27 1.27)) (justify right) hide)
     )
   )
@@
         )
       )
+    )
+  )
+  (symbol (lib_id "Device:D_Schottky") (at 69.85 67.31 0) (unit 1)
+    (in_bom yes) (on_board yes) (dnp no)
+    (property "Reference" "D8" (at 68.58 73.66 0)
+      (effects (font (size 1.27 1.27)))
+    )
+    (property "Value" "1N5819WS" (at 64.77 71.12 0)
+      (effects (font (size 1.27 1.27)))
+    )
+    (property "Footprint" "Diode_SMD:D_SOD-323" (at 69.85 67.31 0)
+      (effects (font (size 1.27 1.27)) hide)
+    )
+    (property "Datasheet" "~" (at 69.85 67.31 0)
+      (effects (font (size 1.27 1.27)) hide)
+    )
+    (property "MPN" "C191023" (at 69.85 67.31 0)
+      (effects (font (size 1.27 1.27)) hide)
+    )
+    (pin "1")
+    (pin "2")
+    (instances
+      (project "DevKit"
+        (path "/768a484b-8a27-40cf-8cad-0f63935b1af0/72793ee1-8b24-4ded-a030-5a38e70b572c"
+          (reference "D8") (unit 1)
+        )
+      )

Commit message: v2
Parts:
- added R3, R4: 22, Resistor_SMD:R_0603_1608Metric, symbol Device:R
- added U7: USBLC6-2SC6, Package_TO_SOT_SMD:SOT-23-6, symbol Power_Protection:USBLC6-2P6
- C45: footprint Capacitor_SMD:C_0603_1608Metric -> GigaVescLibs:C_0603_1608Metric_L
- J15: JLCPosOffset 3,0 -> -3,0; JLCRotOffset 0 -> 180
- J17: value Micro_SD_Card_Det1 -> MicroSD; JLCPosOffset (none) -> 0.3,2.2
- U10: JLCPosOffset (none) -> 0,-3.1
Connections:
- net ESP_USB_D+: now also R4.2; no longer J1.A6 (D+), J1.B6 (D+)
- net ESP_USB_D-: now also R3.2; no longer J1.A7 (D-), J1.B7 (D-)
- net GND: now also U7.2 (GND)
- net at J1.A4 (VBUS), J1.A9 (VBUS), J1.B4 (VBUS)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: now also U7.5 (VBUS)
- new net: R4.1, U7.1 (I/O1)
- new net: R3.1, U7.3 (I/O2)
- new net: J1.A7 (D-), J1.B7 (D-), U7.4 (I/O2)
- new net: J1.A6 (D+), J1.B6 (D+), U7.6 (I/O1)
- no-connect marks 5 -> 4
Other:
- note added: "Can be ommited on budget connect line 1-6 and 3-4"

Commit message: v2.10.0 - Low side shunt and hall sensor - current filters
Parts:
- J17: JLCPosOffset 0.3,2.2 -> 0,2.54
Changed lines of the file:
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@@
       (effects (font (size 1.27 1.27)) hide)
     )
-    (property "JLCPosOffset" "0.3,2.2" (at 114.3 134.62 0)
+    (property "JLCPosOffset" "0,2.54" (at 114.3 134.62 0)
       (effects (font (size 1.27 1.27)) hide)
     )

Commit message: v3.2.0 - Moving to kicad 8
Parts:
- renumbered C45 to C46, J1 to J13, R4 to R27, R3 to R29, R28 to R34, R5 to R35, R6 to R40, R28 to R41, R28 to R42, U7 to U8

Commit message: v3.2.2 - TL494V2
Parts:
- removed J13: USBC Socket, Connector_USB:USB_C_Receptacle_GCT_USB4105-xx-A_16P_TopMnt_Horizontal, symbol Connector:USB_C_Receptacle_USB2.0
- removed U8: USBLC6-2SC6, Package_TO_SOT_SMD:SOT-23-6, symbol Power_Protection:USBLC6-2P6
- added J13: USBC Socket, Connector_USB:USB_C_Receptacle_GCT_USB4105-xx-A_16P_TopMnt_Horizontal, symbol Connector:USB_C_Receptacle_USB2.0_16P
- added U8: USBLC6-2SC6, Package_TO_SOT_SMD:SOT-23-6, symbol Power_Protection:USBLC6-2SC6
Connections:
- net GND: now also J13.A1 (GND), J13.A12 (GND), J13.B1 (GND), J13.B12 (GND), J13.S1 (SHIELD), U8.2 (GND)
- net at R40.2: now also J13.B5 (CC2)
- net at R35.2: now also J13.A5 (CC1)
- net at R27.1: now also U8.1 (I/O1)
- net at R29.1: now also U8.3 (I/O2)
- new net: J13.A7 (D-), J13.B7 (D-), U8.4 (I/O2)
- new net: J13.A4 (VBUS), J13.A9 (VBUS), J13.B4 (VBUS), J13.B9 (VBUS), U8.5 (VBUS)
- new net: J13.A6 (D+), J13.B6 (D+), U8.6 (I/O1)
Other:
- moved on the sheet: R27, R29
