File: Supervisor/RS323.kicad_sch (KiCad schematic)
At the start: 10 parts, among them U5 MAX3232

Commit message: cleanup
Parts:
- removed C11, C12, C13, C14, C15: 100n, Capacitor_SMD:C_0603_1608Metric, symbol Device:C
- removed D5, D6: ESD9B3.3ST5G, Diode_SMD:D_SOD-923, symbol Diode:ESD9B3.3ST5G
- removed U5: MAX3232, Package_SO:SOIC-16_3.9x9.9mm_P1.27mm, symbol Interface_UART:MAX3232
Connections:
- no-connect marks 4 -> 0
