File: Supervisor/AnalogIO.kicad_sch (KiCad schematic)
At the start: 10 parts, among them U7 TLV2372

Commit message: cleanup
Parts:
- U7: MPN (none) -> C27204
Changed lines of the file:
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@@
+			)
+		)
+		(property "MPN" "C27204"
+			(at 165.1 90.17 0)
+			(effects
+				(font
+					(size 1.27 1.27)
+				)
+				(hide yes)
 			)
 		)
@@
 			)
 		)
+		(property "MPN" "C27204"
+			(at 96.52 66.04 0)
+			(effects
+				(font
+					(size 1.27 1.27)
+				)
+				(hide yes)
+			)
+		)
 		(pin "7"
 		)
@@
 			(at 96.52 104.14 0)
 			(effects
+				(font
+					(size 1.27 1.27)
+				)
+				(hide yes)
+			)
+		)
+		(property "MPN" "C27204"
+			(at 96.52 104.14 0)
+			(effects
