File: PowerBoard/TL494V2OC/TL494V2OC.kicad_pcb (KiCad board)
At the start: 2 copper layers, 50 x 75 mm, 66 parts, among them J1 AuxConn, Q1 MMBTA92, Q2 CPC3980, Q5 IRFS4227TRLPBF, U1 TL494, U3 IR2181, U4 TL431

Commit message: v3.3.1 - Supervisor routed
Parts:
- removed R15: 10k, Resistor_SMD:R_0603_1608Metric
- added R27: 10m, Resistor_SMD:R_2512_6332Metric, F.Cu at (83.8, 131.5)
- added R28: 20k, Resistor_SMD:R_0603_1608Metric, B.Cu at (63.8, 105.5)
- added U2: INA213, Package_TO_SOT_SMD:SOT-363_SC-70-6, B.Cu at (76.2, 104.8)
- R9: value 100 -> 5.1k
- moved D5 18.8 mm to (83.2, 136.5), turned to 0 degrees
- moved C13 11.9 mm to (94.8, 131.8), turned to -90 degrees
- moved C16 9.72 mm to (92.2, 131.8)
- moved C10 3.47 mm to (89.8, 127.0)
- moved C14 3.47 mm to (87.2, 127.0)
- moved C17 3.47 mm to (94.8, 127.0)
- moved C2 3.47 mm to (92.2, 127.0)
- moved R9 0.90 mm to (66.0, 104.8), turned to 90 degrees
- moved C8 0.50 mm to (82.5, 105.5)
- moved D3 0.50 mm to (85.0, 106.5)
- moved R18 0.50 mm to (79.5, 105.5)
- moved R19 0.50 mm to (82.5, 104.0)
Connections:
- D5 pad 1: +12V -> Net-(D5-K)
- L1 pad 2: +12V -> Net-(D5-K)
- R9 pad 1: -BATT -> CFB-
- R9 pad 2: Net-(U1-2IN+) -> -BATT
- U1 pad 15: Net-(U1-2IN-) -> CFB-
- U1 pad 16: Net-(U1-2IN+) -> CFB
Routing:
- net Net-(D5-K): track 0.00 -> 38.4 mm, vias 0 -> 6
- net +12V: track 44.2 -> 75.5 mm, vias 2 -> 5
- net CFB: track 0.00 -> 7.79 mm
- net Net-(U1-2IN-): track 7.34 -> 0.00 mm
- net CFB-: track 0.00 -> 4.46 mm
- net Net-(U1-FB): track 5.94 -> 2.27 mm
- net STARTUP: track 65.3 -> 67.9 mm, vias 4 -> 5
- net Net-(U1-2IN+): track 1.97 -> 0.00 mm
- net Net-(U1-REF): track 9.38 -> 10.8 mm
- net Net-(Q1-C): vias 3 -> 8
- net -BATT: vias 226 -> 231
- net +BATT: vias 126 -> 132
- added copper zone on F.Cu, net Net-(D5-K)

Commit message: cleanup
Other:
- board text added: "GigaESC PowerBoard v2.1.0 - TL494OC"
- board text removed: "GigaESC PowerBoard v2.1.0 - TL494"

Commit message: EPC board update
Connections:
- net Net-(Q1-B) renamed DRV-OUT
- net Net-(Q1-C) renamed /SW-NODE
