File: PowerBoard/TL494V2OC/TL494V2OC.kicad_sch (KiCad schematic)
At the start: 66 parts, among them J1 AuxConn, Q1 MMBTA92, Q2 CPC3980, Q5 IRFS4227TRLPBF, U1 TL494, U3 IR2181, U4 TL431

Commit message: v3.3.1 - Supervisor routed
Parts:
- removed R15: 10k, Resistor_SMD:R_0603_1608Metric, symbol Device:R
- added R27: 10m, Resistor_SMD:R_2512_6332Metric, symbol Device:R_US
- added R28: 20k, Resistor_SMD:R_0603_1608Metric, symbol Device:R
- added U2: INA213, Package_TO_SOT_SMD:SOT-363_SC-70-6, symbol Amplifier_Current:INA199xxDCK
- R9: value 100 -> 5.1k; MPN C22775 -> C23186; Mouser 603-RC0805FR-0744K2L -> (none)
Connections:
- net +12V: now also R27.2, U2.5 (-); no longer D5.1 (K), L1.2
- net -BATT: now also R9.2, U2.1 (REF), U2.2 (GND); no longer R9.1
- net STARTUP: now also U2.3 (V+)
- net at C20.1, R11.1, R22.1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: now also R28.1
- net CFB-: now reaches U1.15 (2IN-)
- net CFB-: now also R9.1, R28.2
- net CFB: now reaches U1.16 (2IN+)
- net CFB: now also U2.6; no longer R9.2
- new net: D5.1 (K), L1.2, R27.1, U2.4 (+)
Other:
- note added: "1.016V"
- note added: "2A * 0.01 * 50 = 1V"
- moved on the sheet: C21, R10, R11, R14

Commit message: cleanup
Parts:
- C20: MPN C14663 -> C96446
- U2: MPN (none) -> C129346
Other:
- note added: "or CPC3708 or CPC5603"
Changed lines of the file:
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@@
 		)
 	)
+	(text "or CPC3708\nor CPC5603"
+		(exclude_from_sim no)
+		(at 118.11 158.115 0)
+		(effects
+			(font
+				(size 1.27 1.27)
+			)
+		)
+	)
 	(text "Hot loop"
 		(exclude_from_sim no)
@@
 			)
 		)
-		(property "MPN" "C14663"
+		(property "MPN" "C96446"
 			(at -10.16 101.6 90)
 			(effects
@@
 			(effects
 				(font
+					(size 1.27 1.27)
+				)
+				(hide yes)
+			)
+		)
+		(property "MPN" "C129346"
+			(at 199.39 80.01 90)
+			(effects
+				(font

Commit message: EPC board update
Connections:
- net SW-NODE: now reaches C12.2, D2.1 (K), D2.2 (K), L1.1, Q1.3 (C), Q5.3 (S), R8.1, U3.6 (VS)
- net DRV-OUT: now reaches Q1.1 (B), R13.1, R8.2, U3.7 (HO)
- net IN_V renamed IN-V
Other:
- note added: "2.5V"
- note added: "Bulk Capacitors"
- note added: "DCDC Controller"
- note added: "Division up to 186V => 3.3V Those values have to be the same as on mosfet board"
- note added: "Input Voltage Divider"
- note added: "Mounting Holes"
- note added: "Needs a little leg bending"
- note added: "Output caps 179uF"
- note added: "Resettable Fuse"
- note added: "Startup Circuit"
- note removed: "Division up to 186V => 3.3V !!Those values have to be the same as on mosfet board!!"
- note removed: "For 100x220 enclosure"
- note removed: "Needs a lil' leg bending"
- note removed: "Power supply for 200V applications"
- title: (none) -> Power supply for 200V applications
- moved on the sheet: C10, C12, C13, C14, C15, C16, C17, C2, C20, C21, C25, C26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
